Commit message: 古いGazeboの記述を削除

File: urdf/sciurus17_body.xacro (robot description, xacro)
@@ -72,13 +72,4 @@
       </collision>
     </link>
-    <gazebo reference="${NAME_LINK_BASE}">
-      <material>Gazebo/White</material>
-    </gazebo>
-    <gazebo reference="${NAME_LINK_BODY}">
-      <material>Gazebo/White</material>
-    </gazebo>
-    <gazebo reference="${NAME_LINK_CHEST_CAMERA}">
-      <material>Gazebo/Black</material>
-    </gazebo>
   </xacro:macro>
 </robot>

File: urdf/sciurus17_head.xacro (robot description, xacro)
@@ -84,13 +84,4 @@
       </collision>
     </link>
-    <gazebo reference="${NAME_LINK_NECK_1}">
-      <material>Gazebo/White</material>
-    </gazebo>
-    <gazebo reference="${NAME_LINK_NECK_2}">
-      <material>Gazebo/White</material>
-    </gazebo>
-    <gazebo reference="${NAME_LINK_HEAD_CAMERA}">
-      <material>Gazebo/Black</material>
-    </gazebo>
   </xacro:macro>
 </robot>

File: urdf/sciurus17_left_arm.xacro (robot description, xacro)
@@ -50,5 +50,5 @@
         <origin rpy="0 -1.5708 0" xyz="0.0 0.0 0.0"/>
         <geometry>
-          <mesh filename="package://sciurus17_description/meshes/visual/L_Link2.stl" scale="-1.0 1.0 -1.0"/>
+          <mesh filename="package://sciurus17_description/meshes/visual/L_Link2.stl" scale="1.0 1.0 1.0"/>
         </geometry>
         <material name="${COLOR_LINK_ARM}"/>
@@ -57,5 +57,5 @@
         <origin rpy="0 -1.5708 0" xyz="0.0 0.0 0.0"/>
         <geometry>
-          <mesh filename="package://sciurus17_description/meshes/collision/L_Link2.stl" scale="-1.0 1.0 -1.0"/>
+          <mesh filename="package://sciurus17_description/meshes/collision/L_Link2.stl" scale="1.0 1.0 1.0"/>
         </geometry>
       </collision>
@@ -244,22 +244,4 @@
       <dynamics damping="1.0e-6" friction="0.8"/>
     </joint>
-    <gazebo reference="${NAME_LINK_ARM_L_1}">
-      <material>Gazebo/White</material>
-    </gazebo>
-    <gazebo reference="${NAME_LINK_ARM_L_2}">
-      <material>Gazebo/White</material>
-    </gazebo>
-    <gazebo reference="${NAME_LINK_ARM_L_3}">
-      <material>Gazebo/White</material>
-    </gazebo>
-    <gazebo reference="${NAME_LINK_ARM_L_4}">
-      <material>Gazebo/White</material>
-    </gazebo>
-    <gazebo reference="${NAME_LINK_ARM_L_5}">
-      <material>Gazebo/White</material>
-    </gazebo>
-    <gazebo reference="${NAME_LINK_ARM_L_6}">
-      <material>Gazebo/White</material>
-    </gazebo>
   </xacro:macro>
 </robot>

File: urdf/sciurus17_left_hand.xacro (robot description, xacro)
@@ -87,13 +87,4 @@
       </inertial>
     </link>
-    <gazebo reference="${NAME_LINK_ARM_L_7}">
-      <material>Gazebo/Red</material>
-    </gazebo>
-    <gazebo reference="${NAME_LINK_HAND_L_A}">
-      <material>Gazebo/Red</material>
-    </gazebo>
-    <gazebo reference="${NAME_LINK_HAND_L_B}">
-      <material>Gazebo/Red</material>
-    </gazebo>
   </xacro:macro>
 </robot>

File: urdf/sciurus17_right_arm.xacro (robot description, xacro)
@@ -82,12 +82,12 @@
         <origin rpy="1.5708 0 0" xyz="0.0 0.0 0.0"/>
         <geometry>
-          <mesh filename="package://sciurus17_description/meshes/visual/L_Link3.stl" scale="1.0 -1.0 1.0"/>
-        </geometry>
-        <material name="${COLOR_LINK_ARM}"/>
-      </visual>
-      <collision>
-        <origin rpy="1.5708 0 0" xyz="0.0 0.0 0.0"/>
-        <geometry>
-          <mesh filename="package://sciurus17_description/meshes/collision/L_Link3.stl" scale="1.0 -1.0 1.0"/>
+          <mesh filename="package://sciurus17_description/meshes/visual/L_Link3.stl" scale="1.0 1.0 1.0"/>
+        </geometry>
+        <material name="${COLOR_LINK_ARM}"/>
+      </visual>
+      <collision>
+        <origin rpy="1.5708 0 0" xyz="0.0 0.0 0.0"/>
+        <geometry>
+          <mesh filename="package://sciurus17_description/meshes/collision/L_Link3.stl" scale="1.0 1.0 1.0"/>
         </geometry>
       </collision>
@@ -244,22 +244,4 @@
       <dynamics damping="1.0e-6" friction="0.8"/>
     </joint>
-    <gazebo reference="${NAME_LINK_ARM_R_1}">
-      <material>Gazebo/White</material>
-    </gazebo>
-    <gazebo reference="${NAME_LINK_ARM_R_2}">
-      <material>Gazebo/White</material>
-    </gazebo>
-    <gazebo reference="${NAME_LINK_ARM_R_3}">
-      <material>Gazebo/White</material>
-    </gazebo>
-    <gazebo reference="${NAME_LINK_ARM_R_4}">
-      <material>Gazebo/White</material>
-    </gazebo>
-    <gazebo reference="${NAME_LINK_ARM_R_5}">
-      <material>Gazebo/White</material>
-    </gazebo>
-    <gazebo reference="${NAME_LINK_ARM_R_6}">
-      <material>Gazebo/White</material>
-    </gazebo>
   </xacro:macro>
 </robot>

File: urdf/sciurus17_right_hand.xacro (robot description, xacro)
@@ -89,13 +89,4 @@
       </inertial>
     </link>
-    <gazebo reference="${NAME_LINK_ARM_R_7}">
-      <material>Gazebo/Red</material>
-    </gazebo>
-    <gazebo reference="${NAME_LINK_HAND_R_A}">
-      <material>Gazebo/Red</material>
-    </gazebo>
-    <gazebo reference="${NAME_LINK_HAND_R_B}">
-      <material>Gazebo/Red</material>
-    </gazebo>
   </xacro:macro>
 </robot>
