Commit message: friction値を変更

File: urdf/sciurus17_body.xacro (robot description, xacro)
@@ -31,5 +31,5 @@
         velocity="${VELOCITY_LIMIT}"/>
       <axis xyz="0 0 1"/>
-      <dynamics damping="1.0e-6" friction="0.8"/>
+      <dynamics damping="1.0e-6" friction="0.01"/>
     </joint>
     <link name="body_link">

File: urdf/sciurus17_head.xacro (robot description, xacro)
@@ -12,5 +12,5 @@
         velocity="${VELOCITY_LIMIT}"/>
       <axis xyz="0 0 1"/>
-      <dynamics damping="1.0e-6" friction="0.8"/>
+      <dynamics damping="1.0e-6" friction="0.01"/>
     </joint>
     <link name="neck_yaw_link">
@@ -42,5 +42,5 @@
         velocity="${VELOCITY_LIMIT}"/>
       <axis xyz="0 -1 0"/>
-      <dynamics damping="1.0e-6" friction="0.8"/>
+      <dynamics damping="1.0e-6" friction="0.01"/>
     </joint>
     <link name="neck_pitch_link">

File: urdf/sciurus17_left_arm.xacro (robot description, xacro)
@@ -12,5 +12,5 @@
         velocity="${VELOCITY_LIMIT}"/>
       <axis xyz="0 1 0"/>
-      <dynamics damping="1.0e-6" friction="0.8"/>
+      <dynamics damping="1.0e-6" friction="0.01"/>
     </joint>
     <link name="l_link1">
@@ -44,5 +44,5 @@
         velocity="${VELOCITY_LIMIT}"/>
       <axis xyz="-1 0 0"/>
-      <dynamics damping="1.0e-6" friction="0.8"/>
+      <dynamics damping="1.0e-6" friction="0.01"/>
     </joint>
     <link name="l_link2">
@@ -76,5 +76,5 @@
         velocity="${VELOCITY_LIMIT}"/>
       <axis xyz="0 1 0"/>
-      <dynamics damping="1.0e-6" friction="0.8"/>
+      <dynamics damping="1.0e-6" friction="0.01"/>
     </joint>
     <link name="l_link3">
@@ -108,5 +108,5 @@
         velocity="${VELOCITY_LIMIT}"/>
       <axis xyz="0 0 1"/>
-      <dynamics damping="1.0e-6" friction="0.8"/>
+      <dynamics damping="1.0e-6" friction="0.01"/>
     </joint>
     <link name="l_link4">
@@ -140,5 +140,5 @@
         velocity="${VELOCITY_LIMIT}"/>
       <axis xyz="0 1 0"/>
-      <dynamics damping="1.0e-6" friction="0.8"/>
+      <dynamics damping="1.0e-6" friction="0.01"/>
     </joint>
     <link name="l_link5">
@@ -210,5 +210,5 @@
         velocity="${VELOCITY_LIMIT}"/>
       <axis xyz="0 0 1"/>
-      <dynamics damping="1.0e-6" friction="0.8"/>
+      <dynamics damping="1.0e-6" friction="0.01"/>
     </joint>
     <link name="l_link6">
@@ -242,5 +242,5 @@
         velocity="${VELOCITY_LIMIT}"/>
       <axis xyz="0 1 0"/>
-      <dynamics damping="1.0e-6" friction="0.8"/>
+      <dynamics damping="1.0e-6" friction="0.01"/>
     </joint>
   </xacro:macro>

File: urdf/sciurus17_left_gripper.xacro (robot description, xacro)
@@ -32,5 +32,5 @@
         velocity="${VELOCITY_LIMIT}"/>
       <axis xyz="0 0 1"/>
-      <dynamics damping="1.0e-6" friction="0.8"/>
+      <dynamics damping="1.0e-6" friction="0.01"/>
     </joint>
     <link name="l_gripperA_link">
@@ -65,5 +65,5 @@
       <axis xyz="0 0 -1"/>
       <mimic joint="l_gripper_joint" multiplier="1" offset="0"/>
-      <dynamics damping="1.0e-6" friction="0.8"/>
+      <dynamics damping="1.0e-6" friction="0.01"/>
     </joint>
     <link name="l_gripperB_link">

File: urdf/sciurus17_right_arm.xacro (robot description, xacro)
@@ -12,5 +12,5 @@
         velocity="${VELOCITY_LIMIT}"/>
       <axis xyz="0 -1 0"/>
-      <dynamics damping="1.0e-6" friction="0.8"/>
+      <dynamics damping="1.0e-6" friction="0.01"/>
     </joint>
     <link name="r_link1">
@@ -44,5 +44,5 @@
         velocity="${VELOCITY_LIMIT}"/>
       <axis xyz="-1 0 0"/>
-      <dynamics damping="1.0e-6" friction="0.8"/>
+      <dynamics damping="1.0e-6" friction="0.01"/>
     </joint>
     <link name="r_link2">
@@ -76,5 +76,5 @@
         velocity="${VELOCITY_LIMIT}"/>
       <axis xyz="0 -1 0"/>
-      <dynamics damping="1.0e-6" friction="0.8"/>
+      <dynamics damping="1.0e-6" friction="0.01"/>
     </joint>
     <link name="r_link3">
@@ -108,5 +108,5 @@
         velocity="${VELOCITY_LIMIT}"/>
       <axis xyz="0 0 1"/>
-      <dynamics damping="1.0e-6" friction="0.8"/>
+      <dynamics damping="1.0e-6" friction="0.01"/>
     </joint>
     <link name="r_link4">
@@ -140,5 +140,5 @@
         velocity="${VELOCITY_LIMIT}"/>
       <axis xyz="0 -1 0"/>
-      <dynamics damping="1.0e-6" friction="0.8"/>
+      <dynamics damping="1.0e-6" friction="0.01"/>
     </joint>
     <link name="r_link5">
@@ -210,5 +210,5 @@
         velocity="${VELOCITY_LIMIT}"/>
       <axis xyz="0 0 1"/>
-      <dynamics damping="1.0e-6" friction="0.8"/>
+      <dynamics damping="1.0e-6" friction="0.01"/>
     </joint>
     <link name="r_link6">
@@ -242,5 +242,5 @@
         velocity="${VELOCITY_LIMIT}"/>
       <axis xyz="0 -1 0"/>
-      <dynamics damping="1.0e-6" friction="0.8"/>
+      <dynamics damping="1.0e-6" friction="0.01"/>
     </joint>
   </xacro:macro>

File: urdf/sciurus17_right_gripper.xacro (robot description, xacro)
@@ -32,5 +32,5 @@
         velocity="${VELOCITY_LIMIT}"/>
       <axis xyz="0 0 1"/>
-      <dynamics damping="1.0e-6" friction="0.8"/>
+      <dynamics damping="1.0e-6" friction="0.01"/>
     </joint>
     <link name="r_gripperA_link">
@@ -66,5 +66,5 @@
       <axis xyz="0 0 -1"/>
       <mimic joint="r_gripper_joint" multiplier="1" offset="0"/>
-      <dynamics damping="1.0e-6" friction="0.8"/>
+      <dynamics damping="1.0e-6" friction="0.01"/>
     </joint>
     <link name="r_gripperB_link">
