Commit message: Gazeboのマテリアルを設定

File: urdf/sciurus17_gazebo.xacro (robot description, xacro)
@@ -1,156 +1,109 @@
 <?xml version="1.0"?>
 <robot xmlns:xacro="http://ros.org/wiki/xacro">
-  <xacro:macro name="default_transmission"
-    params="joint_name interface:=position">
-    <transmission name="${joint_name}_trans">
-      <provideFeedback>true</provideFeedback>
-      <implicitSpringDamper>0</implicitSpringDamper>
-      <motorTorqueConstant>0.418</motorTorqueConstant>
-      <type>transmission_interface/SimpleTransmission</type>
-      <joint name="${joint_name}">
-        <xacro:if value="${interface == 'position'}">
-          <hardwareInterface>hardware_interface/PositionJointInterface</hardwareInterface>
-        </xacro:if>
-        <xacro:if value="${interface == 'velocity'}">
-          <hardwareInterface>hardware_interface/VelocityJointInterface</hardwareInterface>
-        </xacro:if>
-        <xacro:if value="${interface == 'effort'}">
-          <hardwareInterface>hardware_interface/EffortJointInterface</hardwareInterface>
-        </xacro:if>
-      </joint>
-      <actuator name="{joint_name}_motor">
-        <xacro:if value="${interface == 'position'}">
-          <hardwareInterface>hardware_interface/PositionJointInterface</hardwareInterface>
-        </xacro:if>
-        <xacro:if value="${interface == 'velocity'}">
-          <hardwareInterface>hardware_interface/VelocityJointInterface</hardwareInterface>
-        </xacro:if>
-        <xacro:if value="${interface == 'effort'}">
-          <hardwareInterface>hardware_interface/EffortJointInterface</hardwareInterface>
-        </xacro:if>
-        <mechanicalReduction>1</mechanicalReduction>
-      </actuator>
-    </transmission>
+  <xacro:macro name="material_gazebo_black">
+    <visual>
+      <material>
+        <ambient>0.2 0.2 0.2 1</ambient>
+        <diffuse>0.0 0.0 0.0 1</diffuse>
+      </material>
+    </visual>
   </xacro:macro>
-  <gazebo reference="body_link">
-    <sensor name='camera1' type='camera'>
-      <update_rate>30</update_rate>
-      <camera name='head'>
-        <horizontal_fov>1.39626</horizontal_fov>
-        <image>
-          <width>1280</width>
-          <height>800</height>
-          <format>R8G8B8</format>
-        </image>
-        <clip>
-          <near>0.02</near>
-          <far>300</far>
-        </clip>
-        <noise>
-          <type>gaussian</type>
-          <mean>0</mean>
-          <stddev>0.007</stddev>
-        </noise>
-      </camera>
-      <plugin name='camera_controller' filename='libgazebo_ros_camera.so'>
-        <alwaysOn>true</alwaysOn>
-        <updateRate>0.0</updateRate>
-        <cameraName>sciurus17/chest_camera_node</cameraName>
-        <imageTopicName>image</imageTopicName>
-        <cameraInfoTopicName>camera_info</cameraInfoTopicName>
-        <frameName>chest_camera_link</frameName>
-        <hackBaseline>0.07</hackBaseline>
-        <distortionK1>0.0</distortionK1>
-        <distortionK2>0.0</distortionK2>
-        <distortionK3>0.0</distortionK3>
-        <distortionT1>0.0</distortionT1>
-        <distortionT2>0.0</distortionT2>
-      </plugin>
-      <pose frame=''>0.114576 0 0.217659 0 0.5236 0</pose>
-    </sensor>
-  </gazebo>
-  <gazebo reference="neck_pitch_link">
-    <sensor name='openni_camera_camera' type='depth'>
-      <always_on>1</always_on>
-      <visualize>1</visualize>
-      <camera name='__default__'>
-        <horizontal_fov>1.047</horizontal_fov>
-        <image>
-          <width>640</width>
-          <height>480</height>
-          <format>B8G8R8</format>
-        </image>
-        <depth_camera>
-          <output>depths</output>
-        </depth_camera>
-        <clip>
-          <near>0.1</near>
-          <far>100</far>
-        </clip>
-      </camera>
-      <plugin name='camera_controller' filename='libgazebo_ros_openni_kinect.so'>
-        <robotNamespace>sciurus17</robotNamespace>
-        <alwaysOn>true</alwaysOn>
-        <updateRate>10.0</updateRate>
-        <cameraName>camera</cameraName>
-        <frameName>/camera_color_optical_frame</frameName>
-        <imageTopicName>color/image_raw</imageTopicName>
-        <depthImageTopicName>depth/image_raw</depthImageTopicName>
-        <pointCloudTopicName>depth_registered/points</pointCloudTopicName>
-        <cameraInfoTopicName>color/camera_info</cameraInfoTopicName>
-        <depthImageCameraInfoTopicName>depth/camera_info</depthImageCameraInfoTopicName>
-        <pointCloudCutoff>0.4</pointCloudCutoff>
-        <hackBaseline>0.07</hackBaseline>
-        <distortionK1>0.0</distortionK1>
-        <distortionK2>0.0</distortionK2>
-        <distortionK3>0.0</distortionK3>
-        <distortionT1>0.0</distortionT1>
-        <distortionT2>0.0</distortionT2>
-        <CxPrime>0.0</CxPrime>
-        <Cx>0.0</Cx>
-        <Cy>0.0</Cy>
-        <focalLength>0.0</focalLength>
-      </plugin>
-      <pose frame=''>0.081785 0.03522 0.091 0 -0 0</pose>
-    </sensor>
-  </gazebo>
-  <joint name="camera_color_optical_joint" type="fixed">
-    <origin xyz="0 0.015 0" rpy="-1.5708 0 -1.5708"/>
-    <parent link="camera_link"/>
-    <child link="camera_color_optical_frame"/>
-  </joint>
-  <link name="camera_color_optical_frame"/>
-  <joint name="camera_depth_optical_joint" type="fixed">
-    <origin xyz="0 0.015 0" rpy="-1.5708 0 -1.5708"/>
-    <parent link="camera_link"/>
-    <child link="camera_depth_optical_frame"/>
-  </joint>
-  <link name="camera_depth_optical_frame"/>
-  <gazebo>
-    <plugin name='gazebo_ros_control1' filename='libgazebo_ros_control.so'>
-      <robotNamespace>/sciurus17/controller1</robotNamespace>
-      <robotSimType>gazebo_ros_control/DefaultRobotHWSim</robotSimType>
-      <legacyModeNS>false</legacyModeNS>
-    </plugin>
-    <plugin name='gazebo_ros_control2' filename='libgazebo_ros_control.so'>
-      <robotNamespace>/sciurus17/controller2</robotNamespace>
-      <robotSimType>gazebo_ros_control/DefaultRobotHWSim</robotSimType>
-      <legacyModeNS>false</legacyModeNS>
-    </plugin>
-    <plugin name='gazebo_ros_control3' filename='libgazebo_ros_control.so'>
-      <robotNamespace>/sciurus17/controller3</robotNamespace>
-      <robotSimType>gazebo_ros_control/DefaultRobotHWSim</robotSimType>
-      <legacyModeNS>false</legacyModeNS>
-    </plugin>
-    <plugin name="r_hand_mimic_joint_plugin" filename="libroboticsgroup_upatras_gazebo_mimic_joint_plugin.so">
-      <joint>r_hand_joint</joint>
-      <mimicJoint>r_hand_mimic_joint</mimicJoint>
-      <multiplier>1.0</multiplier>
-    </plugin>
-    <plugin name="l_hand_mimic_joint_plugin" filename="libroboticsgroup_upatras_gazebo_mimic_joint_plugin.so">
-      <joint>l_hand_joint</joint>
-      <mimicJoint>l_hand_mimic_joint</mimicJoint>
-      <multiplier>1.0</multiplier>
-    </plugin>
-  </gazebo>
+  <xacro:macro name="material_gazebo_white">
+    <visual>
+      <material>
+        <ambient>0.95 0.95 0.95 1</ambient>
+        <diffuse>0.95 0.95 0.95 1</diffuse>
+      </material>
+    </visual>
+  </xacro:macro>
+  <xacro:macro name="material_gazebo_red">
+    <visual>
+      <material>
+        <ambient>1.0 0.3 0.3 1</ambient>
+        <diffuse>1.0 0.0 0.0 1</diffuse>
+      </material>
+    </visual>
+  </xacro:macro>
+  <xacro:macro name="gazebo_robot_settings">
+    <gazebo reference="${NAME_LINK_BASE}">
+      <xacro:material_gazebo_white/>
+    </gazebo>
+    <gazebo reference="${NAME_LINK_BODY}">
+      <xacro:material_gazebo_white/>
+    </gazebo>
+    <gazebo reference="${NAME_LINK_CHEST_CAMERA}">
+      <xacro:material_gazebo_black/>
+    </gazebo>
+    <gazebo reference="${NAME_LINK_NECK_1}">
+      <xacro:material_gazebo_white/>
+    </gazebo>
+    <gazebo reference="${NAME_LINK_NECK_2}">
+      <xacro:material_gazebo_white/>
+    </gazebo>
+    <gazebo reference="${NAME_LINK_HEAD_CAMERA}">
+      <xacro:material_gazebo_black/>
+    </gazebo>
+    <gazebo reference="${NAME_LINK_ARM_R_1}">
+      <xacro:material_gazebo_white/>
+    </gazebo>
+    <gazebo reference="${NAME_LINK_ARM_R_2}">
+      <xacro:material_gazebo_white/>
+    </gazebo>
+    <gazebo reference="${NAME_LINK_ARM_R_3}">
+      <xacro:material_gazebo_white/>
+    </gazebo>
+    <gazebo reference="${NAME_LINK_ARM_R_4}">
+      <xacro:material_gazebo_white/>
+    </gazebo>
+    <gazebo reference="${NAME_LINK_ARM_R_5}">
+      <xacro:material_gazebo_white/>
+    </gazebo>
+    <gazebo reference="${NAME_LINK_ARM_R_6}">
+      <xacro:material_gazebo_white/>
+    </gazebo>
+    <gazebo reference="${NAME_LINK_ARM_R_7}">
+      <xacro:material_gazebo_red/>
+    </gazebo>
+    <gazebo reference="${NAME_LINK_HAND_R_A}">
+      <mu1>0.8</mu1>
+      <mu2>0.8</mu2>
+      <xacro:material_gazebo_red/>
+    </gazebo>
+    <gazebo reference="${NAME_LINK_HAND_R_B}">
+      <mu1>0.8</mu1>
+      <mu2>0.8</mu2>
+      <xacro:material_gazebo_red/>
+    </gazebo>
+    <gazebo reference="${NAME_LINK_ARM_L_1}">
+      <xacro:material_gazebo_white/>
+    </gazebo>
+    <gazebo reference="${NAME_LINK_ARM_L_2}">
+      <xacro:material_gazebo_white/>
+    </gazebo>
+    <gazebo reference="${NAME_LINK_ARM_L_3}">
+      <xacro:material_gazebo_white/>
+    </gazebo>
+    <gazebo reference="${NAME_LINK_ARM_L_4}">
+      <xacro:material_gazebo_white/>
+    </gazebo>
+    <gazebo reference="${NAME_LINK_ARM_L_5}">
+      <xacro:material_gazebo_white/>
+    </gazebo>
+    <gazebo reference="${NAME_LINK_ARM_L_6}">
+      <xacro:material_gazebo_white/>
+    </gazebo>
+    <gazebo reference="${NAME_LINK_ARM_L_7}">
+      <xacro:material_gazebo_red/>
+    </gazebo>
+    <gazebo reference="${NAME_LINK_HAND_L_A}">
+      <mu1>0.8</mu1>
+      <mu2>0.8</mu2>
+      <xacro:material_gazebo_red/>
+    </gazebo>
+    <gazebo reference="${NAME_LINK_HAND_L_B}">
+      <mu1>0.8</mu1>
+      <mu2>0.8</mu2>
+      <xacro:material_gazebo_red/>
+    </gazebo>
+  </xacro:macro>
 </robot>
