Commit message: dummy_mimic joint追加

File: urdf/sciurus17_left_hand.xacro (robot description, xacro)
@@ -54,4 +54,12 @@
       </inertial>
     </link>
+    <!--Dummy joint/link to prevent error with mimic joint
+    See https://github.com/ros-controls/gazebo_ros2_control/issues/173
+    -->
+    <joint name="${NAME_JOINT_HAND_L_B}_mimic" type="fixed">
+      <parent link="world" />
+      <child link="dummy_mimic_fix_l" />
+    </joint>
+    <link name="dummy_mimic_fix_l"/>
     <joint name="${NAME_JOINT_HAND_L_B}" type="revolute">
       <parent link="${NAME_LINK_ARM_L_7}" />

File: urdf/sciurus17_right_hand.xacro (robot description, xacro)
@@ -55,4 +55,12 @@
       </inertial>
     </link>
+    <!--Dummy joint/link to prevent error with mimic joint
+    See https://github.com/ros-controls/gazebo_ros2_control/issues/173
+    -->
+    <joint name="${NAME_JOINT_HAND_R_B}_mimic" type="fixed">
+      <parent link="world" />
+      <child link="dummy_mimic_fix_r" />
+    </joint>
+    <link name="dummy_mimic_fix_r"/>
     <joint name="${NAME_JOINT_HAND_R_B}" type="revolute">
       <parent link="${NAME_LINK_ARM_R_7}" />
