Commit message: hand表記をgripperへ変更 (#8)
* hand表記をgripperへ変更

* property名修正

* 設定順序修正

* hand表記をgripperへ変更

File: urdf/sciurus17.gazebo_ros2_control.xacro (robot description, xacro)
@@ -8,6 +8,6 @@
       <joint name="${NAME_JOINT_BODY}">
         <command_interface name="position">
-          <param name="min">${NAME_JOINT_BODY_LOWER_LIMIT}</param>
-          <param name="max">${NAME_JOINT_BODY_UPPER_LIMIT}</param>
+          <param name="min">${JOINT_BODY_LOWER_LIMIT}</param>
+          <param name="max">${JOINT_BODY_UPPER_LIMIT}</param>
         </command_interface>
         <state_interface name="position">
@@ -116,17 +116,17 @@
         <state_interface name="effort"/>
       </joint>
-      <joint name="${NAME_JOINT_HAND_R_A}">
-        <command_interface name="position">
-          <param name="min">${JOINT_HAND_R_LOWER_LIMIT}"</param>
-          <param name="max">${JOINT_HAND_R_UPPER_LIMIT}"</param>
-        </command_interface>
-        <state_interface name="position">
-          <param name="initial_value">0.0</param>
-        </state_interface>
-        <state_interface name="velocity"/>
-        <state_interface name="effort"/>
-      </joint>
-      <joint name="${NAME_JOINT_HAND_R_B}">
-        <param name="mimic">${NAME_JOINT_HAND_R_A}</param>
+      <joint name="${NAME_JOINT_GRIPPER_R_A}">
+        <command_interface name="position">
+          <param name="min">${JOINT_GRIPPER_R_LOWER_LIMIT}"</param>
+          <param name="max">${JOINT_GRIPPER_R_UPPER_LIMIT}"</param>
+        </command_interface>
+        <state_interface name="position">
+          <param name="initial_value">0.0</param>
+        </state_interface>
+        <state_interface name="velocity"/>
+        <state_interface name="effort"/>
+      </joint>
+      <joint name="${NAME_JOINT_GRIPPER_R_B}">
+        <param name="mimic">${NAME_JOINT_GRIPPER_R_A}</param>
         <param name="multiplier">1</param>
         <command_interface name="position"/>
@@ -212,17 +212,17 @@
         <state_interface name="effort"/>
       </joint>
-      <joint name="${NAME_JOINT_HAND_L_A}">
-        <command_interface name="position">
-          <param name="min">${JOINT_HAND_L_LOWER_LIMIT}"</param>
-          <param name="max">${JOINT_HAND_L_UPPER_LIMIT}"</param>
-        </command_interface>
-        <state_interface name="position">
-          <param name="initial_value">0.0</param>
-        </state_interface>
-        <state_interface name="velocity"/>
-        <state_interface name="effort"/>
-      </joint>
-      <joint name="${NAME_JOINT_HAND_L_B}">
-        <param name="mimic">${NAME_JOINT_HAND_L_A}</param>
+      <joint name="${NAME_JOINT_GRIPPER_L_A}">
+        <command_interface name="position">
+          <param name="min">${JOINT_GRIPPER_L_LOWER_LIMIT}"</param>
+          <param name="max">${JOINT_GRIPPER_L_UPPER_LIMIT}"</param>
+        </command_interface>
+        <state_interface name="position">
+          <param name="initial_value">0.0</param>
+        </state_interface>
+        <state_interface name="velocity"/>
+        <state_interface name="effort"/>
+      </joint>
+      <joint name="${NAME_JOINT_GRIPPER_L_B}">
+        <param name="mimic">${NAME_JOINT_GRIPPER_L_A}</param>
         <param name="multiplier">1</param>
         <command_interface name="position"/>

File: urdf/sciurus17.ros2_control.xacro (robot description, xacro)
@@ -12,6 +12,6 @@
       <joint name="${NAME_JOINT_BODY}">
         <command_interface name="position">
-          <param name="min">${NAME_JOINT_BODY_LOWER_LIMIT}</param>
-          <param name="max">${NAME_JOINT_BODY_UPPER_LIMIT}</param>
+          <param name="min">${JOINT_BODY_LOWER_LIMIT}</param>
+          <param name="max">${JOINT_BODY_UPPER_LIMIT}</param>
         </command_interface>
         <state_interface name="position"/>
@@ -110,8 +110,8 @@
         <param name="current_to_effort">2.20</param>
       </joint>
-      <joint name="${NAME_JOINT_HAND_R_A}">
-        <command_interface name="position">
-          <param name="min">${JOINT_HAND_R_LOWER_LIMIT}"</param>
-          <param name="max">${JOINT_HAND_R_UPPER_LIMIT}"</param>
+      <joint name="${NAME_JOINT_GRIPPER_R_A}">
+        <command_interface name="position">
+          <param name="min">${JOINT_GRIPPER_R_LOWER_LIMIT}"</param>
+          <param name="max">${JOINT_GRIPPER_R_UPPER_LIMIT}"</param>
         </command_interface>
         <state_interface name="position"/>
@@ -190,8 +190,8 @@
         <param name="current_to_effort">2.20</param>
       </joint>
-      <joint name="${NAME_JOINT_HAND_L_A}">
-        <command_interface name="position">
-          <param name="min">${JOINT_HAND_L_LOWER_LIMIT}"</param>
-          <param name="max">${JOINT_HAND_L_UPPER_LIMIT}"</param>
+      <joint name="${NAME_JOINT_GRIPPER_L_A}">
+        <command_interface name="position">
+          <param name="min">${JOINT_GRIPPER_L_LOWER_LIMIT}"</param>
+          <param name="max">${JOINT_GRIPPER_L_UPPER_LIMIT}"</param>
         </command_interface>
         <state_interface name="position"/>

File: urdf/sciurus17.urdf.xacro (robot description, xacro)
@@ -10,7 +10,7 @@
   <xacro:include filename="$(find sciurus17_description)/urdf/sciurus17_head.xacro"/>
   <xacro:include filename="$(find sciurus17_description)/urdf/sciurus17_right_arm.xacro"/>
-  <xacro:include filename="$(find sciurus17_description)/urdf/sciurus17_right_hand.xacro"/>
+  <xacro:include filename="$(find sciurus17_description)/urdf/sciurus17_right_gripper.xacro"/>
   <xacro:include filename="$(find sciurus17_description)/urdf/sciurus17_left_arm.xacro"/>
-  <xacro:include filename="$(find sciurus17_description)/urdf/sciurus17_left_hand.xacro"/>
+  <xacro:include filename="$(find sciurus17_description)/urdf/sciurus17_left_gripper.xacro"/>
   <xacro:include filename="$(find sciurus17_description)/urdf/sciurus17_gazebo.xacro"/>
   <xacro:include filename="$(find sciurus17_description)/urdf/sciurus17.gazebo_ros2_control.xacro"/>
@@ -47,6 +47,6 @@
   <xacro:property name="NAME_LINK_ARM_R_6" value="r_link6"/>
   <xacro:property name="NAME_LINK_ARM_R_7" value="r_link7"/>
-  <xacro:property name="NAME_LINK_HAND_R_A" value="r_handA_link"/>
-  <xacro:property name="NAME_LINK_HAND_R_B" value="r_handB_link"/>
+  <xacro:property name="NAME_LINK_GRIPPER_R_A" value="r_gripperA_link"/>
+  <xacro:property name="NAME_LINK_GRIPPER_R_B" value="r_gripperB_link"/>
   <xacro:property name="NAME_LINK_ARMARKER_R" value="r_link5_armarker"/>
   <xacro:property name="NAME_LINK_ARM_L_1" value="l_link1"/>
@@ -57,9 +57,9 @@
   <xacro:property name="NAME_LINK_ARM_L_6" value="l_link6"/>
   <xacro:property name="NAME_LINK_ARM_L_7" value="l_link7"/>
-  <xacro:property name="NAME_LINK_HAND_L_A" value="l_handA_link"/>
-  <xacro:property name="NAME_LINK_HAND_L_B" value="l_handB_link"/>
+  <xacro:property name="NAME_LINK_GRIPPER_L_A" value="l_gripperA_link"/>
+  <xacro:property name="NAME_LINK_GRIPPER_L_B" value="l_gripperB_link"/>
   <xacro:property name="NAME_LINK_ARMARKER_L" value="l_link5_armarker"/>
+  <xacro:property name="NAME_JOINT_BASE" value="base_link_to_world_joint"/>
   <xacro:property name="NAME_JOINT_BODY" value="waist_yaw_joint"/>
-  <xacro:property name="NAME_JOINT_BASE" value="base_link_to_world_joint"/>
   <xacro:property name="NAME_JOINT_NECK_1" value="neck_yaw_joint"/>
   <xacro:property name="NAME_JOINT_NECK_2" value="neck_pitch_joint"/>
@@ -73,6 +73,6 @@
   <xacro:property name="NAME_JOINT_ARM_R_6" value="r_arm_joint6"/>
   <xacro:property name="NAME_JOINT_ARM_R_7" value="r_arm_joint7"/>
-  <xacro:property name="NAME_JOINT_HAND_R_A" value="r_hand_joint"/>
-  <xacro:property name="NAME_JOINT_HAND_R_B" value="r_hand_mimic_joint"/>
+  <xacro:property name="NAME_JOINT_GRIPPER_R_A" value="r_gripper_joint"/>
+  <xacro:property name="NAME_JOINT_GRIPPER_R_B" value="r_gripper_mimic_joint"/>
   <xacro:property name="NAME_JOINT_ARMARKER_R" value="r_arm_armarker"/>
   <xacro:property name="NAME_JOINT_ARM_L_1" value="l_arm_joint1"/>
@@ -83,11 +83,11 @@
   <xacro:property name="NAME_JOINT_ARM_L_6" value="l_arm_joint6"/>
   <xacro:property name="NAME_JOINT_ARM_L_7" value="l_arm_joint7"/>
-  <xacro:property name="NAME_JOINT_HAND_L_A" value="l_hand_joint"/>
-  <xacro:property name="NAME_JOINT_HAND_L_B" value="l_hand_mimic_joint"/>
+  <xacro:property name="NAME_JOINT_GRIPPER_L_A" value="l_gripper_joint"/>
+  <xacro:property name="NAME_JOINT_GRIPPER_L_B" value="l_gripper_mimic_joint"/>
   <xacro:property name="NAME_JOINT_ARMARKER_L" value="l_arm_armarker"/>
   <xacro:property name="EFFORT_LIMIT" value="4.0"/>
   <xacro:property name="VELOCITY_LIMIT" value="5.969211435"/>
-  <xacro:property name="NAME_JOINT_BODY_LOWER_LIMIT" value="${radians(-110)}"/>
-  <xacro:property name="NAME_JOINT_BODY_UPPER_LIMIT" value="${radians(110)}"/>
+  <xacro:property name="JOINT_BODY_LOWER_LIMIT" value="${radians(-110)}"/>
+  <xacro:property name="JOINT_BODY_UPPER_LIMIT" value="${radians(110)}"/>
   <xacro:property name="JOINT_NECK_1_LOWER_LIMIT" value="${radians(-165)}"/>
   <xacro:property name="JOINT_NECK_1_UPPER_LIMIT" value="${radians(165)}"/>
@@ -112,6 +112,6 @@
   <!-- Gazeboの挙動がlimit付近で不安定なため、limitをサーボの可動範囲より少し大きくする -->
   <!-- 参照: https://github.com/rt-net/sciurus17_description/pull/6 -->
-  <xacro:property name="JOINT_HAND_R_LOWER_LIMIT" value="${radians(-0.01)}"/>
-  <xacro:property name="JOINT_HAND_R_UPPER_LIMIT" value="${radians(86)}"/>
+  <xacro:property name="JOINT_GRIPPER_R_LOWER_LIMIT" value="${radians(-0.01)}"/>
+  <xacro:property name="JOINT_GRIPPER_R_UPPER_LIMIT" value="${radians(86)}"/>
   <xacro:property name="JOINT_ARM_L_1_LOWER_LIMIT" value="${radians(-90)}"/>
   <xacro:property name="JOINT_ARM_L_1_UPPER_LIMIT" value="${radians(90)}"/>
@@ -130,13 +130,13 @@
   <xacro:property name="JOINT_ARM_L_7_LOWER_LIMIT" value="${radians(-170)}"/>
   <xacro:property name="JOINT_ARM_L_7_UPPER_LIMIT" value="${radians(170)}"/>
-  <xacro:property name="JOINT_HAND_L_LOWER_LIMIT" value="${radians(-86)}"/>
+  <xacro:property name="JOINT_GRIPPER_L_LOWER_LIMIT" value="${radians(-86)}"/>
   <!-- Gazeboの挙動がlimit付近で不安定なため、limitをサーボの可動範囲より少し大きくする -->
   <!-- 参照: https://github.com/rt-net/sciurus17_description/pull/6 -->
-  <xacro:property name="JOINT_HAND_L_UPPER_LIMIT" value="${radians(0.01)}"/>
+  <xacro:property name="JOINT_GRIPPER_L_UPPER_LIMIT" value="${radians(0.01)}"/>
   <xacro:property name="COLOR_LINK_BASE" value="white"/>
   <xacro:property name="COLOR_LINK_BODY" value="white"/>
   <xacro:property name="COLOR_LINK_HEAD" value="white"/>
   <xacro:property name="COLOR_LINK_ARM" value="white"/>
-  <xacro:property name="COLOR_LINK_HAND" value="red"/>
+  <xacro:property name="COLOR_LINK_GRIPPER" value="red"/>
   <xacro:property name="COLOR_LINK_CAMERA" value="white"/>
   <!-- Used for fixing robot 'base_link'  to Gazebo 'world' -->
@@ -149,7 +149,7 @@
   <xacro:sciurus17_head/>
   <xacro:sciurus17_right_arm/>
-  <xacro:sciurus17_right_hand/>
+  <xacro:sciurus17_right_gripper/>
   <xacro:sciurus17_left_arm/>
-  <xacro:sciurus17_left_hand/>
+  <xacro:sciurus17_left_gripper/>
   <xacro:unless value="$(arg use_gazebo)">
     <xacro:sciurus17_ros2_control_settings/>

File: urdf/sciurus17_left_gripper.xacro (robot description, xacro)
@@ -1,5 +1,5 @@
 <?xml version="1.0"?>
 <robot xmlns:xacro="http://ros.org/wiki/xacro">
-  <xacro:macro name="sciurus17_left_hand">
+  <xacro:macro name="sciurus17_left_gripper">
     <link name="${NAME_LINK_ARM_L_7}">
       <visual>
@@ -8,5 +8,5 @@
           <mesh filename="package://sciurus17_description/meshes/visual/L_Link7.stl" scale="1.0 1.0 1.0"/>
         </geometry>
-        <material name="${COLOR_LINK_HAND}"/>
+        <material name="${COLOR_LINK_GRIPPER}"/>
       </visual>
       <collision>
@@ -22,11 +22,11 @@
       </inertial>
     </link>
-    <joint name="${NAME_JOINT_HAND_L_A}" type="revolute">
+    <joint name="${NAME_JOINT_GRIPPER_L_A}" type="revolute">
       <parent link="${NAME_LINK_ARM_L_7}" />
-      <child link="${NAME_LINK_HAND_L_A}" />
+      <child link="${NAME_LINK_GRIPPER_L_A}" />
       <origin xyz="0.012 0.024 0.0" rpy="0 0 0"/>
       <limit
-        lower="${JOINT_HAND_L_LOWER_LIMIT}"
-        upper="${JOINT_HAND_L_UPPER_LIMIT}"
+        lower="${JOINT_GRIPPER_L_LOWER_LIMIT}"
+        upper="${JOINT_GRIPPER_L_UPPER_LIMIT}"
         effort="${EFFORT_LIMIT}"
         velocity="${VELOCITY_LIMIT}"/>
@@ -34,16 +34,16 @@
       <dynamics damping="1.0e-6" friction="0.8"/>
     </joint>
-    <link name="${NAME_LINK_HAND_L_A}">
+    <link name="${NAME_LINK_GRIPPER_L_A}">
       <visual>
         <origin rpy="0 0 0" xyz="0.0 0.0 0.0"/>
         <geometry>
-          <mesh filename="package://sciurus17_description/meshes/visual/L_HandA.stl" scale="1.0 1.0 1.0"/>
+          <mesh filename="package://sciurus17_description/meshes/visual/L_GripperA.stl" scale="1.0 1.0 1.0"/>
         </geometry>
-        <material name="${COLOR_LINK_HAND}"/>
+        <material name="${COLOR_LINK_GRIPPER}"/>
       </visual>
       <collision>
         <origin rpy="0 0 0" xyz="0.0 0.0 0.0"/>
         <geometry>
-          <mesh filename="package://sciurus17_description/meshes/collision/L_HandA.stl" scale="1.0 1.0 1.0"/>
+          <mesh filename="package://sciurus17_description/meshes/collision/L_GripperA.stl" scale="1.0 1.0 1.0"/>
         </geometry>
       </collision>
@@ -57,34 +57,34 @@
     See https://github.com/ros-controls/gazebo_ros2_control/issues/173
     -->
-    <joint name="${NAME_JOINT_HAND_L_B}_mimic" type="fixed">
+    <joint name="${NAME_JOINT_GRIPPER_L_B}_mimic" type="fixed">
       <parent link="world" />
       <child link="dummy_mimic_fix_l" />
     </joint>
     <link name="dummy_mimic_fix_l"/>
-    <joint name="${NAME_JOINT_HAND_L_B}" type="revolute">
+    <joint name="${NAME_JOINT_GRIPPER_L_B}" type="revolute">
       <parent link="${NAME_LINK_ARM_L_7}" />
-      <child link="${NAME_LINK_HAND_L_B}" />
+      <child link="${NAME_LINK_GRIPPER_L_B}" />
       <origin xyz="-0.012 0.024 0.0" rpy="0 0 0"/>
       <limit
-        lower="${JOINT_HAND_L_LOWER_LIMIT}"
-        upper="${JOINT_HAND_L_UPPER_LIMIT}"
+        lower="${JOINT_GRIPPER_L_LOWER_LIMIT}"
+        upper="${JOINT_GRIPPER_L_UPPER_LIMIT}"
         effort="${EFFORT_LIMIT}"
         velocity="${VELOCITY_LIMIT}"/>
       <axis xyz="0 0 -1"/>
-      <mimic joint="${NAME_JOINT_HAND_L_A}" multiplier="1" offset="0"/>
+      <mimic joint="${NAME_JOINT_GRIPPER_L_A}" multiplier="1" offset="0"/>
       <dynamics damping="1.0e-6" friction="0.8"/>
     </joint>
-    <link name="${NAME_LINK_HAND_L_B}">
+    <link name="${NAME_LINK_GRIPPER_L_B}">
       <visual>
         <origin rpy="0 0 0" xyz="0.0 0.0 0.0"/>
         <geometry>
-          <mesh filename="package://sciurus17_description/meshes/visual/L_HandB.stl" scale="1.0 1.0 1.0"/>
+          <mesh filename="package://sciurus17_description/meshes/visual/L_GripperB.stl" scale="1.0 1.0 1.0"/>
         </geometry>
-        <material name="${COLOR_LINK_HAND}"/>
+        <material name="${COLOR_LINK_GRIPPER}"/>
       </visual>
       <collision>
         <origin rpy="0 0 0" xyz="0.0 0.0 0.0"/>
         <geometry>
-          <mesh filename="package://sciurus17_description/meshes/collision/L_HandB.stl" scale="1.0 1.0 1.0"/>
+          <mesh filename="package://sciurus17_description/meshes/collision/L_GripperB.stl" scale="1.0 1.0 1.0"/>
         </geometry>
       </collision>

File: urdf/sciurus17_right_gripper.xacro (robot description, xacro)
@@ -1,5 +1,5 @@
 <?xml version="1.0"?>
 <robot xmlns:xacro="http://ros.org/wiki/xacro">
-  <xacro:macro name="sciurus17_right_hand">
+  <xacro:macro name="sciurus17_right_gripper">
     <link name="${NAME_LINK_ARM_R_7}">
       <visual>
@@ -8,5 +8,5 @@
           <mesh filename="package://sciurus17_description/meshes/visual/R_Link7.stl" scale="1.0 1.0 1.0"/>
         </geometry>
-        <material name="${COLOR_LINK_HAND}"/>
+        <material name="${COLOR_LINK_GRIPPER}"/>
       </visual>
       <collision>
@@ -22,11 +22,11 @@
       </inertial>
     </link>
-    <joint name="${NAME_JOINT_HAND_R_A}" type="revolute">
+    <joint name="${NAME_JOINT_GRIPPER_R_A}" type="revolute">
       <parent link="${NAME_LINK_ARM_R_7}" />
-      <child link="${NAME_LINK_HAND_R_A}" />
+      <child link="${NAME_LINK_GRIPPER_R_A}" />
       <origin xyz="0.012 -0.024 0.0" rpy="0 0 0"/>
       <limit
-        lower="${JOINT_HAND_R_LOWER_LIMIT}"
-        upper="${JOINT_HAND_R_UPPER_LIMIT}"
+        lower="${JOINT_GRIPPER_R_LOWER_LIMIT}"
+        upper="${JOINT_GRIPPER_R_UPPER_LIMIT}"
         effort="${EFFORT_LIMIT}"
         velocity="${VELOCITY_LIMIT}"/>
@@ -34,17 +34,17 @@
       <dynamics damping="1.0e-6" friction="0.8"/>
     </joint>
-    <link name="${NAME_LINK_HAND_R_A}">
+    <link name="${NAME_LINK_GRIPPER_R_A}">
       <visual>
         <!--origin rpy="3.14159 0 0" xyz="0.0 0.0 0.0"/-->
         <origin rpy="0 0 0" xyz="0.0 0.0 0.0"/>
         <geometry>
-          <mesh filename="package://sciurus17_description/meshes/visual/R_HandA.stl" scale="1.0 1.0 1.0"/>
+          <mesh filename="package://sciurus17_description/meshes/visual/R_GripperA.stl" scale="1.0 1.0 1.0"/>
         </geometry>
-        <material name="${COLOR_LINK_HAND}"/>
+        <material name="${COLOR_LINK_GRIPPER}"/>
       </visual>
       <collision>
         <origin rpy="0 0 0" xyz="0.0 0.0 0.0"/>
         <geometry>
-          <mesh filename="package://sciurus17_description/meshes/collision/R_HandA.stl" scale="1.0 1.0 1.0"/>
+          <mesh filename="package://sciurus17_description/meshes/collision/R_GripperA.stl" scale="1.0 1.0 1.0"/>
         </geometry>
       </collision>
@@ -58,35 +58,35 @@
     See https://github.com/ros-controls/gazebo_ros2_control/issues/173
     -->
-    <joint name="${NAME_JOINT_HAND_R_B}_mimic" type="fixed">
+    <joint name="${NAME_JOINT_GRIPPER_R_B}_mimic" type="fixed">
       <parent link="world" />
       <child link="dummy_mimic_fix_r" />
     </joint>
     <link name="dummy_mimic_fix_r"/>
-    <joint name="${NAME_JOINT_HAND_R_B}" type="revolute">
+    <joint name="${NAME_JOINT_GRIPPER_R_B}" type="revolute">
       <parent link="${NAME_LINK_ARM_R_7}" />
-      <child link="${NAME_LINK_HAND_R_B}" />
+      <child link="${NAME_LINK_GRIPPER_R_B}" />
       <origin xyz="-0.012 -0.024 0.0" rpy="0 0 0"/>
       <limit
-        lower="${JOINT_HAND_R_LOWER_LIMIT}"
-        upper="${JOINT_HAND_R_UPPER_LIMIT}"
+        lower="${JOINT_GRIPPER_R_LOWER_LIMIT}"
+        upper="${JOINT_GRIPPER_R_UPPER_LIMIT}"
         effort="${EFFORT_LIMIT}"
         velocity="${VELOCITY_LIMIT}"/>
       <axis xyz="0 0 -1"/>
-      <mimic joint="${NAME_JOINT_HAND_R_A}" multiplier="1" offset="0"/>
+      <mimic joint="${NAME_JOINT_GRIPPER_R_A}" multiplier="1" offset="0"/>
       <dynamics damping="1.0e-6" friction="0.8"/>
     </joint>
-    <link name="${NAME_LINK_HAND_R_B}">
+    <link name="${NAME_LINK_GRIPPER_R_B}">
       <visual>
         <!-- origin rpy="3.14159 0 0" xyz="0.0 0.0 0.0"/ -->
         <origin rpy="0 0 0" xyz="0.0 0.0 0.0"/>
         <geometry>
-          <mesh filename="package://sciurus17_description/meshes/visual/R_HandB.stl" scale="1.0 1.0 1.0"/>
+          <mesh filename="package://sciurus17_description/meshes/visual/R_GripperB.stl" scale="1.0 1.0 1.0"/>
         </geometry>
-        <material name="${COLOR_LINK_HAND}"/>
+        <material name="${COLOR_LINK_GRIPPER}"/>
       </visual>
       <collision>
         <origin rpy="0 0 0" xyz="0.0 0.0 0.0"/>
         <geometry>
-          <mesh filename="package://sciurus17_description/meshes/collision/R_HandB.stl" scale="1.0 1.0 1.0"/>
+          <mesh filename="package://sciurus17_description/meshes/collision/R_GripperB.stl" scale="1.0 1.0 1.0"/>
         </geometry>
       </collision>
