Commit message: リンク名とジョイント名のproperty定義を廃止

File: urdf/sciurus17.gazebo_ros2_control.xacro (robot description, xacro)
@@ -6,5 +6,5 @@
         <plugin>gz_ros2_control/GazeboSimSystem</plugin>
       </hardware>
-      <joint name="${NAME_JOINT_BODY}">
+      <joint name="waist_yaw_joint">
         <command_interface name="position">
           <param name="min">${JOINT_BODY_LOWER_LIMIT}</param>
@@ -17,5 +17,5 @@
         <state_interface name="effort"/>
       </joint>
-      <joint name="${NAME_JOINT_NECK_1}">
+      <joint name="neck_yaw_joint">
         <command_interface name="position">
           <param name="min">${JOINT_NECK_1_LOWER_LIMIT}</param>
@@ -28,5 +28,5 @@
         <state_interface name="effort"/>
       </joint>
-      <joint name="${NAME_JOINT_NECK_2}">
+      <joint name="neck_pitch_joint">
         <command_interface name="position">
           <param name="min">${JOINT_NECK_2_LOWER_LIMIT}</param>
@@ -39,5 +39,5 @@
         <state_interface name="effort"/>
       </joint>
-      <joint name="${NAME_JOINT_ARM_R_1}">
+      <joint name="r_arm_joint1">
         <command_interface name="position">
           <param name="min">${JOINT_ARM_R_1_LOWER_LIMIT}</param>
@@ -50,5 +50,5 @@
         <state_interface name="effort"/>
       </joint>
-      <joint name="${NAME_JOINT_ARM_R_2}">
+      <joint name="r_arm_joint2">
         <command_interface name="position">
           <param name="min">${JOINT_ARM_R_2_LOWER_LIMIT}</param>
@@ -61,5 +61,5 @@
         <state_interface name="effort"/>
       </joint>
-      <joint name="${NAME_JOINT_ARM_R_3}">
+      <joint name="r_arm_joint3">
         <command_interface name="position">
           <param name="min">${JOINT_ARM_R_3_LOWER_LIMIT}</param>
@@ -72,5 +72,5 @@
         <state_interface name="effort"/>
       </joint>
-      <joint name="${NAME_JOINT_ARM_R_4}">
+      <joint name="r_arm_joint4">
         <command_interface name="position">
           <param name="min">${JOINT_ARM_R_4_LOWER_LIMIT}</param>
@@ -83,5 +83,5 @@
         <state_interface name="effort"/>
       </joint>
-      <joint name="${NAME_JOINT_ARM_R_5}">
+      <joint name="r_arm_joint5">
         <command_interface name="position">
           <param name="min">${JOINT_ARM_R_5_LOWER_LIMIT}</param>
@@ -94,5 +94,5 @@
         <state_interface name="effort"/>
       </joint>
-      <joint name="${NAME_JOINT_ARM_R_6}">
+      <joint name="r_arm_joint6">
         <command_interface name="position">
           <param name="min">${JOINT_ARM_R_6_LOWER_LIMIT}</param>
@@ -105,5 +105,5 @@
         <state_interface name="effort"/>
       </joint>
-      <joint name="${NAME_JOINT_ARM_R_7}">
+      <joint name="r_arm_joint7">
         <command_interface name="position">
           <param name="min">${JOINT_ARM_R_7_LOWER_LIMIT}</param>
@@ -116,5 +116,5 @@
         <state_interface name="effort"/>
       </joint>
-      <joint name="${NAME_JOINT_GRIPPER_R_A}">
+      <joint name="r_gripper_joint">
         <command_interface name="position">
           <param name="min">${JOINT_GRIPPER_R_LOWER_LIMIT}</param>
@@ -127,6 +127,6 @@
         <state_interface name="effort"/>
       </joint>
-      <joint name="${NAME_JOINT_GRIPPER_R_B}">
-        <param name="mimic">${NAME_JOINT_GRIPPER_R_A}</param>
+      <joint name="r_gripper_mimic_joint">
+        <param name="mimic">r_gripper_joint</param>
         <param name="multiplier">1</param>
         <state_interface name="position"/>
@@ -134,5 +134,5 @@
         <state_interface name="effort"/>
       </joint>
-      <joint name="${NAME_JOINT_ARM_L_1}">
+      <joint name="l_arm_joint1">
         <command_interface name="position">
           <param name="min">${JOINT_ARM_L_1_LOWER_LIMIT}</param>
@@ -145,5 +145,5 @@
         <state_interface name="effort"/>
       </joint>
-      <joint name="${NAME_JOINT_ARM_L_2}">
+      <joint name="l_arm_joint2">
         <command_interface name="position">
           <param name="min">${JOINT_ARM_L_2_LOWER_LIMIT}</param>
@@ -156,5 +156,5 @@
         <state_interface name="effort"/>
       </joint>
-      <joint name="${NAME_JOINT_ARM_L_3}">
+      <joint name="l_arm_joint3">
         <command_interface name="position">
           <param name="min">${JOINT_ARM_L_3_LOWER_LIMIT}</param>
@@ -167,5 +167,5 @@
         <state_interface name="effort"/>
       </joint>
-      <joint name="${NAME_JOINT_ARM_L_4}">
+      <joint name="l_arm_joint4">
         <command_interface name="position">
           <param name="min">${JOINT_ARM_L_4_LOWER_LIMIT}</param>
@@ -178,5 +178,5 @@
         <state_interface name="effort"/>
       </joint>
-      <joint name="${NAME_JOINT_ARM_L_5}">
+      <joint name="l_arm_joint5">
         <command_interface name="position">
           <param name="min">${JOINT_ARM_L_5_LOWER_LIMIT}</param>
@@ -189,5 +189,5 @@
         <state_interface name="effort"/>
       </joint>
-      <joint name="${NAME_JOINT_ARM_L_6}">
+      <joint name="l_arm_joint6">
         <command_interface name="position">
           <param name="min">${JOINT_ARM_L_6_LOWER_LIMIT}</param>
@@ -200,5 +200,5 @@
         <state_interface name="effort"/>
       </joint>
-      <joint name="${NAME_JOINT_ARM_L_7}">
+      <joint name="l_arm_joint7">
         <command_interface name="position">
           <param name="min">${JOINT_ARM_L_7_LOWER_LIMIT}</param>
@@ -211,5 +211,5 @@
         <state_interface name="effort"/>
       </joint>
-      <joint name="${NAME_JOINT_GRIPPER_L_A}">
+      <joint name="l_gripper_joint">
         <command_interface name="position">
           <param name="min">${JOINT_GRIPPER_L_LOWER_LIMIT}</param>
@@ -222,6 +222,6 @@
         <state_interface name="effort"/>
       </joint>
-      <joint name="${NAME_JOINT_GRIPPER_L_B}">
-        <param name="mimic">${NAME_JOINT_GRIPPER_L_A}</param>
+      <joint name="l_gripper_mimic_joint">
+        <param name="mimic">l_gripper_joint</param>
         <param name="multiplier">1</param>
         <state_interface name="position"/>

File: urdf/sciurus17.ros2_control.xacro (robot description, xacro)
@@ -15,5 +15,5 @@
         </xacro:unless>
       </hardware>
-      <joint name="${NAME_JOINT_BODY}">
+      <joint name="waist_yaw_joint">
         <command_interface name="position">
           <param name="min">${JOINT_BODY_LOWER_LIMIT}</param>
@@ -25,5 +25,5 @@
         <param name="current_to_effort">3.60</param>
       </joint>
-      <joint name="${NAME_JOINT_NECK_1}">
+      <joint name="neck_yaw_joint">
         <command_interface name="position">
           <param name="min">${JOINT_NECK_1_LOWER_LIMIT}</param>
@@ -35,5 +35,5 @@
         <param name="current_to_effort">2.20</param>
       </joint>
-      <joint name="${NAME_JOINT_NECK_2}">
+      <joint name="neck_pitch_joint">
         <command_interface name="position">
           <param name="min">${JOINT_NECK_2_LOWER_LIMIT}</param>
@@ -45,5 +45,5 @@
         <param name="current_to_effort">2.20</param>
       </joint>
-      <joint name="${NAME_JOINT_ARM_R_1}">
+      <joint name="r_arm_joint1">
         <command_interface name="position">
           <param name="min">${JOINT_ARM_R_1_LOWER_LIMIT}</param>
@@ -55,5 +55,5 @@
         <param name="current_to_effort">3.60</param>
       </joint>
-      <joint name="${NAME_JOINT_ARM_R_2}">
+      <joint name="r_arm_joint2">
         <command_interface name="position">
           <param name="min">${JOINT_ARM_R_2_LOWER_LIMIT}</param>
@@ -65,5 +65,5 @@
         <param name="current_to_effort">3.60</param>
       </joint>
-      <joint name="${NAME_JOINT_ARM_R_3}">
+      <joint name="r_arm_joint3">
         <command_interface name="position">
           <param name="min">${JOINT_ARM_R_3_LOWER_LIMIT}</param>
@@ -75,5 +75,5 @@
         <param name="current_to_effort">2.20</param>
       </joint>
-      <joint name="${NAME_JOINT_ARM_R_4}">
+      <joint name="r_arm_joint4">
         <command_interface name="position">
           <param name="min">${JOINT_ARM_R_4_LOWER_LIMIT}</param>
@@ -85,5 +85,5 @@
         <param name="current_to_effort">2.00</param>
       </joint>
-      <joint name="${NAME_JOINT_ARM_R_5}">
+      <joint name="r_arm_joint5">
         <command_interface name="position">
           <param name="min">${JOINT_ARM_R_5_LOWER_LIMIT}</param>
@@ -95,5 +95,5 @@
         <param name="current_to_effort">2.20</param>
       </joint>
-      <joint name="${NAME_JOINT_ARM_R_6}">
+      <joint name="r_arm_joint6">
         <command_interface name="position">
           <param name="min">${JOINT_ARM_R_6_LOWER_LIMIT}</param>
@@ -105,5 +105,5 @@
         <param name="current_to_effort">2.20</param>
       </joint>
-      <joint name="${NAME_JOINT_ARM_R_7}">
+      <joint name="r_arm_joint7">
         <command_interface name="position">
           <param name="min">${JOINT_ARM_R_7_LOWER_LIMIT}</param>
@@ -115,5 +115,5 @@
         <param name="current_to_effort">2.20</param>
       </joint>
-      <joint name="${NAME_JOINT_GRIPPER_R_A}">
+      <joint name="r_gripper_joint">
         <command_interface name="position">
           <param name="min">${JOINT_GRIPPER_R_LOWER_LIMIT}</param>
@@ -125,5 +125,5 @@
         <param name="current_to_effort">2.20</param>
       </joint>
-      <joint name="${NAME_JOINT_ARM_L_1}">
+      <joint name="l_arm_joint1">
         <command_interface name="position">
           <param name="min">${JOINT_ARM_L_1_LOWER_LIMIT}</param>
@@ -135,5 +135,5 @@
         <param name="current_to_effort">3.60</param>
       </joint>
-      <joint name="${NAME_JOINT_ARM_L_2}">
+      <joint name="l_arm_joint2">
         <command_interface name="position">
           <param name="min">${JOINT_ARM_L_2_LOWER_LIMIT}</param>
@@ -145,5 +145,5 @@
         <param name="current_to_effort">3.60</param>
       </joint>
-      <joint name="${NAME_JOINT_ARM_L_3}">
+      <joint name="l_arm_joint3">
         <command_interface name="position">
           <param name="min">${JOINT_ARM_L_3_LOWER_LIMIT}</param>
@@ -155,5 +155,5 @@
         <param name="current_to_effort">2.20</param>
       </joint>
-      <joint name="${NAME_JOINT_ARM_L_4}">
+      <joint name="l_arm_joint4">
         <command_interface name="position">
           <param name="min">${JOINT_ARM_L_4_LOWER_LIMIT}</param>
@@ -165,5 +165,5 @@
         <param name="current_to_effort">2.00</param>
       </joint>
-      <joint name="${NAME_JOINT_ARM_L_5}">
+      <joint name="l_arm_joint5">
         <command_interface name="position">
           <param name="min">${JOINT_ARM_L_5_LOWER_LIMIT}</param>
@@ -175,5 +175,5 @@
         <param name="current_to_effort">2.20</param>
       </joint>
-      <joint name="${NAME_JOINT_ARM_L_6}">
+      <joint name="l_arm_joint6">
         <command_interface name="position">
           <param name="min">${JOINT_ARM_L_6_LOWER_LIMIT}</param>
@@ -185,5 +185,5 @@
         <param name="current_to_effort">2.20</param>
       </joint>
-      <joint name="${NAME_JOINT_ARM_L_7}">
+      <joint name="l_arm_joint7">
         <command_interface name="position">
           <param name="min">${JOINT_ARM_L_7_LOWER_LIMIT}</param>
@@ -195,5 +195,5 @@
         <param name="current_to_effort">2.20</param>
       </joint>
-      <joint name="${NAME_JOINT_GRIPPER_L_A}">
+      <joint name="l_gripper_joint">
         <command_interface name="position">
           <param name="min">${JOINT_GRIPPER_L_LOWER_LIMIT}</param>

File: urdf/sciurus17.urdf.xacro (robot description, xacro)
@@ -42,56 +42,4 @@
     <color rgba="0.8984375 0.0 0.0703125 1"/>
   </material>
-  <xacro:property name="NAME_LINK_BASE" value="base_link"/>
-  <xacro:property name="NAME_LINK_BODY" value="body_link"/>
-  <xacro:property name="NAME_LINK_NECK_1" value="neck_yaw_link"/>
-  <xacro:property name="NAME_LINK_NECK_2" value="neck_pitch_link"/>
-  <xacro:property name="NAME_LINK_HEAD_CAMERA" value="${NAME_HEAD_CAMERA_PREFIX}_link"/>
-  <xacro:property name="NAME_LINK_CHEST_CAMERA" value="${NAME_CHEST_CAMERA_PREFIX}_link"/>
-  <xacro:property name="NAME_LINK_ARM_R_1" value="r_link1"/>
-  <xacro:property name="NAME_LINK_ARM_R_2" value="r_link2"/>
-  <xacro:property name="NAME_LINK_ARM_R_3" value="r_link3"/>
-  <xacro:property name="NAME_LINK_ARM_R_4" value="r_link4"/>
-  <xacro:property name="NAME_LINK_ARM_R_5" value="r_link5"/>
-  <xacro:property name="NAME_LINK_ARM_R_6" value="r_link6"/>
-  <xacro:property name="NAME_LINK_ARM_R_7" value="r_link7"/>
-  <xacro:property name="NAME_LINK_GRIPPER_R_A" value="r_gripperA_link"/>
-  <xacro:property name="NAME_LINK_GRIPPER_R_B" value="r_gripperB_link"/>
-  <xacro:property name="NAME_LINK_ARMARKER_R" value="r_link5_armarker"/>
-  <xacro:property name="NAME_LINK_ARM_L_1" value="l_link1"/>
-  <xacro:property name="NAME_LINK_ARM_L_2" value="l_link2"/>
-  <xacro:property name="NAME_LINK_ARM_L_3" value="l_link3"/>
-  <xacro:property name="NAME_LINK_ARM_L_4" value="l_link4"/>
-  <xacro:property name="NAME_LINK_ARM_L_5" value="l_link5"/>
-  <xacro:property name="NAME_LINK_ARM_L_6" value="l_link6"/>
-  <xacro:property name="NAME_LINK_ARM_L_7" value="l_link7"/>
-  <xacro:property name="NAME_LINK_GRIPPER_L_A" value="l_gripperA_link"/>
-  <xacro:property name="NAME_LINK_GRIPPER_L_B" value="l_gripperB_link"/>
-  <xacro:property name="NAME_LINK_ARMARKER_L" value="l_link5_armarker"/>
-  <xacro:property name="NAME_JOINT_BASE" value="base_link_to_world_joint"/>
-  <xacro:property name="NAME_JOINT_BODY" value="waist_yaw_joint"/>
-  <xacro:property name="NAME_JOINT_NECK_1" value="neck_yaw_joint"/>
-  <xacro:property name="NAME_JOINT_NECK_2" value="neck_pitch_joint"/>
-  <xacro:property name="NAME_JOINT_HEAD_CAMERA" value="head_camera_joint"/>
-  <xacro:property name="NAME_JOINT_CHEST_CAMERA" value="chest_camera_joint"/>
-  <xacro:property name="NAME_JOINT_ARM_R_1" value="r_arm_joint1"/>
-  <xacro:property name="NAME_JOINT_ARM_R_2" value="r_arm_joint2"/>
-  <xacro:property name="NAME_JOINT_ARM_R_3" value="r_arm_joint3"/>
-  <xacro:property name="NAME_JOINT_ARM_R_4" value="r_arm_joint4"/>
-  <xacro:property name="NAME_JOINT_ARM_R_5" value="r_arm_joint5"/>
-  <xacro:property name="NAME_JOINT_ARM_R_6" value="r_arm_joint6"/>
-  <xacro:property name="NAME_JOINT_ARM_R_7" value="r_arm_joint7"/>
-  <xacro:property name="NAME_JOINT_GRIPPER_R_A" value="r_gripper_joint"/>
-  <xacro:property name="NAME_JOINT_GRIPPER_R_B" value="r_gripper_mimic_joint"/>
-  <xacro:property name="NAME_JOINT_ARMARKER_R" value="r_arm_armarker"/>
-  <xacro:property name="NAME_JOINT_ARM_L_1" value="l_arm_joint1"/>
-  <xacro:property name="NAME_JOINT_ARM_L_2" value="l_arm_joint2"/>
-  <xacro:property name="NAME_JOINT_ARM_L_3" value="l_arm_joint3"/>
-  <xacro:property name="NAME_JOINT_ARM_L_4" value="l_arm_joint4"/>
-  <xacro:property name="NAME_JOINT_ARM_L_5" value="l_arm_joint5"/>
-  <xacro:property name="NAME_JOINT_ARM_L_6" value="l_arm_joint6"/>
-  <xacro:property name="NAME_JOINT_ARM_L_7" value="l_arm_joint7"/>
-  <xacro:property name="NAME_JOINT_GRIPPER_L_A" value="l_gripper_joint"/>
-  <xacro:property name="NAME_JOINT_GRIPPER_L_B" value="l_gripper_mimic_joint"/>
-  <xacro:property name="NAME_JOINT_ARMARKER_L" value="l_arm_armarker"/>
   <xacro:property name="EFFORT_LIMIT" value="4.0"/>
   <xacro:property name="VELOCITY_LIMIT" value="5.969211435"/>
@@ -153,7 +101,7 @@
   <!-- Used for fixing robot 'base_link'  to Gazebo 'world' -->
   <link name="world"/>
-  <joint name="${NAME_JOINT_BASE}" type="fixed">
+  <joint name="base_link_to_world_joint" type="fixed">
     <parent link="world"/>
-    <child link="${NAME_LINK_BASE}"/>
+    <child link="base_link"/>
   </joint>
   <xacro:sciurus17_body/>
@@ -171,5 +119,5 @@
     <joint name="${NAME_HEAD_CAMERA_PREFIX}_color_joint" type="fixed">
       <origin xyz="0 0.015 0" rpy="0 0 0" />
-      <parent link="${NAME_LINK_HEAD_CAMERA}" />
+      <parent link="head_camera_link" />
       <child link="${NAME_HEAD_CAMERA_PREFIX}_color_frame" />
     </joint>

File: urdf/sciurus17_body.xacro (robot description, xacro)
@@ -2,5 +2,5 @@
 <robot xmlns:xacro="http://ros.org/wiki/xacro">
   <xacro:macro name="sciurus17_body">
-    <link name="${NAME_LINK_BASE}">
+    <link name="base_link">
       <visual>
         <geometry>
@@ -21,7 +21,7 @@
       </inertial>
     </link>
-    <joint name="${NAME_JOINT_BODY}" type="revolute">
-      <parent link="${NAME_LINK_BASE}" />
-      <child link="${NAME_LINK_BODY}" />
+    <joint name="waist_yaw_joint" type="revolute">
+      <parent link="base_link" />
+      <child link="body_link" />
       <origin xyz="0.0 0.0 0.1315" rpy="0 0 0"/>
       <limit
@@ -33,5 +33,5 @@
       <dynamics damping="1.0e-6" friction="0.8"/>
     </joint>
-    <link name="${NAME_LINK_BODY}">
+    <link name="body_link">
       <visual>
         <geometry>
@@ -52,10 +52,10 @@
       </inertial>
     </link>
-    <joint name="${NAME_JOINT_CHEST_CAMERA}" type="fixed">
-      <parent link="${NAME_LINK_BODY}" />
-      <child link="${NAME_LINK_CHEST_CAMERA}" />
+    <joint name="chest_camera_joint" type="fixed">
+      <parent link="body_link" />
+      <child link="chest_camera_link" />
       <origin xyz="0.114576 0.0 0.217659" rpy="-2.7925268032 0 -1.5707963268"/>
     </joint>
-    <link name="${NAME_LINK_CHEST_CAMERA}"/>
+    <link name="chest_camera_link"/>
   </xacro:macro>
 </robot>

File: urdf/sciurus17_gazebo.xacro (robot description, xacro)
@@ -31,14 +31,14 @@
       </plugin>
     </gazebo>
-    <gazebo reference="${NAME_LINK_BASE}">
-      <xacro:material_gazebo_white/>
-    </gazebo>
-    <gazebo reference="${NAME_LINK_BODY}">
-      <xacro:material_gazebo_white/>
-    </gazebo>
-    <gazebo reference="${NAME_LINK_NECK_1}">
-      <xacro:material_gazebo_white/>
-    </gazebo>
-    <gazebo reference="${NAME_LINK_NECK_2}">
+    <gazebo reference="base_link">
+      <xacro:material_gazebo_white/>
+    </gazebo>
+    <gazebo reference="body_link">
+      <xacro:material_gazebo_white/>
+    </gazebo>
+    <gazebo reference="neck_yaw_link">
+      <xacro:material_gazebo_white/>
+    </gazebo>
+    <gazebo reference="neck_pitch_link">
       <xacro:material_gazebo_white/>
     </gazebo>
@@ -98,11 +98,11 @@
     </xacro:if>
     <xacro:if value="${USE_GAZEBO_CHEST_CAMERA}">
-      <gazebo reference="${NAME_LINK_CHEST_CAMERA}">
+      <gazebo reference="chest_camera_link">
         <sensor name="${NAME_CHEST_CAMERA_PREFIX}" type="camera">
-          <pose relative_to="${NAME_LINK_CHEST_CAMERA}">0 0 0 ${radians(90)} ${radians(-90)} 0</pose>
+          <pose relative_to="chest_camera_link">0 0 0 ${radians(90)} ${radians(-90)} 0</pose>
           <update_rate>10</update_rate>
           <always_on>true</always_on>
           <topic>${NAME_CHEST_CAMERA_PREFIX}/image_raw</topic>
-          <frame_id>${NAME_LINK_CHEST_CAMERA}</frame_id>
+          <frame_id>chest_camera_link</frame_id>
           <camera name="${NAME_CHEST_CAMERA_PREFIX}">
             <xacro:property name="chest_camera_width" value="640"/>
@@ -140,62 +140,62 @@
       </gazebo>
     </xacro:if>
-    <gazebo reference="${NAME_LINK_ARM_R_1}">
-      <xacro:material_gazebo_white/>
-    </gazebo>
-    <gazebo reference="${NAME_LINK_ARM_R_2}">
-      <xacro:material_gazebo_white/>
-    </gazebo>
-    <gazebo reference="${NAME_LINK_ARM_R_3}">
-      <xacro:material_gazebo_white/>
-    </gazebo>
-    <gazebo reference="${NAME_LINK_ARM_R_4}">
-      <xacro:material_gazebo_white/>
-    </gazebo>
-    <gazebo reference="${NAME_LINK_ARM_R_5}">
-      <xacro:material_gazebo_white/>
-    </gazebo>
-    <gazebo reference="${NAME_LINK_ARM_R_6}">
-      <xacro:material_gazebo_white/>
-    </gazebo>
-    <gazebo reference="${NAME_LINK_ARM_R_7}">
-      <xacro:material_gazebo_red/>
-    </gazebo>
-    <gazebo reference="${NAME_LINK_GRIPPER_R_A}">
-      <mu1>0.8</mu1>
-      <mu2>0.8</mu2>
-      <xacro:material_gazebo_red/>
-    </gazebo>
-    <gazebo reference="${NAME_LINK_GRIPPER_R_B}">
-      <mu1>0.8</mu1>
-      <mu2>0.8</mu2>
-      <xacro:material_gazebo_red/>
-    </gazebo>
-    <gazebo reference="${NAME_LINK_ARM_L_1}">
-      <xacro:material_gazebo_white/>
-    </gazebo>
-    <gazebo reference="${NAME_LINK_ARM_L_2}">
-      <xacro:material_gazebo_white/>
-    </gazebo>
-    <gazebo reference="${NAME_LINK_ARM_L_3}">
-      <xacro:material_gazebo_white/>
-    </gazebo>
-    <gazebo reference="${NAME_LINK_ARM_L_4}">
-      <xacro:material_gazebo_white/>
-    </gazebo>
-    <gazebo reference="${NAME_LINK_ARM_L_5}">
-      <xacro:material_gazebo_white/>
-    </gazebo>
-    <gazebo reference="${NAME_LINK_ARM_L_6}">
-      <xacro:material_gazebo_white/>
-    </gazebo>
-    <gazebo reference="${NAME_LINK_ARM_L_7}">
-      <xacro:material_gazebo_red/>
-    </gazebo>
-    <gazebo reference="${NAME_LINK_GRIPPER_L_A}">
-      <mu1>0.8</mu1>
-      <mu2>0.8</mu2>
-      <xacro:material_gazebo_red/>
-    </gazebo>
-    <gazebo reference="${NAME_LINK_GRIPPER_L_B}">
+    <gazebo reference="r_link1">
+      <xacro:material_gazebo_white/>
+    </gazebo>
+    <gazebo reference="r_link2">
+      <xacro:material_gazebo_white/>
+    </gazebo>
+    <gazebo reference="r_link3">
+      <xacro:material_gazebo_white/>
+    </gazebo>
+    <gazebo reference="r_link4">
+      <xacro:material_gazebo_white/>
+    </gazebo>
+    <gazebo reference="r_link5">
+      <xacro:material_gazebo_white/>
+    </gazebo>
+    <gazebo reference="r_link6">
+      <xacro:material_gazebo_white/>
+    </gazebo>
+    <gazebo reference="r_link7">
+      <xacro:material_gazebo_red/>
+    </gazebo>
+    <gazebo reference="r_gripperA_link">
+      <mu1>0.8</mu1>
+      <mu2>0.8</mu2>
+      <xacro:material_gazebo_red/>
+    </gazebo>
+    <gazebo reference="r_gripperB_link">
+      <mu1>0.8</mu1>
+      <mu2>0.8</mu2>
+      <xacro:material_gazebo_red/>
+    </gazebo>
+    <gazebo reference="l_link1">
+      <xacro:material_gazebo_white/>
+    </gazebo>
+    <gazebo reference="l_link2">
+      <xacro:material_gazebo_white/>
+    </gazebo>
+    <gazebo reference="l_link3">
+      <xacro:material_gazebo_white/>
+    </gazebo>
+    <gazebo reference="l_link4">
+      <xacro:material_gazebo_white/>
+    </gazebo>
+    <gazebo reference="l_link5">
+      <xacro:material_gazebo_white/>
+    </gazebo>
+    <gazebo reference="l_link6">
+      <xacro:material_gazebo_white/>
+    </gazebo>
+    <gazebo reference="l_link7">
+      <xacro:material_gazebo_red/>
+    </gazebo>
+    <gazebo reference="l_gripperA_link">
+      <mu1>0.8</mu1>
+      <mu2>0.8</mu2>
+      <xacro:material_gazebo_red/>
+    </gazebo>
+    <gazebo reference="l_gripperB_link">
       <mu1>0.8</mu1>
       <mu2>0.8</mu2>
