Commit message: リンク名とジョイント名のproperty定義を廃止

File: urdf/sciurus17_head.xacro (robot description, xacro)
@@ -2,7 +2,7 @@
 <robot xmlns:xacro="http://ros.org/wiki/xacro">
   <xacro:macro name="sciurus17_head">
-    <joint name="${NAME_JOINT_NECK_1}" type="revolute">
-      <parent link="${NAME_LINK_BODY}" />
-      <child link="${NAME_LINK_NECK_1}" />
+    <joint name="neck_yaw_joint" type="revolute">
+      <parent link="body_link" />
+      <child link="neck_yaw_link" />
       <origin xyz="0.08083 0.0 0.3395" rpy="0 0 0"/>
       <limit
@@ -14,5 +14,5 @@
       <dynamics damping="1.0e-6" friction="0.8"/>
     </joint>
-    <link name="${NAME_LINK_NECK_1}">
+    <link name="neck_yaw_link">
       <visual>
         <geometry>
@@ -32,7 +32,7 @@
       </inertial>
     </link>
-    <joint name="${NAME_JOINT_NECK_2}" type="revolute">
-      <parent link="${NAME_LINK_NECK_1}" />
-      <child link="${NAME_LINK_NECK_2}" />
+    <joint name="neck_pitch_joint" type="revolute">
+      <parent link="neck_yaw_link" />
+      <child link="neck_pitch_link" />
       <origin xyz="0.0 0.0 0.054" rpy="0 0 0"/>
       <limit
@@ -44,5 +44,5 @@
       <dynamics damping="1.0e-6" friction="0.8"/>
     </joint>
-    <link name="${NAME_LINK_NECK_2}">
+    <link name="neck_pitch_link">
       <visual>
         <origin rpy="1.5708 0 0" xyz="0.0 0.0 0.0"/>
@@ -64,10 +64,10 @@
       </inertial>
     </link>
-    <joint name="${NAME_JOINT_HEAD_CAMERA}" type="fixed">
-      <parent link="${NAME_LINK_NECK_2}" />
-      <child link="${NAME_LINK_HEAD_CAMERA}" />
+    <joint name="head_camera_joint" type="fixed">
+      <parent link="neck_pitch_link" />
+      <child link="head_camera_link" />
       <origin xyz="0.081785 0.020 0.091" rpy="0 0 0"/>
     </joint>
-    <link name="${NAME_LINK_HEAD_CAMERA}"/>
+    <link name="head_camera_link"/>
   </xacro:macro>
 </robot>

File: urdf/sciurus17_left_arm.xacro (robot description, xacro)
@@ -2,7 +2,7 @@
 <robot xmlns:xacro="http://ros.org/wiki/xacro">
   <xacro:macro name="sciurus17_left_arm">
-    <joint name="${NAME_JOINT_ARM_L_1}" type="revolute">
-      <parent link="${NAME_LINK_BODY}" />
-      <child link="${NAME_LINK_ARM_L_1}" />
+    <joint name="l_arm_joint1" type="revolute">
+      <parent link="body_link" />
+      <child link="l_link1" />
       <origin xyz="0.08083 0.0965 0.2885" rpy="0 0 0"/>
       <limit
@@ -14,5 +14,5 @@
       <dynamics damping="1.0e-6" friction="0.8"/>
     </joint>
-    <link name="${NAME_LINK_ARM_L_1}">
+    <link name="l_link1">
       <visual>
         <origin rpy="-1.5708 0 0" xyz="0.0 0.0 0.0"/>
@@ -34,7 +34,7 @@
       </inertial>
     </link>
-    <joint name="${NAME_JOINT_ARM_L_2}" type="revolute">
-      <parent link="${NAME_LINK_ARM_L_1}" />
-      <child link="${NAME_LINK_ARM_L_2}" />
+    <joint name="l_arm_joint2" type="revolute">
+      <parent link="l_link1" />
+      <child link="l_link2" />
       <origin xyz="0.0 0.064 0.0" rpy="0 0 0"/>
       <limit
@@ -46,5 +46,5 @@
       <dynamics damping="1.0e-6" friction="0.8"/>
     </joint>
-    <link name="${NAME_LINK_ARM_L_2}">
+    <link name="l_link2">
       <visual>
         <origin rpy="0 -1.5708 0" xyz="0.0 0.0 0.0"/>
@@ -66,7 +66,7 @@
       </inertial>
     </link>
-    <joint name="${NAME_JOINT_ARM_L_3}" type="revolute">
-      <parent link="${NAME_LINK_ARM_L_2}" />
-      <child link="${NAME_LINK_ARM_L_3}" />
+    <joint name="l_arm_joint3" type="revolute">
+      <parent link="l_link2" />
+      <child link="l_link3" />
       <origin xyz="0.0 0.065 0.0" rpy="0 0 0"/>
       <limit
@@ -78,5 +78,5 @@
       <dynamics damping="1.0e-6" friction="0.8"/>
     </joint>
-    <link name="${NAME_LINK_ARM_L_3}">
+    <link name="l_link3">
       <visual>
         <origin rpy="-1.5708 0 0" xyz="0.0 0.0 0.0"/>
@@ -98,7 +98,7 @@
       </inertial>
     </link>
-    <joint name="${NAME_JOINT_ARM_L_4}" type="revolute">
-      <parent link="${NAME_LINK_ARM_L_3}" />
-      <child link="${NAME_LINK_ARM_L_4}" />
+    <joint name="l_arm_joint4" type="revolute">
+      <parent link="l_link3" />
+      <child link="l_link4" />
       <origin xyz="0.0 0.185 0.0" rpy="0 0 0"/>
       <limit
@@ -110,5 +110,5 @@
       <dynamics damping="1.0e-6" friction="0.8"/>
     </joint>
-    <link name="${NAME_LINK_ARM_L_4}">
+    <link name="l_link4">
       <visual>
         <origin rpy="0 0 0" xyz="0.0 0.0 0.0"/>
@@ -130,7 +130,7 @@
       </inertial>
     </link>
-    <joint name="${NAME_JOINT_ARM_L_5}" type="revolute">
-      <parent link="${NAME_LINK_ARM_L_4}" />
-      <child link="${NAME_LINK_ARM_L_5}" />
+    <joint name="l_arm_joint5" type="revolute">
+      <parent link="l_link4" />
+      <child link="l_link5" />
       <origin xyz="0.0 0.121 0.0" rpy="0 0 0"/>
       <limit
@@ -142,5 +142,5 @@
       <dynamics damping="1.0e-6" friction="0.8"/>
     </joint>
-    <link name="${NAME_LINK_ARM_L_5}">
+    <link name="l_link5">
       <visual>
         <origin rpy="-1.5708 0 0" xyz="0.0 0.0 0.0"/>
@@ -180,10 +180,10 @@
       </inertial>
     </link>
-    <joint name="${NAME_JOINT_ARMARKER_L}" type="fixed">
-      <parent link="${NAME_LINK_ARM_L_5}" />
-      <child link="${NAME_LINK_ARMARKER_L}" />
+    <joint name="l_arm_armarker" type="fixed">
+      <parent link="l_link5" />
+      <child link="l_link5_armarker" />
       <origin xyz="0.0467 0.093 0.0" rpy="0 0 0"/>
     </joint>
-    <link name="${NAME_LINK_ARMARKER_L}">
+    <link name="l_link5_armarker">
       <visual>
         <origin rpy="0 0 0" xyz="0.0 0.0 0.0"/>
@@ -200,7 +200,7 @@
       </collision>
     </link>
-    <joint name="${NAME_JOINT_ARM_L_6}" type="revolute">
-      <parent link="${NAME_LINK_ARM_L_5}" />
-      <child link="${NAME_LINK_ARM_L_6}" />
+    <joint name="l_arm_joint6" type="revolute">
+      <parent link="l_link5" />
+      <child link="l_link6" />
       <origin xyz="0.0 0.129 0.0" rpy="0 0 0"/>
       <limit
@@ -212,5 +212,5 @@
       <dynamics damping="1.0e-6" friction="0.8"/>
     </joint>
-    <link name="${NAME_LINK_ARM_L_6}">
+    <link name="l_link6">
       <visual>
         <origin rpy="0 0 0" xyz="0.0 0.0 0.0"/>
@@ -232,7 +232,7 @@
       </inertial>
     </link>
-    <joint name="${NAME_JOINT_ARM_L_7}" type="revolute">
-      <parent link="${NAME_LINK_ARM_L_6}" />
-      <child link="${NAME_LINK_ARM_L_7}" />
+    <joint name="l_arm_joint7" type="revolute">
+      <parent link="l_link6" />
+      <child link="l_link7" />
       <origin xyz="0.0 0.0191 0.0" rpy="0 0 0"/>
       <limit

File: urdf/sciurus17_left_gripper.xacro (robot description, xacro)
@@ -2,5 +2,5 @@
 <robot xmlns:xacro="http://ros.org/wiki/xacro">
   <xacro:macro name="sciurus17_left_gripper">
-    <link name="${NAME_LINK_ARM_L_7}">
+    <link name="l_link7">
       <visual>
         <origin rpy="1.5708 0 0" xyz="0.0 0.0 0.0"/>
@@ -22,7 +22,7 @@
       </inertial>
     </link>
-    <joint name="${NAME_JOINT_GRIPPER_L_A}" type="revolute">
-      <parent link="${NAME_LINK_ARM_L_7}" />
-      <child link="${NAME_LINK_GRIPPER_L_A}" />
+    <joint name="l_gripper_joint" type="revolute">
+      <parent link="l_link7" />
+      <child link="l_gripperA_link" />
       <origin xyz="0.012 0.024 0.0" rpy="0 0 0"/>
       <limit
@@ -34,5 +34,5 @@
       <dynamics damping="1.0e-6" friction="0.8"/>
     </joint>
-    <link name="${NAME_LINK_GRIPPER_L_A}">
+    <link name="l_gripperA_link">
       <visual>
         <origin rpy="0 0 0" xyz="0.0 0.0 0.0"/>
@@ -54,7 +54,7 @@
       </inertial>
     </link>
-    <joint name="${NAME_JOINT_GRIPPER_L_B}" type="revolute">
-      <parent link="${NAME_LINK_ARM_L_7}" />
-      <child link="${NAME_LINK_GRIPPER_L_B}" />
+    <joint name="l_gripper_mimic_joint" type="revolute">
+      <parent link="l_link7" />
+      <child link="l_gripperB_link" />
       <origin xyz="-0.012 0.024 0.0" rpy="0 0 0"/>
       <limit
@@ -64,8 +64,8 @@
         velocity="${VELOCITY_LIMIT}"/>
       <axis xyz="0 0 -1"/>
-      <mimic joint="${NAME_JOINT_GRIPPER_L_A}" multiplier="1" offset="0"/>
+      <mimic joint="l_gripper_joint" multiplier="1" offset="0"/>
       <dynamics damping="1.0e-6" friction="0.8"/>
     </joint>
-    <link name="${NAME_LINK_GRIPPER_L_B}">
+    <link name="l_gripperB_link">
       <visual>
         <origin rpy="0 0 0" xyz="0.0 0.0 0.0"/>

File: urdf/sciurus17_right_arm.xacro (robot description, xacro)
@@ -2,7 +2,7 @@
 <robot xmlns:xacro="http://ros.org/wiki/xacro">
   <xacro:macro name="sciurus17_right_arm">
-    <joint name="${NAME_JOINT_ARM_R_1}" type="revolute">
-      <parent link="${NAME_LINK_BODY}" />
-      <child link="${NAME_LINK_ARM_R_1}" />
+    <joint name="r_arm_joint1" type="revolute">
+      <parent link="body_link" />
+      <child link="r_link1" />
       <origin xyz="0.08083 -0.0965 0.2885" rpy="0 0 0"/>
       <limit
@@ -14,5 +14,5 @@
       <dynamics damping="1.0e-6" friction="0.8"/>
     </joint>
-    <link name="${NAME_LINK_ARM_R_1}">
+    <link name="r_link1">
       <visual>
         <origin rpy="1.5708 0 0" xyz="0.0 0.0 0.0"/>
@@ -34,7 +34,7 @@
       </inertial>
     </link>
-    <joint name="${NAME_JOINT_ARM_R_2}" type="revolute">
-      <parent link="${NAME_LINK_ARM_R_1}" />
-      <child link="${NAME_LINK_ARM_R_2}" />
+    <joint name="r_arm_joint2" type="revolute">
+      <parent link="r_link1" />
+      <child link="r_link2" />
       <origin xyz="0.0 -0.064 0.0" rpy="0 0 0"/>
       <limit
@@ -46,5 +46,5 @@
       <dynamics damping="1.0e-6" friction="0.8"/>
     </joint>
-    <link name="${NAME_LINK_ARM_R_2}">
+    <link name="r_link2">
       <visual>
         <origin rpy="0 1.5708 0" xyz="0.0 0.0 0.0"/>
@@ -66,7 +66,7 @@
       </inertial>
     </link>
-    <joint name="${NAME_JOINT_ARM_R_3}" type="revolute">
-      <parent link="${NAME_LINK_ARM_R_2}" />
-      <child link="${NAME_LINK_ARM_R_3}" />
+    <joint name="r_arm_joint3" type="revolute">
+      <parent link="r_link2" />
+      <child link="r_link3" />
       <origin xyz="0.0 -0.065 0.0" rpy="0 0 0"/>
       <limit
@@ -78,5 +78,5 @@
       <dynamics damping="1.0e-6" friction="0.8"/>
     </joint>
-    <link name="${NAME_LINK_ARM_R_3}">
+    <link name="r_link3">
       <visual>
         <origin rpy="1.5708 0 0" xyz="0.0 0.0 0.0"/>
@@ -98,7 +98,7 @@
       </inertial>
     </link>
-    <joint name="${NAME_JOINT_ARM_R_4}" type="revolute">
-      <parent link="${NAME_LINK_ARM_R_3}" />
-      <child link="${NAME_LINK_ARM_R_4}" />
+    <joint name="r_arm_joint4" type="revolute">
+      <parent link="r_link3" />
+      <child link="r_link4" />
       <origin xyz="0.0 -0.185 0.0" rpy="0 0 0"/>
       <limit
@@ -110,5 +110,5 @@
       <dynamics damping="1.0e-6" friction="0.8"/>
     </joint>
-    <link name="${NAME_LINK_ARM_R_4}">
+    <link name="r_link4">
       <visual>
         <origin rpy="0 0 0" xyz="0.0 0.0 0.0"/>
@@ -130,7 +130,7 @@
       </inertial>
     </link>
-    <joint name="${NAME_JOINT_ARM_R_5}" type="revolute">
-      <parent link="${NAME_LINK_ARM_R_4}" />
-      <child link="${NAME_LINK_ARM_R_5}" />
+    <joint name="r_arm_joint5" type="revolute">
+      <parent link="r_link4" />
+      <child link="r_link5" />
       <origin xyz="0.0 -0.121 0.0" rpy="0 0 0"/>
       <limit
@@ -142,5 +142,5 @@
       <dynamics damping="1.0e-6" friction="0.8"/>
     </joint>
-    <link name="${NAME_LINK_ARM_R_5}">
+    <link name="r_link5">
       <visual>
         <origin rpy="1.5708 0 0" xyz="0.0 0.0 0.0"/>
@@ -180,10 +180,10 @@
       </inertial>
     </link>
-    <joint name="${NAME_JOINT_ARMARKER_R}" type="fixed">
-      <parent link="${NAME_LINK_ARM_R_5}" />
-      <child link="${NAME_LINK_ARMARKER_R}" />
+    <joint name="r_arm_armarker" type="fixed">
+      <parent link="r_link5" />
+      <child link="r_link5_armarker" />
       <origin xyz="0.0467 -0.093 0.0" rpy="0 0 0"/>
     </joint>
-    <link name="${NAME_LINK_ARMARKER_R}">
+    <link name="r_link5_armarker">
       <visual>
         <origin rpy="0 0 0" xyz="0.0 0.0 0.0"/>
@@ -200,7 +200,7 @@
       </collision>
     </link>
-    <joint name="${NAME_JOINT_ARM_R_6}" type="revolute">
-      <parent link="${NAME_LINK_ARM_R_5}" />
-      <child link="${NAME_LINK_ARM_R_6}" />
+    <joint name="r_arm_joint6" type="revolute">
+      <parent link="r_link5" />
+      <child link="r_link6" />
       <origin xyz="0.0 -0.129 0.0" rpy="0 0 0"/>
       <limit
@@ -212,5 +212,5 @@
       <dynamics damping="1.0e-6" friction="0.8"/>
     </joint>
-    <link name="${NAME_LINK_ARM_R_6}">
+    <link name="r_link6">
       <visual>
         <origin rpy="0 0 0" xyz="0.0 0.0 0.0"/>
@@ -232,7 +232,7 @@
       </inertial>
     </link>
-    <joint name="${NAME_JOINT_ARM_R_7}" type="revolute">
-      <parent link="${NAME_LINK_ARM_R_6}" />
-      <child link="${NAME_LINK_ARM_R_7}" />
+    <joint name="r_arm_joint7" type="revolute">
+      <parent link="r_link6" />
+      <child link="r_link7" />
       <origin xyz="0.0 -0.0191 0.0" rpy="0 0 0"/>
       <limit

File: urdf/sciurus17_right_gripper.xacro (robot description, xacro)
@@ -2,5 +2,5 @@
 <robot xmlns:xacro="http://ros.org/wiki/xacro">
   <xacro:macro name="sciurus17_right_gripper">
-    <link name="${NAME_LINK_ARM_R_7}">
+    <link name="r_link7">
       <visual>
         <origin rpy="1.5708 0 0" xyz="0.0 0.0 0.0"/>
@@ -22,7 +22,7 @@
       </inertial>
     </link>
-    <joint name="${NAME_JOINT_GRIPPER_R_A}" type="revolute">
-      <parent link="${NAME_LINK_ARM_R_7}" />
-      <child link="${NAME_LINK_GRIPPER_R_A}" />
+    <joint name="r_gripper_joint" type="revolute">
+      <parent link="r_link7" />
+      <child link="r_gripperA_link" />
       <origin xyz="0.012 -0.024 0.0" rpy="0 0 0"/>
       <limit
@@ -34,5 +34,5 @@
       <dynamics damping="1.0e-6" friction="0.8"/>
     </joint>
-    <link name="${NAME_LINK_GRIPPER_R_A}">
+    <link name="r_gripperA_link">
       <visual>
         <!--origin rpy="3.14159 0 0" xyz="0.0 0.0 0.0"/-->
@@ -55,7 +55,7 @@
       </inertial>
     </link>
-    <joint name="${NAME_JOINT_GRIPPER_R_B}" type="revolute">
-      <parent link="${NAME_LINK_ARM_R_7}" />
-      <child link="${NAME_LINK_GRIPPER_R_B}" />
+    <joint name="r_gripper_mimic_joint" type="revolute">
+      <parent link="r_link7" />
+      <child link="r_gripperB_link" />
       <origin xyz="-0.012 -0.024 0.0" rpy="0 0 0"/>
       <limit
@@ -65,8 +65,8 @@
         velocity="${VELOCITY_LIMIT}"/>
       <axis xyz="0 0 -1"/>
-      <mimic joint="${NAME_JOINT_GRIPPER_R_A}" multiplier="1" offset="0"/>
+      <mimic joint="r_gripper_joint" multiplier="1" offset="0"/>
       <dynamics damping="1.0e-6" friction="0.8"/>
     </joint>
-    <link name="${NAME_LINK_GRIPPER_R_B}">
+    <link name="r_gripperB_link">
       <visual>
         <!-- origin rpy="3.14159 0 0" xyz="0.0 0.0 0.0"/ -->
