Commit message: add mock components support

File: urdf/sciurus17.ros2_control.xacro (robot description, xacro)
@@ -4,9 +4,14 @@
     <ros2_control name="sciurus17" type="system">
       <hardware>
-        <plugin>sciurus17_hardware/Sciurus17Hardware</plugin>
-        <param name="port_name">${PORT_NAME}</param>
-        <param name="baudrate">${BAUDRATE}</param>
-        <param name="timeout_seconds">${TIMEOUT_SECONDS}</param>
-        <param name="manipulator_config_file_path">${MANIPULATOR_CONFIG_FILE_PATH}</param>
+        <xacro:if value="${USE_MOCK_COMPONENTS}">
+          <plugin>mock_components/GenericSystem</plugin>
+        </xacro:if>
+        <xacro:unless value="${USE_MOCK_COMPONENTS}">
+          <plugin>sciurus17_hardware/Sciurus17Hardware</plugin>
+          <param name="port_name">${PORT_NAME}</param>
+          <param name="baudrate">${BAUDRATE}</param>
+          <param name="timeout_seconds">${TIMEOUT_SECONDS}</param>
+          <param name="manipulator_config_file_path">${MANIPULATOR_CONFIG_FILE_PATH}</param>
+        </xacro:unless>
       </hardware>
       <joint name="${NAME_JOINT_BODY}">

File: urdf/sciurus17.urdf.xacro (robot description, xacro)
@@ -18,4 +18,5 @@
   <xacro:arg name="use_gazebo_head_camera" default="false" />
   <xacro:arg name="use_gazebo_chest_camera" default="false" />
+  <xacro:arg name="use_mock_components" default="false" />
   <xacro:arg name="port_name" default="/dev/sciurus17spine" />
   <xacro:arg name="baudrate" default="3000000" />
@@ -26,4 +27,5 @@
   <xacro:property name="USE_GAZEBO_HEAD_CAMERA" value="$(arg use_gazebo_head_camera)"/>
   <xacro:property name="USE_GAZEBO_CHEST_CAMERA" value="$(arg use_gazebo_chest_camera)"/>
+  <xacro:property name="USE_MOCK_COMPONENTS" value="$(arg use_mock_components)"/>
   <xacro:property name="PORT_NAME" value="$(arg port_name)"/>
   <xacro:property name="BAUDRATE" value="$(arg baudrate)"/>
