Commit message: 引数のproperty定義を廃止

File: urdf/sciurus17.ros2_control.xacro (robot description, xacro)
@@ -1,16 +1,21 @@
 <?xml version="1.0"?>
 <robot xmlns:xacro="http://www.ros.org/wiki/xacro">
-  <xacro:macro name="sciurus17_ros2_control_settings">
+  <xacro:macro name="sciurus17_ros2_control_settings"
+               params="use_mock_components:=false
+                       port_name:=/dev/sciurus17spine
+                       baudrate:=3000000
+                       timeout_seconds:=1.0
+                       manipulator_config_file_path:=''">
     <ros2_control name="sciurus17" type="system">
       <hardware>
-        <xacro:if value="${USE_MOCK_COMPONENTS}">
+        <xacro:if value="${use_mock_components}">
           <plugin>mock_components/GenericSystem</plugin>
         </xacro:if>
-        <xacro:unless value="${USE_MOCK_COMPONENTS}">
+        <xacro:unless value="${use_mock_components}">
           <plugin>sciurus17_hardware/Sciurus17Hardware</plugin>
-          <param name="port_name">${PORT_NAME}</param>
-          <param name="baudrate">${BAUDRATE}</param>
-          <param name="timeout_seconds">${TIMEOUT_SECONDS}</param>
-          <param name="manipulator_config_file_path">${MANIPULATOR_CONFIG_FILE_PATH}</param>
+          <param name="port_name">${port_name}</param>
+          <param name="baudrate">${baudrate}</param>
+          <param name="timeout_seconds">${timeout_seconds}</param>
+          <param name="manipulator_config_file_path">${manipulator_config_file_path}</param>
         </xacro:unless>
       </hardware>

File: urdf/sciurus17.urdf.xacro (robot description, xacro)
@@ -25,13 +25,4 @@
   <xacro:arg name="gz_control_config_package" default="" />
   <xacro:arg name="gz_control_config_file_path" default="" />
-  <xacro:property name="USE_GAZEBO_HEAD_CAMERA" value="$(arg use_gazebo_head_camera)"/>
-  <xacro:property name="USE_GAZEBO_CHEST_CAMERA" value="$(arg use_gazebo_chest_camera)"/>
-  <xacro:property name="USE_MOCK_COMPONENTS" value="$(arg use_mock_components)"/>
-  <xacro:property name="PORT_NAME" value="$(arg port_name)"/>
-  <xacro:property name="BAUDRATE" value="$(arg baudrate)"/>
-  <xacro:property name="TIMEOUT_SECONDS" value="$(arg timeout_seconds)"/>
-  <xacro:property name="MANIPULATOR_CONFIG_FILE_PATH" value="$(arg manipulator_config_file_path)"/>
-  <xacro:property name="GZ_CONTROL_CONFIG_PACKAGE" value="$(arg gz_control_config_package)"/>
-  <xacro:property name="GZ_CONTROL_CONFIG_FILE_PATH" value="$(arg gz_control_config_file_path)"/>
   <xacro:property name="NAME_HEAD_CAMERA_PREFIX" value="head_camera"/>
   <xacro:property name="NAME_CHEST_CAMERA_PREFIX" value="chest_camera"/>
@@ -107,8 +98,17 @@
   <xacro:sciurus17_left_gripper/>
   <xacro:unless value="$(arg use_gazebo)">
-    <xacro:sciurus17_ros2_control_settings/>
+    <xacro:sciurus17_ros2_control_settings
+      use_mock_components="$(arg use_mock_components)"
+      port_name="$(arg port_name)"
+      baudrate="$(arg baudrate)"
+      timeout_seconds="$(arg timeout_seconds)"
+      manipulator_config_file_path="$(arg manipulator_config_file_path)"/>
   </xacro:unless>
   <xacro:if value="$(arg use_gazebo)">
-    <xacro:gazebo_robot_settings/>
+    <xacro:gazebo_robot_settings
+      use_gazebo_head_camera="$(arg use_gazebo_head_camera)"
+      use_gazebo_chest_camera="$(arg use_gazebo_chest_camera)"
+      gz_control_config_package="$(arg gz_control_config_package)"
+      gz_control_config_file_path="$(arg gz_control_config_file_path)"/>
     <xacro:sciurus17_gazebo_ros2_control_settings/>
     <joint name="${NAME_HEAD_CAMERA_PREFIX}_color_joint" type="fixed">

File: urdf/sciurus17_gazebo.xacro (robot description, xacro)
@@ -25,8 +25,12 @@
     </visual>
   </xacro:macro>
-  <xacro:macro name="gazebo_robot_settings">
+  <xacro:macro name="gazebo_robot_settings"
+               params="use_gazebo_head_camera:=false
+               use_gazebo_chest_camera:=false
+               gz_control_config_package:=''
+               gz_control_config_file_path:=''">
     <gazebo>
       <plugin filename="libgz_ros2_control-system.so" name="gz_ros2_control::GazeboSimROS2ControlPlugin">
-        <parameters>$(find ${GZ_CONTROL_CONFIG_PACKAGE})/${GZ_CONTROL_CONFIG_FILE_PATH}</parameters>
+        <parameters>$(find ${gz_control_config_package})/${gz_control_config_file_path}</parameters>
       </plugin>
     </gazebo>
@@ -48,5 +52,5 @@
       </plugin>
     </gazebo>
-    <xacro:if value="${USE_GAZEBO_HEAD_CAMERA}">
+    <xacro:if value="${use_gazebo_head_camera}">
       <gazebo reference="${NAME_HEAD_CAMERA_PREFIX}_color_frame">
         <sensor name="sim_realsense_d415" type="rgbd_camera">
@@ -97,5 +101,5 @@
       </gazebo>
     </xacro:if>
-    <xacro:if value="${USE_GAZEBO_CHEST_CAMERA}">
+    <xacro:if value="${use_gazebo_chest_camera}">
       <gazebo reference="chest_camera_link">
         <sensor name="${NAME_CHEST_CAMERA_PREFIX}" type="camera">

Commit message: ワークショップ用の追記箇所を削除

File: urdf/sciurus17.ros2_control.xacro (robot description, xacro)
@@ -11,7 +11,5 @@
       <hardware>
         <xacro:if value="${use_isaacsim}">
-          <plugin>topic_based_ros2_control/TopicBasedSystem</plugin>
-          <param name="joint_commands_topic">/joint_command</param>
-          <param name="joint_states_topic">/joint_states</param>
+          <!-- 追記箇所 -->
         </xacro:if>
         <xacro:unless value="${use_isaacsim}">

File: urdf/sciurus17.urdf.xacro (robot description, xacro)
@@ -114,16 +114,5 @@
   </xacro:if>
   <xacro:if value="${'$(arg use_gazebo)' == 'true' or '$(arg use_isaacsim)' == 'true'}">
-    <joint name="head_camera_color_joint" type="fixed">
-      <origin xyz="0 0.015 0" rpy="0 0 0" />
-      <parent link="head_camera_link" />
-      <child link="head_camera_color_frame" />
-    </joint>
-    <link name="head_camera_color_frame"/>
-    <joint name="head_camera_color_optical_joint" type="fixed">
-      <origin xyz="0 0 0" rpy="${radians(-90)} 0 ${radians(-90)}" />
-      <parent link="head_camera_color_frame" />
-      <child link="head_camera_color_optical_frame" />
-    </joint>
-    <link name="head_camera_color_optical_frame"/>
+    <!-- 追記箇所 -->
   </xacro:if>
 </robot>
