Commit message: hand表記をgripperへ変更

File: urdf/sciurus17_left_gripper.xacro (robot description, xacro)
@@ -38,5 +38,5 @@
         <origin rpy="0 0 0" xyz="0.0 0.0 0.0"/>
         <geometry>
-          <mesh filename="package://sciurus17_description/meshes/visual/L_HandA.stl" scale="1.0 1.0 1.0"/>
+          <mesh filename="package://sciurus17_description/meshes/visual/L_GripperA.stl" scale="1.0 1.0 1.0"/>
         </geometry>
         <material name="${COLOR_LINK_GRIPPER}"/>
@@ -45,5 +45,5 @@
         <origin rpy="0 0 0" xyz="0.0 0.0 0.0"/>
         <geometry>
-          <mesh filename="package://sciurus17_description/meshes/collision/L_HandA.stl" scale="1.0 1.0 1.0"/>
+          <mesh filename="package://sciurus17_description/meshes/collision/L_GripperA.stl" scale="1.0 1.0 1.0"/>
         </geometry>
       </collision>
@@ -79,5 +79,5 @@
         <origin rpy="0 0 0" xyz="0.0 0.0 0.0"/>
         <geometry>
-          <mesh filename="package://sciurus17_description/meshes/visual/L_HandB.stl" scale="1.0 1.0 1.0"/>
+          <mesh filename="package://sciurus17_description/meshes/visual/L_GripperB.stl" scale="1.0 1.0 1.0"/>
         </geometry>
         <material name="${COLOR_LINK_GRIPPER}"/>
@@ -86,5 +86,5 @@
         <origin rpy="0 0 0" xyz="0.0 0.0 0.0"/>
         <geometry>
-          <mesh filename="package://sciurus17_description/meshes/collision/L_HandB.stl" scale="1.0 1.0 1.0"/>
+          <mesh filename="package://sciurus17_description/meshes/collision/L_GripperB.stl" scale="1.0 1.0 1.0"/>
         </geometry>
       </collision>

File: urdf/sciurus17_right_gripper.xacro (robot description, xacro)
@@ -39,5 +39,5 @@
         <origin rpy="0 0 0" xyz="0.0 0.0 0.0"/>
         <geometry>
-          <mesh filename="package://sciurus17_description/meshes/visual/R_HandA.stl" scale="1.0 1.0 1.0"/>
+          <mesh filename="package://sciurus17_description/meshes/visual/R_GripperA.stl" scale="1.0 1.0 1.0"/>
         </geometry>
         <material name="${COLOR_LINK_GRIPPER}"/>
@@ -46,5 +46,5 @@
         <origin rpy="0 0 0" xyz="0.0 0.0 0.0"/>
         <geometry>
-          <mesh filename="package://sciurus17_description/meshes/collision/R_HandA.stl" scale="1.0 1.0 1.0"/>
+          <mesh filename="package://sciurus17_description/meshes/collision/R_GripperA.stl" scale="1.0 1.0 1.0"/>
         </geometry>
       </collision>
@@ -81,5 +81,5 @@
         <origin rpy="0 0 0" xyz="0.0 0.0 0.0"/>
         <geometry>
-          <mesh filename="package://sciurus17_description/meshes/visual/R_HandB.stl" scale="1.0 1.0 1.0"/>
+          <mesh filename="package://sciurus17_description/meshes/visual/R_GripperB.stl" scale="1.0 1.0 1.0"/>
         </geometry>
         <material name="${COLOR_LINK_GRIPPER}"/>
@@ -88,5 +88,5 @@
         <origin rpy="0 0 0" xyz="0.0 0.0 0.0"/>
         <geometry>
-          <mesh filename="package://sciurus17_description/meshes/collision/R_HandB.stl" scale="1.0 1.0 1.0"/>
+          <mesh filename="package://sciurus17_description/meshes/collision/R_GripperB.stl" scale="1.0 1.0 1.0"/>
         </geometry>
       </collision>

Commit message: エラー回避用のdummyジョイントの定義を削除

File: urdf/sciurus17_left_gripper.xacro (robot description, xacro)
@@ -54,12 +54,4 @@
       </inertial>
     </link>
-    <!--Dummy joint/link to prevent error with mimic joint
-    See https://github.com/ros-controls/gazebo_ros2_control/issues/173
-    -->
-    <joint name="${NAME_JOINT_GRIPPER_L_B}_mimic" type="fixed">
-      <parent link="world" />
-      <child link="dummy_mimic_fix_l" />
-    </joint>
-    <link name="dummy_mimic_fix_l"/>
     <joint name="${NAME_JOINT_GRIPPER_L_B}" type="revolute">
       <parent link="${NAME_LINK_ARM_L_7}" />

File: urdf/sciurus17_right_gripper.xacro (robot description, xacro)
@@ -55,12 +55,4 @@
       </inertial>
     </link>
-    <!--Dummy joint/link to prevent error with mimic joint
-    See https://github.com/ros-controls/gazebo_ros2_control/issues/173
-    -->
-    <joint name="${NAME_JOINT_GRIPPER_R_B}_mimic" type="fixed">
-      <parent link="world" />
-      <child link="dummy_mimic_fix_r" />
-    </joint>
-    <link name="dummy_mimic_fix_r"/>
     <joint name="${NAME_JOINT_GRIPPER_R_B}" type="revolute">
       <parent link="${NAME_LINK_ARM_R_7}" />
