Commit message: link、joint名のproperty化

File: urdf/sciurus17.urdf.xacro (robot description, xacro)
@@ -13,4 +13,56 @@
     <color rgba="0.8984375 0.0 0.0703125 1"/>
   </material>
+  <xacro:property name="NAME_LINK_BASE" value="base_link"/>
+  <xacro:property name="NAME_LINK_BODY" value="body_link"/>
+  <xacro:property name="NAME_LINK_NECK_1" value="neck_yaw_link"/>
+  <xacro:property name="NAME_LINK_NECK_2" value="neck_pitch_link"/>
+  <xacro:property name="NAME_LINK_CAMERA" value="camera_link"/>
+  <xacro:property name="NAME_LINK_CHEST_CAMERA" value="chest_camera_link"/>
+  <xacro:property name="NAME_LINK_ARM_R_1" value="r_link1"/>
+  <xacro:property name="NAME_LINK_ARM_R_2" value="r_link2"/>
+  <xacro:property name="NAME_LINK_ARM_R_3" value="r_link3"/>
+  <xacro:property name="NAME_LINK_ARM_R_4" value="r_link4"/>
+  <xacro:property name="NAME_LINK_ARM_R_5" value="r_link5"/>
+  <xacro:property name="NAME_LINK_ARM_R_6" value="r_link6"/>
+  <xacro:property name="NAME_LINK_ARM_R_7" value="r_link7"/>
+  <xacro:property name="NAME_LINK_HAND_R_A" value="r_handA_link"/>
+  <xacro:property name="NAME_LINK_HAND_R_B" value="r_handB_link"/>
+  <xacro:property name="NAME_LINK_ARMARKER_R" value="r_link5_armarker"/>
+  <xacro:property name="NAME_LINK_ARM_L_1" value="l_link1"/>
+  <xacro:property name="NAME_LINK_ARM_L_2" value="l_link2"/>
+  <xacro:property name="NAME_LINK_ARM_L_3" value="l_link3"/>
+  <xacro:property name="NAME_LINK_ARM_L_4" value="l_link4"/>
+  <xacro:property name="NAME_LINK_ARM_L_5" value="l_link5"/>
+  <xacro:property name="NAME_LINK_ARM_L_6" value="l_link6"/>
+  <xacro:property name="NAME_LINK_ARM_L_7" value="l_link7"/>
+  <xacro:property name="NAME_LINK_HAND_L_A" value="l_handA_link"/>
+  <xacro:property name="NAME_LINK_HAND_L_B" value="l_handB_link"/>
+  <xacro:property name="NAME_LINK_ARMARKER_L" value="l_link5_armarker"/>
+  <xacro:property name="NAME_JOINT_BODY" value="waist_yaw_joint"/>
+  <xacro:property name="NAME_JOINT_BASE" value="base_link_to_world_joint"/>
+  <xacro:property name="NAME_JOINT_NECK_1" value="neck_yaw_joint"/>
+  <xacro:property name="NAME_JOINT_NECK_2" value="neck_pitch_joint"/>
+  <xacro:property name="NAME_JOINT_CAMERA" value="head_camera_joint"/>
+  <xacro:property name="NAME_JOINT_CHEST_CAMERA" value="chest_camera_joint"/>
+  <xacro:property name="NAME_JOINT_ARM_R_1" value="r_arm_joint1"/>
+  <xacro:property name="NAME_JOINT_ARM_R_2" value="r_arm_joint2"/>
+  <xacro:property name="NAME_JOINT_ARM_R_3" value="r_arm_joint3"/>
+  <xacro:property name="NAME_JOINT_ARM_R_4" value="r_arm_joint4"/>
+  <xacro:property name="NAME_JOINT_ARM_R_5" value="r_arm_joint5"/>
+  <xacro:property name="NAME_JOINT_ARM_R_6" value="r_arm_joint6"/>
+  <xacro:property name="NAME_JOINT_ARM_R_7" value="r_arm_joint7"/>
+  <xacro:property name="NAME_JOINT_HAND_R_A" value="r_hand_joint"/>
+  <xacro:property name="NAME_JOINT_HAND_R_B" value="r_hand_mimic_joint"/>
+  <xacro:property name="NAME_JOINT_ARMARKER_R" value="r_arm_armarker"/>
+  <xacro:property name="NAME_JOINT_ARM_L_1" value="l_arm_joint1"/>
+  <xacro:property name="NAME_JOINT_ARM_L_2" value="l_arm_joint2"/>
+  <xacro:property name="NAME_JOINT_ARM_L_3" value="l_arm_joint3"/>
+  <xacro:property name="NAME_JOINT_ARM_L_4" value="l_arm_joint4"/>
+  <xacro:property name="NAME_JOINT_ARM_L_5" value="l_arm_joint5"/>
+  <xacro:property name="NAME_JOINT_ARM_L_6" value="l_arm_joint6"/>
+  <xacro:property name="NAME_JOINT_ARM_L_7" value="l_arm_joint7"/>
+  <xacro:property name="NAME_JOINT_HAND_L_A" value="l_hand_joint"/>
+  <xacro:property name="NAME_JOINT_HAND_L_B" value="l_hand_mimic_joint"/>
+  <xacro:property name="NAME_JOINT_ARMARKER_L" value="l_arm_armarker"/>
   <xacro:property name="EFFORT_LIMIT" value="4.0"/>
   <xacro:property name="VELOCITY_LIMIT" value="5.969211435"/>
@@ -59,7 +111,7 @@
   <!-- Used for fixing robot 'base_link'  to Gazebo 'world' -->
   <link name="world"/>
-  <joint name="base_link_to_world_joint" type="fixed">
+  <joint name="${NAME_JOINT_BASE}" type="fixed">
     <parent link="world"/>
-    <child link="base_link"/>
+    <child link="${NAME_LINK_BASE}"/>
   </joint>
   <xacro:sciurus17_body

File: urdf/sciurus17_body.xacro (robot description, xacro)
@@ -10,5 +10,5 @@
             camera_color
     ">
-    <link name="base_link">
+    <link name="${NAME_LINK_BASE}">
       <visual>
         <geometry>
@@ -29,7 +29,7 @@
       </inertial>
     </link>
-    <joint name="waist_yaw_joint" type="revolute">
-      <parent link="base_link" />
-      <child link="body_link" />
+    <joint name="${NAME_JOINT_BODY}" type="revolute">
+      <parent link="${NAME_LINK_BASE}" />
+      <child link="${NAME_LINK_BODY}" />
       <origin xyz="0.0 0.0 0.1315" rpy="0 0 0"/>
       <limit
@@ -41,5 +41,5 @@
       <dynamics damping="1.0e-6" friction="0.8"/>
     </joint>
-    <link name="body_link">
+    <link name="${NAME_LINK_BODY}">
       <visual>
         <geometry>
@@ -60,10 +60,10 @@
       </inertial>
     </link>
-    <joint name="chest_camera_joint" type="fixed">
-      <parent link="body_link" />
-      <child link="chest_camera_link" />
+    <joint name="${NAME_JOINT_CHEST_CAMERA}" type="fixed">
+      <parent link="${NAME_LINK_BODY}" />
+      <child link="${NAME_LINK_CHEST_CAMERA}" />
       <origin xyz="0.114576 0.0 0.217659" rpy="-2.7925268032 0 -1.5707963268"/>
     </joint>
-    <link name="chest_camera_link">
+    <link name="${NAME_LINK_CHEST_CAMERA}">
       <visual>
         <origin xyz="0 0 0" rpy="0 0 0"/>
@@ -80,11 +80,11 @@
       </collision>
     </link>
-    <gazebo reference="base_link">
+    <gazebo reference="${NAME_LINK_BASE}">
       <material>Gazebo/White</material>
     </gazebo>
-    <gazebo reference="body_link">
+    <gazebo reference="${NAME_LINK_BODY}">
       <material>Gazebo/White</material>
     </gazebo>
-    <gazebo reference="chest_camera_link">
+    <gazebo reference="${NAME_LINK_CHEST_CAMERA}">
       <material>Gazebo/Black</material>
     </gazebo>

File: urdf/sciurus17_head.xacro (robot description, xacro)
@@ -11,7 +11,7 @@
             camera_color
             ">
-    <joint name="neck_yaw_joint" type="revolute">
-      <parent link="body_link" />
-      <child link="neck_yaw_link" />
+    <joint name="${NAME_JOINT_NECK_1}" type="revolute">
+      <parent link="${NAME_LINK_BODY}" />
+      <child link="${NAME_LINK_NECK_1}" />
       <origin xyz="0.08083 0.0 0.3395" rpy="0 0 0"/>
       <limit
@@ -23,5 +23,5 @@
       <dynamics damping="1.0e-6" friction="0.8"/>
     </joint>
-    <link name="neck_yaw_link">
+    <link name="${NAME_LINK_NECK_1}">
       <visual>
         <geometry>
@@ -41,7 +41,7 @@
       </inertial>
     </link>
-    <joint name="neck_pitch_joint" type="revolute">
-      <parent link="neck_yaw_link" />
-      <child link="neck_pitch_link" />
+    <joint name="${NAME_JOINT_NECK_2}" type="revolute">
+      <parent link="${NAME_LINK_NECK_1}" />
+      <child link="${NAME_LINK_NECK_2}" />
       <origin xyz="0.0 0.0 0.054" rpy="0 0 0"/>
       <limit
@@ -53,5 +53,5 @@
       <dynamics damping="1.0e-6" friction="0.8"/>
     </joint>
-    <link name="neck_pitch_link">
+    <link name="${NAME_LINK_NECK_2}">
       <visual>
         <origin rpy="1.5708 0 0" xyz="0.0 0.0 0.0"/>
@@ -73,10 +73,10 @@
       </inertial>
     </link>
-    <joint name="head_camera_joint" type="fixed">
-      <parent link="neck_pitch_link" />
-      <child link="camera_link" />
+    <joint name="${NAME_JOINT_CAMERA}" type="fixed">
+      <parent link="${NAME_LINK_NECK_2}" />
+      <child link="${NAME_LINK_CAMERA}" />
       <origin xyz="0.081785 0.020 0.091" rpy="0 0 0"/>
     </joint>
-    <link name="camera_link">
+    <link name="${NAME_LINK_CAMERA}">
       <visual>
         <origin xyz="0 0 0" rpy="0 0 0"/>
@@ -93,11 +93,11 @@
       </collision>
     </link>
-    <gazebo reference="neck_yaw_link">
+    <gazebo reference="${NAME_LINK_NECK_1}">
       <material>Gazebo/White</material>
     </gazebo>
-    <gazebo reference="neck_pitch_link">
+    <gazebo reference="${NAME_LINK_NECK_2}">
       <material>Gazebo/White</material>
     </gazebo>
-    <gazebo reference="camera_link">
+    <gazebo reference="${NAME_LINK_CAMERA}">
       <material>Gazebo/Black</material>
     </gazebo>

File: urdf/sciurus17_left_arm.xacro (robot description, xacro)
@@ -20,7 +20,7 @@
             arm_color
             ">
-    <joint name="l_arm_joint1" type="revolute">
-      <parent link="body_link" />
-      <child link="l_link1" />
+    <joint name="${NAME_JOINT_ARM_L_1}" type="revolute">
+      <parent link="${NAME_LINK_BODY}" />
+      <child link="${NAME_LINK_ARM_L_1}" />
       <origin xyz="0.08083 0.0965 0.2885" rpy="0 0 0"/>
       <limit
@@ -32,5 +32,5 @@
       <dynamics damping="1.0e-6" friction="0.8"/>
     </joint>
-    <link name="l_link1">
+    <link name="${NAME_LINK_ARM_L_1}">
       <visual>
         <origin rpy="-1.5708 0 0" xyz="0.0 0.0 0.0"/>
@@ -52,7 +52,7 @@
       </inertial>
     </link>
-    <joint name="l_arm_joint2" type="revolute">
-      <parent link="l_link1" />
-      <child link="l_link2" />
+    <joint name="${NAME_JOINT_ARM_L_2}" type="revolute">
+      <parent link="${NAME_LINK_ARM_L_1}" />
+      <child link="${NAME_LINK_ARM_L_2}" />
       <origin xyz="0.0 0.064 0.0" rpy="0 0 0"/>
       <limit
@@ -64,5 +64,5 @@
       <dynamics damping="1.0e-6" friction="0.8"/>
     </joint>
-    <link name="l_link2">
+    <link name="${NAME_LINK_ARM_L_2}">
       <visual>
         <origin rpy="0 -1.5708 0" xyz="0.0 0.0 0.0"/>
@@ -84,7 +84,7 @@
       </inertial>
     </link>
-    <joint name="l_arm_joint3" type="revolute">
-      <parent link="l_link2" />
-      <child link="l_link3" />
+    <joint name="${NAME_JOINT_ARM_L_3}" type="revolute">
+      <parent link="${NAME_LINK_ARM_L_2}" />
+      <child link="${NAME_LINK_ARM_L_3}" />
       <origin xyz="0.0 0.065 0.0" rpy="0 0 0"/>
       <limit
@@ -96,5 +96,5 @@
       <dynamics damping="1.0e-6" friction="0.8"/>
     </joint>
-    <link name="l_link3">
+    <link name="${NAME_LINK_ARM_L_3}">
       <visual>
         <origin rpy="-1.5708 0 0" xyz="0.0 0.0 0.0"/>
@@ -116,7 +116,7 @@
       </inertial>
     </link>
-    <joint name="l_arm_joint4" type="revolute">
-      <parent link="l_link3" />
-      <child link="l_link4" />
+    <joint name="${NAME_JOINT_ARM_L_4}" type="revolute">
+      <parent link="${NAME_LINK_ARM_L_3}" />
+      <child link="${NAME_LINK_ARM_L_4}" />
       <origin xyz="0.0 0.185 0.0" rpy="0 0 0"/>
       <limit
@@ -128,5 +128,5 @@
       <dynamics damping="1.0e-6" friction="0.8"/>
     </joint>
-    <link name="l_link4">
+    <link name="${NAME_LINK_ARM_L_4}">
       <visual>
         <origin rpy="0 0 0" xyz="0.0 0.0 0.0"/>
@@ -148,7 +148,7 @@
       </inertial>
     </link>
-    <joint name="l_arm_joint5" type="revolute">
-      <parent link="l_link4" />
-      <child link="l_link5" />
+    <joint name="${NAME_JOINT_ARM_L_5}" type="revolute">
+      <parent link="${NAME_LINK_ARM_L_4}" />
+      <child link="${NAME_LINK_ARM_L_5}" />
       <origin xyz="0.0 0.121 0.0" rpy="0 0 0"/>
       <limit
@@ -160,5 +160,5 @@
       <dynamics damping="1.0e-6" friction="0.8"/>
     </joint>
-    <link name="l_link5">
+    <link name="${NAME_LINK_ARM_L_5}">
       <visual>
         <origin rpy="-1.5708 0 0" xyz="0.0 0.0 0.0"/>
@@ -198,10 +198,10 @@
       </inertial>
     </link>
-    <joint name="l_arm_armarker" type="fixed">
-      <parent link="l_link5" />
-      <child link="l_link5_armarker" />
+    <joint name="${NAME_JOINT_ARMARKER_L}" type="fixed">
+      <parent link="${NAME_LINK_ARM_L_5}" />
+      <child link="${NAME_LINK_ARMARKER_L}" />
       <origin xyz="0.0467 0.093 0.0" rpy="0 0 0"/>
     </joint>
-    <link name="l_link5_armarker">
+    <link name="${NAME_LINK_ARMARKER_L}">
       <visual>
         <origin rpy="0 0 0" xyz="0.0 0.0 0.0"/>
@@ -218,7 +218,7 @@
       </collision>
     </link>
-    <joint name="l_arm_joint6" type="revolute">
-      <parent link="l_link5" />
-      <child link="l_link6" />
+    <joint name="${NAME_JOINT_ARM_L_6}" type="revolute">
+      <parent link="${NAME_LINK_ARM_L_5}" />
+      <child link="${NAME_LINK_ARM_L_6}" />
       <origin xyz="0.0 0.129 0.0" rpy="0 0 0"/>
       <limit
@@ -230,5 +230,5 @@
       <dynamics damping="1.0e-6" friction="0.8"/>
     </joint>
-    <link name="l_link6">
+    <link name="${NAME_LINK_ARM_L_6}">
       <visual>
         <origin rpy="0 0 0" xyz="0.0 0.0 0.0"/>
@@ -250,7 +250,7 @@
       </inertial>
     </link>
-    <joint name="l_arm_joint7" type="revolute">
-      <parent link="l_link6" />
-      <child link="l_link7" />
+    <joint name="${NAME_JOINT_ARM_L_7}" type="revolute">
+      <parent link="${NAME_LINK_ARM_L_6}" />
+      <child link="${NAME_LINK_ARM_L_7}" />
       <origin xyz="0.0 0.0191 0.0" rpy="0 0 0"/>
       <limit
@@ -262,20 +262,20 @@
       <dynamics damping="1.0e-6" friction="0.8"/>
     </joint>
-    <gazebo reference="l_link1">
-      <material>Gazebo/White</material>
-    </gazebo>
-    <gazebo reference="l_link2">
-      <material>Gazebo/White</material>
-    </gazebo>
-    <gazebo reference="l_link3">
-      <material>Gazebo/White</material>
-    </gazebo>
-    <gazebo reference="l_link4">
-      <material>Gazebo/White</material>
-    </gazebo>
-    <gazebo reference="l_link5">
-      <material>Gazebo/White</material>
-    </gazebo>
-    <gazebo reference="l_link6">
+    <gazebo reference="${NAME_LINK_ARM_L_1}">
+      <material>Gazebo/White</material>
+    </gazebo>
+    <gazebo reference="${NAME_LINK_ARM_L_2}">
+      <material>Gazebo/White</material>
+    </gazebo>
+    <gazebo reference="${NAME_LINK_ARM_L_3}">
+      <material>Gazebo/White</material>
+    </gazebo>
+    <gazebo reference="${NAME_LINK_ARM_L_4}">
+      <material>Gazebo/White</material>
+    </gazebo>
+    <gazebo reference="${NAME_LINK_ARM_L_5}">
+      <material>Gazebo/White</material>
+    </gazebo>
+    <gazebo reference="${NAME_LINK_ARM_L_6}">
       <material>Gazebo/White</material>
     </gazebo>

File: urdf/sciurus17_left_hand.xacro (robot description, xacro)
@@ -8,5 +8,5 @@
             hand_color
             ">
-    <link name="l_link7">
+    <link name="${NAME_LINK_ARM_L_7}">
       <visual>
         <origin rpy="1.5708 0 0" xyz="0.0 0.0 0.0"/>
@@ -28,7 +28,7 @@
       </inertial>
     </link>
-    <joint name="l_hand_joint" type="revolute">
-      <parent link="l_link7" />
-      <child link="l_handA_link" />
+    <joint name="${NAME_JOINT_HAND_L_A}" type="revolute">
+      <parent link="${NAME_LINK_ARM_L_7}" />
+      <child link="${NAME_LINK_HAND_L_A}" />
       <origin xyz="0.012 0.024 0.0" rpy="0 0 0"/>
       <limit
@@ -40,5 +40,5 @@
       <dynamics damping="1.0e-6" friction="0.8"/>
     </joint>
-    <link name="l_handA_link">
+    <link name="${NAME_LINK_HAND_L_A}">
       <visual>
         <origin rpy="0 0 0" xyz="0.0 0.0 0.0"/>
@@ -60,7 +60,7 @@
       </inertial>
     </link>
-    <joint name="l_hand_mimic_joint" type="revolute">
-      <parent link="l_link7" />
-      <child link="l_handB_link" />
+    <joint name="${NAME_JOINT_HAND_L_B}" type="revolute">
+      <parent link="${NAME_LINK_ARM_L_7}" />
+      <child link="${NAME_LINK_HAND_L_B}" />
       <origin xyz="-0.012 0.024 0.0" rpy="0 0 0"/>
       <limit
@@ -70,8 +70,8 @@
         velocity="${hand_joints_velocity_limit}"/>
       <axis xyz="0 0 -1"/>
-      <mimic joint="l_hand_joint" multiplier="1" offset="0"/>
+      <mimic joint="${NAME_JOINT_HAND_L_A}" multiplier="1" offset="0"/>
       <dynamics damping="1.0e-6" friction="0.8"/>
     </joint>
-    <link name="l_handB_link">
+    <link name="${NAME_LINK_HAND_L_B}">
       <visual>
         <origin rpy="0 0 0" xyz="0.0 0.0 0.0"/>
@@ -93,11 +93,11 @@
       </inertial>
     </link>
-    <gazebo reference="l_link7">
+    <gazebo reference="${NAME_LINK_ARM_L_7}">
       <material>Gazebo/Red</material>
     </gazebo>
-    <gazebo reference="l_handA_link">
+    <gazebo reference="${NAME_LINK_HAND_L_A}">
       <material>Gazebo/Red</material>
     </gazebo>
-    <gazebo reference="l_handB_link">
+    <gazebo reference="${NAME_LINK_HAND_L_B}">
       <material>Gazebo/Red</material>
     </gazebo>

File: urdf/sciurus17_right_arm.xacro (robot description, xacro)
@@ -20,7 +20,7 @@
             arm_color
             ">
-    <joint name="r_arm_joint1" type="revolute">
-      <parent link="body_link" />
-      <child link="r_link1" />
+    <joint name="${NAME_JOINT_ARM_R_1}" type="revolute">
+      <parent link="${NAME_LINK_BODY}" />
+      <child link="${NAME_LINK_ARM_R_1}" />
       <origin xyz="0.08083 -0.0965 0.2885" rpy="0 0 0"/>
       <limit
@@ -32,5 +32,5 @@
       <dynamics damping="1.0e-6" friction="0.8"/>
     </joint>
-    <link name="r_link1">
+    <link name="${NAME_LINK_ARM_R_1}">
       <visual>
         <origin rpy="1.5708 0 0" xyz="0.0 0.0 0.0"/>
@@ -52,7 +52,7 @@
       </inertial>
     </link>
-    <joint name="r_arm_joint2" type="revolute">
-      <parent link="r_link1" />
-      <child link="r_link2" />
+    <joint name="${NAME_JOINT_ARM_R_2}" type="revolute">
+      <parent link="${NAME_LINK_ARM_R_1}" />
+      <child link="${NAME_LINK_ARM_R_2}" />
       <origin xyz="0.0 -0.064 0.0" rpy="0 0 0"/>
       <limit
@@ -64,5 +64,5 @@
       <dynamics damping="1.0e-6" friction="0.8"/>
     </joint>
-    <link name="r_link2">
+    <link name="${NAME_LINK_ARM_R_2}">
       <visual>
         <origin rpy="0 1.5708 0" xyz="0.0 0.0 0.0"/>
@@ -84,7 +84,7 @@
       </inertial>
     </link>
-    <joint name="r_arm_joint3" type="revolute">
-      <parent link="r_link2" />
-      <child link="r_link3" />
+    <joint name="${NAME_JOINT_ARM_R_3}" type="revolute">
+      <parent link="${NAME_LINK_ARM_R_2}" />
+      <child link="${NAME_LINK_ARM_R_3}" />
       <origin xyz="0.0 -0.065 0.0" rpy="0 0 0"/>
       <limit
@@ -96,5 +96,5 @@
       <dynamics damping="1.0e-6" friction="0.8"/>
     </joint>
-    <link name="r_link3">
+    <link name="${NAME_LINK_ARM_R_3}">
       <visual>
         <origin rpy="1.5708 0 0" xyz="0.0 0.0 0.0"/>
@@ -116,7 +116,7 @@
       </inertial>
     </link>
-    <joint name="r_arm_joint4" type="revolute">
-      <parent link="r_link3" />
-      <child link="r_link4" />
+    <joint name="${NAME_JOINT_ARM_R_4}" type="revolute">
+      <parent link="${NAME_LINK_ARM_R_3}" />
+      <child link="${NAME_LINK_ARM_R_4}" />
       <origin xyz="0.0 -0.185 0.0" rpy="0 0 0"/>
       <limit
@@ -128,5 +128,5 @@
       <dynamics damping="1.0e-6" friction="0.8"/>
     </joint>
-    <link name="r_link4">
+    <link name="${NAME_LINK_ARM_R_4}">
       <visual>
         <origin rpy="0 0 0" xyz="0.0 0.0 0.0"/>
@@ -148,7 +148,7 @@
       </inertial>
     </link>
-    <joint name="r_arm_joint5" type="revolute">
-      <parent link="r_link4" />
-      <child link="r_link5" />
+    <joint name="${NAME_JOINT_ARM_R_5}" type="revolute">
+      <parent link="${NAME_LINK_ARM_R_4}" />
+      <child link="${NAME_LINK_ARM_R_5}" />
       <origin xyz="0.0 -0.121 0.0" rpy="0 0 0"/>
       <limit
@@ -160,5 +160,5 @@
       <dynamics damping="1.0e-6" friction="0.8"/>
     </joint>
-    <link name="r_link5">
+    <link name="${NAME_LINK_ARM_R_5}">
       <visual>
         <origin rpy="1.5708 0 0" xyz="0.0 0.0 0.0"/>
@@ -198,10 +198,10 @@
       </inertial>
     </link>
-    <joint name="r_arm_armarker" type="fixed">
-      <parent link="r_link5" />
-      <child link="r_link5_armarker" />
+    <joint name="${NAME_JOINT_ARMARKER_R}" type="fixed">
+      <parent link="${NAME_LINK_ARM_R_5}" />
+      <child link="${NAME_LINK_ARMARKER_R}" />
       <origin xyz="0.0467 -0.093 0.0" rpy="0 0 0"/>
     </joint>
-    <link name="r_link5_armarker">
+    <link name="${NAME_LINK_ARMARKER_R}">
       <visual>
         <origin rpy="0 0 0" xyz="0.0 0.0 0.0"/>
@@ -218,7 +218,7 @@
       </collision>
     </link>
-    <joint name="r_arm_joint6" type="revolute">
-      <parent link="r_link5" />
-      <child link="r_link6" />
+    <joint name="${NAME_JOINT_ARM_R_6}" type="revolute">
+      <parent link="${NAME_LINK_ARM_R_5}" />
+      <child link="${NAME_LINK_ARM_R_6}" />
       <origin xyz="0.0 -0.129 0.0" rpy="0 0 0"/>
       <limit
@@ -230,5 +230,5 @@
       <dynamics damping="1.0e-6" friction="0.8"/>
     </joint>
-    <link name="r_link6">
+    <link name="${NAME_LINK_ARM_R_6}">
       <visual>
         <origin rpy="0 0 0" xyz="0.0 0.0 0.0"/>
@@ -250,7 +250,7 @@
       </inertial>
     </link>
-    <joint name="r_arm_joint7" type="revolute">
-      <parent link="r_link6" />
-      <child link="r_link7" />
+    <joint name="${NAME_JOINT_ARM_R_7}" type="revolute">
+      <parent link="${NAME_LINK_ARM_R_6}" />
+      <child link="${NAME_LINK_ARM_R_7}" />
       <origin xyz="0.0 -0.0191 0.0" rpy="0 0 0"/>
       <limit
@@ -262,20 +262,20 @@
       <dynamics damping="1.0e-6" friction="0.8"/>
     </joint>
-    <gazebo reference="r_link1">
-      <material>Gazebo/White</material>
-    </gazebo>
-    <gazebo reference="r_link2">
-      <material>Gazebo/White</material>
-    </gazebo>
-    <gazebo reference="r_link3">
-      <material>Gazebo/White</material>
-    </gazebo>
-    <gazebo reference="r_link4">
-      <material>Gazebo/White</material>
-    </gazebo>
-    <gazebo reference="r_link5">
-      <material>Gazebo/White</material>
-    </gazebo>
-    <gazebo reference="r_link6">
+    <gazebo reference="${NAME_LINK_ARM_R_1}">
+      <material>Gazebo/White</material>
+    </gazebo>
+    <gazebo reference="${NAME_LINK_ARM_R_2}">
+      <material>Gazebo/White</material>
+    </gazebo>
+    <gazebo reference="${NAME_LINK_ARM_R_3}">
+      <material>Gazebo/White</material>
+    </gazebo>
+    <gazebo reference="${NAME_LINK_ARM_R_4}">
+      <material>Gazebo/White</material>
+    </gazebo>
+    <gazebo reference="${NAME_LINK_ARM_R_5}">
+      <material>Gazebo/White</material>
+    </gazebo>
+    <gazebo reference="${NAME_LINK_ARM_R_6}">
       <material>Gazebo/White</material>
     </gazebo>
