Commit message: link、joint名のproperty化

File: urdf/sciurus17_right_hand.xacro (robot description, xacro)
@@ -8,5 +8,5 @@
             hand_color
             ">
-    <link name="r_link7">
+    <link name="${NAME_LINK_ARM_R_7}">
       <visual>
         <origin rpy="1.5708 0 0" xyz="0.0 0.0 0.0"/>
@@ -28,7 +28,7 @@
       </inertial>
     </link>
-    <joint name="r_hand_joint" type="revolute">
-      <parent link="r_link7" />
-      <child link="r_handA_link" />
+    <joint name="${NAME_JOINT_HAND_R_A}" type="revolute">
+      <parent link="${NAME_LINK_ARM_R_7}" />
+      <child link="${NAME_LINK_HAND_R_A}" />
       <origin xyz="0.012 -0.024 0.0" rpy="0 0 0"/>
       <limit
@@ -40,5 +40,5 @@
       <dynamics damping="1.0e-6" friction="0.8"/>
     </joint>
-    <link name="r_handA_link">
+    <link name="${NAME_LINK_HAND_R_A}">
       <visual>
         <!--origin rpy="3.14159 0 0" xyz="0.0 0.0 0.0"/-->
@@ -61,7 +61,7 @@
       </inertial>
     </link>
-    <joint name="r_hand_mimic_joint" type="revolute">
-      <parent link="r_link7" />
-      <child link="r_handB_link" />
+    <joint name="${NAME_JOINT_HAND_R_B}" type="revolute">
+      <parent link="${NAME_LINK_ARM_R_7}" />
+      <child link="${NAME_LINK_HAND_R_B}" />
       <origin xyz="-0.012 -0.024 0.0" rpy="0 0 0"/>
       <limit
@@ -71,8 +71,8 @@
         velocity="${hand_joints_velocity_limit}"/>
       <axis xyz="0 0 -1"/>
-      <mimic joint="r_hand_joint" multiplier="1" offset="0"/>
+      <mimic joint="${NAME_JOINT_HAND_R_A}" multiplier="1" offset="0"/>
       <dynamics damping="1.0e-6" friction="0.8"/>
     </joint>
-    <link name="r_handB_link">
+    <link name="${NAME_LINK_HAND_R_B}">
       <visual>
         <!-- origin rpy="3.14159 0 0" xyz="0.0 0.0 0.0"/ -->
@@ -95,11 +95,11 @@
       </inertial>
     </link>
-    <gazebo reference="r_link7">
+    <gazebo reference="${NAME_LINK_ARM_R_7}">
       <material>Gazebo/Red</material>
     </gazebo>
-    <gazebo reference="r_handA_link">
+    <gazebo reference="${NAME_LINK_HAND_R_A}">
       <material>Gazebo/Red</material>
     </gazebo>
-    <gazebo reference="r_handB_link">
+    <gazebo reference="${NAME_LINK_HAND_R_B}">
       <material>Gazebo/Red</material>
     </gazebo>

Commit message: joint limitをpropertyで定義

File: urdf/sciurus17.urdf.xacro (robot description, xacro)
@@ -67,4 +67,42 @@
   <xacro:property name="EFFORT_LIMIT" value="4.0"/>
   <xacro:property name="VELOCITY_LIMIT" value="5.969211435"/>
+  <xacro:property name="NAME_JOINT_BODY_LOWER_LIMIT" value="${radians(-110)}"/>
+  <xacro:property name="NAME_JOINT_BODY_UPPER_LIMIT" value="${radians(110)}"/>
+  <xacro:property name="JOINT_NECK_1_LOWER_LIMIT" value="${radians(-165)}"/>
+  <xacro:property name="JOINT_NECK_1_UPPER_LIMIT" value="${radians(165)}"/>
+  <xacro:property name="JOINT_NECK_2_LOWER_LIMIT" value="${radians(-90)}"/>
+  <xacro:property name="JOINT_NECK_2_UPPER_LIMIT" value="${radians(55)}"/>
+  <xacro:property name="JOINT_ARM_R_1_LOWER_LIMIT" value="${radians(-90)}"/>
+  <xacro:property name="JOINT_ARM_R_1_UPPER_LIMIT" value="${radians(90)}"/>
+  <xacro:property name="JOINT_ARM_R_2_LOWER_LIMIT" value="${radians(-90)}"/>
+  <xacro:property name="JOINT_ARM_R_2_UPPER_LIMIT" value="${radians(0)}"/>
+  <xacro:property name="JOINT_ARM_R_3_LOWER_LIMIT" value="${radians(-90)}"/>
+  <xacro:property name="JOINT_ARM_R_3_UPPER_LIMIT" value="${radians(90)}"/>
+  <xacro:property name="JOINT_ARM_R_4_LOWER_LIMIT" value="${radians(0)}"/>
+  <xacro:property name="JOINT_ARM_R_4_UPPER_LIMIT" value="${radians(157)}"/>
+  <xacro:property name="JOINT_ARM_R_5_LOWER_LIMIT" value="${radians(-90)}"/>
+  <xacro:property name="JOINT_ARM_R_5_UPPER_LIMIT" value="${radians(90)}"/>
+  <xacro:property name="JOINT_ARM_R_6_LOWER_LIMIT" value="${radians(-120)}"/>
+  <xacro:property name="JOINT_ARM_R_6_UPPER_LIMIT" value="${radians(60)}"/>
+  <xacro:property name="JOINT_ARM_R_7_LOWER_LIMIT" value="${radians(-170)}"/>
+  <xacro:property name="JOINT_ARM_R_7_UPPER_LIMIT" value="${radians(170)}"/>
+  <xacro:property name="JOINT_HAND_R_LOWER_LIMIT" value="${radians(0)}"/>
+  <xacro:property name="JOINT_HAND_R_UPPER_LIMIT" value="${radians(86)}"/>
+  <xacro:property name="JOINT_ARM_L_1_LOWER_LIMIT" value="${radians(-90)}"/>
+  <xacro:property name="JOINT_ARM_L_1_UPPER_LIMIT" value="${radians(90)}"/>
+  <xacro:property name="JOINT_ARM_L_2_LOWER_LIMIT" value="${radians(0)}"/>
+  <xacro:property name="JOINT_ARM_L_2_UPPER_LIMIT" value="${radians(90)}"/>
+  <xacro:property name="JOINT_ARM_L_3_LOWER_LIMIT" value="${radians(-90)}"/>
+  <xacro:property name="JOINT_ARM_L_3_UPPER_LIMIT" value="${radians(90)}"/>
+  <xacro:property name="JOINT_ARM_L_4_LOWER_LIMIT" value="${radians(-157)}"/>
+  <xacro:property name="JOINT_ARM_L_4_UPPER_LIMIT" value="${radians(0)}"/>
+  <xacro:property name="JOINT_ARM_L_5_LOWER_LIMIT" value="${radians(-90)}"/>
+  <xacro:property name="JOINT_ARM_L_5_UPPER_LIMIT" value="${radians(90)}"/>
+  <xacro:property name="JOINT_ARM_L_6_LOWER_LIMIT" value="${radians(-60)}"/>
+  <xacro:property name="JOINT_ARM_L_6_UPPER_LIMIT" value="${radians(120)}"/>
+  <xacro:property name="JOINT_ARM_L_7_LOWER_LIMIT" value="${radians(-170)}"/>
+  <xacro:property name="JOINT_ARM_L_7_UPPER_LIMIT" value="${radians(170)}"/>
+  <xacro:property name="JOINT_HAND_L_LOWER_LIMIT" value="${radians(-86)}"/>
+  <xacro:property name="JOINT_HAND_L_UPPER_LIMIT" value="${radians(0)}"/>
   <xacro:arg name="use_gazebo_simulation" default="false" />
   <xacro:arg name="load_trans1" default="false" />
@@ -116,6 +154,6 @@
   </joint>
   <xacro:sciurus17_body
-    waist_yaw_upper_limit="${radians(-110)}"
-    waist_yaw_lower_limit="${radians(110)}"
+    waist_yaw_upper_limit="${NAME_JOINT_BODY_LOWER_LIMIT}"
+    waist_yaw_lower_limit="${NAME_JOINT_BODY_UPPER_LIMIT}"
     waist_yaw_effort_limit="${EFFORT_LIMIT}"
     waist_yaw_velocity_limit="${VELOCITY_LIMIT}"
@@ -125,8 +163,8 @@
   </xacro:sciurus17_body>
   <xacro:sciurus17_head
-    neck_yaw_lower_limit="${radians(-165)}"
-    neck_yaw_upper_limit="${radians(165)}"
-    neck_pitch_lower_limit="${radians(-90)}"
-    neck_pitch_upper_limit="${radians(55)}"
+    neck_yaw_lower_limit="${JOINT_NECK_1_LOWER_LIMIT}"
+    neck_yaw_upper_limit="${JOINT_NECK_1_UPPER_LIMIT}"
+    neck_pitch_lower_limit="${JOINT_NECK_2_LOWER_LIMIT}"
+    neck_pitch_upper_limit="${JOINT_NECK_2_UPPER_LIMIT}"
     neck_joints_effort_limit="${EFFORT_LIMIT}"
     neck_joints_velocity_limit="${VELOCITY_LIMIT}"
@@ -135,18 +173,18 @@
   </xacro:sciurus17_head>
   <xacro:sciurus17_right_arm
-    arm_joint1_lower_limit="${radians(-90)}"
-    arm_joint1_upper_limit="${radians(90)}"
-    arm_joint2_lower_limit="${radians(-90)}"
-    arm_joint2_upper_limit="${radians(0)}"
-    arm_joint3_lower_limit="${radians(-90)}"
-    arm_joint3_upper_limit="${radians(90)}"
-    arm_joint4_lower_limit="${radians(0)}"
-    arm_joint4_upper_limit="${radians(157)}"
-    arm_joint5_lower_limit="${radians(-90)}"
-    arm_joint5_upper_limit="${radians(90)}"
-    arm_joint6_lower_limit="${radians(-120)}"
-    arm_joint6_upper_limit="${radians(60)}"
-    arm_joint7_lower_limit="${radians(-170)}"
-    arm_joint7_upper_limit="${radians(170)}"
+    arm_joint1_lower_limit="${JOINT_ARM_R_1_LOWER_LIMIT}"
+    arm_joint1_upper_limit="${JOINT_ARM_R_1_UPPER_LIMIT}"
+    arm_joint2_lower_limit="${JOINT_ARM_R_2_LOWER_LIMIT}"
+    arm_joint2_upper_limit="${JOINT_ARM_R_2_UPPER_LIMIT}"
+    arm_joint3_lower_limit="${JOINT_ARM_R_3_LOWER_LIMIT}"
+    arm_joint3_upper_limit="${JOINT_ARM_R_3_UPPER_LIMIT}"
+    arm_joint4_lower_limit="${JOINT_ARM_R_4_LOWER_LIMIT}"
+    arm_joint4_upper_limit="${JOINT_ARM_R_4_UPPER_LIMIT}"
+    arm_joint5_lower_limit="${JOINT_ARM_R_5_LOWER_LIMIT}"
+    arm_joint5_upper_limit="${JOINT_ARM_R_5_UPPER_LIMIT}"
+    arm_joint6_lower_limit="${JOINT_ARM_R_6_LOWER_LIMIT}"
+    arm_joint6_upper_limit="${JOINT_ARM_R_6_UPPER_LIMIT}"
+    arm_joint7_lower_limit="${JOINT_ARM_R_7_LOWER_LIMIT}"
+    arm_joint7_upper_limit="${JOINT_ARM_R_7_UPPER_LIMIT}"
     arm_joints_effort_limit="${EFFORT_LIMIT}"
     arm_joints_velocity_limit="${VELOCITY_LIMIT}"
@@ -154,6 +192,6 @@
   </xacro:sciurus17_right_arm>
   <xacro:sciurus17_right_hand
-    hand_joints_lower_limit="${radians(0)}"
-    hand_joints_upper_limit="${radians(86)}"
+    hand_joints_lower_limit="${JOINT_HAND_R_LOWER_LIMIT}"
+    hand_joints_upper_limit="${JOINT_HAND_R_UPPER_LIMIT}"
     hand_joints_effort_limit="${EFFORT_LIMIT}"
     hand_joints_velocity_limit="${VELOCITY_LIMIT}"
@@ -161,18 +199,18 @@
   </xacro:sciurus17_right_hand>
   <xacro:sciurus17_left_arm
-    arm_joint1_lower_limit="${radians(-90)}"
-    arm_joint1_upper_limit="${radians(90)}"
-    arm_joint2_lower_limit="${radians(0)}"
-    arm_joint2_upper_limit="${radians(90)}"
-    arm_joint3_lower_limit="${radians(-90)}"
-    arm_joint3_upper_limit="${radians(90)}"
-    arm_joint4_lower_limit="${radians(-157)}"
-    arm_joint4_upper_limit="${radians(0)}"
-    arm_joint5_lower_limit="${radians(-90)}"
-    arm_joint5_upper_limit="${radians(90)}"
-    arm_joint6_lower_limit="${radians(-60)}"
-    arm_joint6_upper_limit="${radians(120)}"
-    arm_joint7_lower_limit="${radians(-170)}"
-    arm_joint7_upper_limit="${radians(170)}"
+    arm_joint1_lower_limit="${JOINT_ARM_L_1_LOWER_LIMIT}"
+    arm_joint1_upper_limit="${JOINT_ARM_L_1_UPPER_LIMIT}"
+    arm_joint2_lower_limit="${JOINT_ARM_L_2_LOWER_LIMIT}"
+    arm_joint2_upper_limit="${JOINT_ARM_L_2_UPPER_LIMIT}"
+    arm_joint3_lower_limit="${JOINT_ARM_L_3_LOWER_LIMIT}"
+    arm_joint3_upper_limit="${JOINT_ARM_L_3_UPPER_LIMIT}"
+    arm_joint4_lower_limit="${JOINT_ARM_L_4_LOWER_LIMIT}"
+    arm_joint4_upper_limit="${JOINT_ARM_L_4_UPPER_LIMIT}"
+    arm_joint5_lower_limit="${JOINT_ARM_L_5_LOWER_LIMIT}"
+    arm_joint5_upper_limit="${JOINT_ARM_L_5_UPPER_LIMIT}"
+    arm_joint6_lower_limit="${JOINT_ARM_L_6_LOWER_LIMIT}"
+    arm_joint6_upper_limit="${JOINT_ARM_L_6_UPPER_LIMIT}"
+    arm_joint7_lower_limit="${JOINT_ARM_L_7_LOWER_LIMIT}"
+    arm_joint7_upper_limit="${JOINT_ARM_L_7_UPPER_LIMIT}"
     arm_joints_effort_limit="${EFFORT_LIMIT}"
     arm_joints_velocity_limit="${VELOCITY_LIMIT}"
@@ -180,6 +218,6 @@
   </xacro:sciurus17_left_arm>
   <xacro:sciurus17_left_hand
-    hand_joints_lower_limit="${radians(-86)}"
-    hand_joints_upper_limit="${radians(0)}"
+    hand_joints_lower_limit="${JOINT_HAND_L_LOWER_LIMIT}"
+    hand_joints_upper_limit="${JOINT_HAND_L_UPPER_LIMIT}"
     hand_joints_effort_limit="${EFFORT_LIMIT}"
     hand_joints_velocity_limit="${VELOCITY_LIMIT}"

Commit message: colorをpropertyで定義

File: urdf/sciurus17.urdf.xacro (robot description, xacro)
@@ -105,4 +105,10 @@
   <xacro:property name="JOINT_HAND_L_LOWER_LIMIT" value="${radians(-86)}"/>
   <xacro:property name="JOINT_HAND_L_UPPER_LIMIT" value="${radians(0)}"/>
+  <xacro:property name="COLOR_LINK_BASE" value="white"/>
+  <xacro:property name="COLOR_LINK_BODY" value="white"/>
+  <xacro:property name="COLOR_LINK_HEAD" value="white"/>
+  <xacro:property name="COLOR_LINK_ARM" value="white"/>
+  <xacro:property name="COLOR_LINK_HAND" value="red"/>
+  <xacro:property name="COLOR_LINK_CAMERA" value="white"/>
   <xacro:arg name="use_gazebo_simulation" default="false" />
   <xacro:arg name="load_trans1" default="false" />
@@ -158,7 +164,7 @@
     waist_yaw_effort_limit="${EFFORT_LIMIT}"
     waist_yaw_velocity_limit="${VELOCITY_LIMIT}"
-    base_color="white"
-    body_color="white"
-    camera_color="white">
+    base_color="${COLOR_LINK_BASE}"
+    body_color="${COLOR_LINK_BODY}"
+    camera_color="${COLOR_LINK_CAMERA}">
   </xacro:sciurus17_body>
   <xacro:sciurus17_head
@@ -169,6 +175,6 @@
     neck_joints_effort_limit="${EFFORT_LIMIT}"
     neck_joints_velocity_limit="${VELOCITY_LIMIT}"
-    head_color="white"
-    camera_color="white">
+    head_color="${COLOR_LINK_HEAD}"
+    camera_color="${COLOR_LINK_CAMERA}">
   </xacro:sciurus17_head>
   <xacro:sciurus17_right_arm
@@ -189,5 +195,5 @@
     arm_joints_effort_limit="${EFFORT_LIMIT}"
     arm_joints_velocity_limit="${VELOCITY_LIMIT}"
-    arm_color="white">
+    arm_color="${COLOR_LINK_ARM}">
   </xacro:sciurus17_right_arm>
   <xacro:sciurus17_right_hand
@@ -196,5 +202,5 @@
     hand_joints_effort_limit="${EFFORT_LIMIT}"
     hand_joints_velocity_limit="${VELOCITY_LIMIT}"
-    hand_color="red">
+    hand_color="${COLOR_LINK_HAND}">
   </xacro:sciurus17_right_hand>
   <xacro:sciurus17_left_arm
@@ -215,5 +221,5 @@
     arm_joints_effort_limit="${EFFORT_LIMIT}"
     arm_joints_velocity_limit="${VELOCITY_LIMIT}"
-    arm_color="white">
+    arm_color="${COLOR_LINK_ARM}">
   </xacro:sciurus17_left_arm>
   <xacro:sciurus17_left_hand
@@ -222,5 +228,5 @@
     hand_joints_effort_limit="${EFFORT_LIMIT}"
     hand_joints_velocity_limit="${VELOCITY_LIMIT}"
-    hand_color="red">
+    hand_color="${COLOR_LINK_HAND}">
   </xacro:sciurus17_left_hand>
 </robot>
