Commit message: macroの引数によるパラメータ設定を削除

File: urdf/sciurus17.urdf.xacro (robot description, xacro)
@@ -159,74 +159,9 @@
     <child link="${NAME_LINK_BASE}"/>
   </joint>
-  <xacro:sciurus17_body
-    waist_yaw_upper_limit="${NAME_JOINT_BODY_LOWER_LIMIT}"
-    waist_yaw_lower_limit="${NAME_JOINT_BODY_UPPER_LIMIT}"
-    waist_yaw_effort_limit="${EFFORT_LIMIT}"
-    waist_yaw_velocity_limit="${VELOCITY_LIMIT}"
-    base_color="${COLOR_LINK_BASE}"
-    body_color="${COLOR_LINK_BODY}"
-    camera_color="${COLOR_LINK_CAMERA}">
-  </xacro:sciurus17_body>
-  <xacro:sciurus17_head
-    neck_yaw_lower_limit="${JOINT_NECK_1_LOWER_LIMIT}"
-    neck_yaw_upper_limit="${JOINT_NECK_1_UPPER_LIMIT}"
-    neck_pitch_lower_limit="${JOINT_NECK_2_LOWER_LIMIT}"
-    neck_pitch_upper_limit="${JOINT_NECK_2_UPPER_LIMIT}"
-    neck_joints_effort_limit="${EFFORT_LIMIT}"
-    neck_joints_velocity_limit="${VELOCITY_LIMIT}"
-    head_color="${COLOR_LINK_HEAD}"
-    camera_color="${COLOR_LINK_CAMERA}">
-  </xacro:sciurus17_head>
-  <xacro:sciurus17_right_arm
-    arm_joint1_lower_limit="${JOINT_ARM_R_1_LOWER_LIMIT}"
-    arm_joint1_upper_limit="${JOINT_ARM_R_1_UPPER_LIMIT}"
-    arm_joint2_lower_limit="${JOINT_ARM_R_2_LOWER_LIMIT}"
-    arm_joint2_upper_limit="${JOINT_ARM_R_2_UPPER_LIMIT}"
-    arm_joint3_lower_limit="${JOINT_ARM_R_3_LOWER_LIMIT}"
-    arm_joint3_upper_limit="${JOINT_ARM_R_3_UPPER_LIMIT}"
-    arm_joint4_lower_limit="${JOINT_ARM_R_4_LOWER_LIMIT}"
-    arm_joint4_upper_limit="${JOINT_ARM_R_4_UPPER_LIMIT}"
-    arm_joint5_lower_limit="${JOINT_ARM_R_5_LOWER_LIMIT}"
-    arm_joint5_upper_limit="${JOINT_ARM_R_5_UPPER_LIMIT}"
-    arm_joint6_lower_limit="${JOINT_ARM_R_6_LOWER_LIMIT}"
-    arm_joint6_upper_limit="${JOINT_ARM_R_6_UPPER_LIMIT}"
-    arm_joint7_lower_limit="${JOINT_ARM_R_7_LOWER_LIMIT}"
-    arm_joint7_upper_limit="${JOINT_ARM_R_7_UPPER_LIMIT}"
-    arm_joints_effort_limit="${EFFORT_LIMIT}"
-    arm_joints_velocity_limit="${VELOCITY_LIMIT}"
-    arm_color="${COLOR_LINK_ARM}">
-  </xacro:sciurus17_right_arm>
-  <xacro:sciurus17_right_hand
-    hand_joints_lower_limit="${JOINT_HAND_R_LOWER_LIMIT}"
-    hand_joints_upper_limit="${JOINT_HAND_R_UPPER_LIMIT}"
-    hand_joints_effort_limit="${EFFORT_LIMIT}"
-    hand_joints_velocity_limit="${VELOCITY_LIMIT}"
-    hand_color="${COLOR_LINK_HAND}">
-  </xacro:sciurus17_right_hand>
-  <xacro:sciurus17_left_arm
-    arm_joint1_lower_limit="${JOINT_ARM_L_1_LOWER_LIMIT}"
-    arm_joint1_upper_limit="${JOINT_ARM_L_1_UPPER_LIMIT}"
-    arm_joint2_lower_limit="${JOINT_ARM_L_2_LOWER_LIMIT}"
-    arm_joint2_upper_limit="${JOINT_ARM_L_2_UPPER_LIMIT}"
-    arm_joint3_lower_limit="${JOINT_ARM_L_3_LOWER_LIMIT}"
-    arm_joint3_upper_limit="${JOINT_ARM_L_3_UPPER_LIMIT}"
-    arm_joint4_lower_limit="${JOINT_ARM_L_4_LOWER_LIMIT}"
-    arm_joint4_upper_limit="${JOINT_ARM_L_4_UPPER_LIMIT}"
-    arm_joint5_lower_limit="${JOINT_ARM_L_5_LOWER_LIMIT}"
-    arm_joint5_upper_limit="${JOINT_ARM_L_5_UPPER_LIMIT}"
-    arm_joint6_lower_limit="${JOINT_ARM_L_6_LOWER_LIMIT}"
-    arm_joint6_upper_limit="${JOINT_ARM_L_6_UPPER_LIMIT}"
-    arm_joint7_lower_limit="${JOINT_ARM_L_7_LOWER_LIMIT}"
-    arm_joint7_upper_limit="${JOINT_ARM_L_7_UPPER_LIMIT}"
-    arm_joints_effort_limit="${EFFORT_LIMIT}"
-    arm_joints_velocity_limit="${VELOCITY_LIMIT}"
-    arm_color="${COLOR_LINK_ARM}">
-  </xacro:sciurus17_left_arm>
-  <xacro:sciurus17_left_hand
-    hand_joints_lower_limit="${JOINT_HAND_L_LOWER_LIMIT}"
-    hand_joints_upper_limit="${JOINT_HAND_L_UPPER_LIMIT}"
-    hand_joints_effort_limit="${EFFORT_LIMIT}"
-    hand_joints_velocity_limit="${VELOCITY_LIMIT}"
-    hand_color="${COLOR_LINK_HAND}">
-  </xacro:sciurus17_left_hand>
+  <xacro:sciurus17_body/>
+  <xacro:sciurus17_head/>
+  <xacro:sciurus17_right_arm/>
+  <xacro:sciurus17_right_hand/>
+  <xacro:sciurus17_left_arm/>
+  <xacro:sciurus17_left_hand/>
 </robot>

File: urdf/sciurus17_body.xacro (robot description, xacro)
@@ -1,13 +1,5 @@
 <?xml version="1.0"?>
 <robot xmlns:xacro="http://ros.org/wiki/xacro">
-  <xacro:macro name="sciurus17_body"
-    params="waist_yaw_upper_limit
-            waist_yaw_lower_limit
-            waist_yaw_effort_limit
-            waist_yaw_velocity_limit
-            base_color
-            body_color
-            camera_color
-    ">
+  <xacro:macro name="sciurus17_body">
     <link name="${NAME_LINK_BASE}">
       <visual>
@@ -15,5 +7,5 @@
           <mesh filename="package://sciurus17_description/meshes/visual/Base.stl" scale="1.0 1.0 1.0"/>
         </geometry>
-        <material name="${base_color}"/>
+        <material name="${COLOR_LINK_BASE}"/>
       </visual>
       <collision>
@@ -34,8 +26,8 @@
       <origin xyz="0.0 0.0 0.1315" rpy="0 0 0"/>
       <limit
-        lower="${waist_yaw_upper_limit}"
-        upper="${waist_yaw_lower_limit}"
-        effort="${waist_yaw_effort_limit}"
-        velocity="${waist_yaw_velocity_limit}"/>
+        lower="${NAME_JOINT_BODY_LOWER_LIMIT}"
+        upper="${NAME_JOINT_BODY_UPPER_LIMIT}"
+        effort="${EFFORT_LIMIT}"
+        velocity="${VELOCITY_LIMIT}"/>
       <axis xyz="0 0 1"/>
       <dynamics damping="1.0e-6" friction="0.8"/>
@@ -46,5 +38,5 @@
           <mesh filename="package://sciurus17_description/meshes/visual/Body.stl" scale="1.0 1.0 1.0"/>
         </geometry>
-        <material name="${body_color}"/>
+        <material name="${COLOR_LINK_BODY}"/>
       </visual>
       <collision>
@@ -71,5 +63,5 @@
           <cylinder length="0.002" radius="0.003"/>
         </geometry>
-        <material name="${camera_color}"/>
+        <material name="${COLOR_LINK_CAMERA}"/>
       </visual>
       <collision>

File: urdf/sciurus17_head.xacro (robot description, xacro)
@@ -1,14 +1,5 @@
 <?xml version="1.0"?>
 <robot xmlns:xacro="http://ros.org/wiki/xacro">
-  <xacro:macro name="sciurus17_head"
-    params="neck_yaw_lower_limit
-            neck_yaw_upper_limit
-            neck_pitch_lower_limit
-            neck_pitch_upper_limit
-            neck_joints_effort_limit
-            neck_joints_velocity_limit
-            head_color
-            camera_color
-            ">
+  <xacro:macro name="sciurus17_head">
     <joint name="${NAME_JOINT_NECK_1}" type="revolute">
       <parent link="${NAME_LINK_BODY}" />
@@ -16,8 +7,8 @@
       <origin xyz="0.08083 0.0 0.3395" rpy="0 0 0"/>
       <limit
-        lower="${neck_yaw_lower_limit}"
-        upper="${neck_yaw_upper_limit}"
-        effort="${neck_joints_effort_limit}"
-        velocity="${neck_joints_velocity_limit}"/>
+        lower="${JOINT_NECK_1_LOWER_LIMIT}"
+        upper="${JOINT_NECK_1_UPPER_LIMIT}"
+        effort="${EFFORT_LIMIT}"
+        velocity="${VELOCITY_LIMIT}"/>
       <axis xyz="0 0 1"/>
       <dynamics damping="1.0e-6" friction="0.8"/>
@@ -28,5 +19,5 @@
           <mesh filename="package://sciurus17_description/meshes/visual/Neck1.stl" scale="1.0 1.0 1.0"/>
         </geometry>
-        <material name="${head_color}"/>
+        <material name="${COLOR_LINK_HEAD}"/>
       </visual>
       <collision>
@@ -46,8 +37,8 @@
       <origin xyz="0.0 0.0 0.054" rpy="0 0 0"/>
       <limit
-        lower="${neck_pitch_lower_limit}"
-        upper="${neck_pitch_upper_limit}"
-        effort="${neck_joints_effort_limit}"
-        velocity="${neck_joints_velocity_limit}"/>
+        lower="${JOINT_NECK_2_LOWER_LIMIT}"
+        upper="${JOINT_NECK_2_UPPER_LIMIT}"
+        effort="${EFFORT_LIMIT}"
+        velocity="${VELOCITY_LIMIT}"/>
       <axis xyz="0 -1 0"/>
       <dynamics damping="1.0e-6" friction="0.8"/>
@@ -59,5 +50,5 @@
           <mesh filename="package://sciurus17_description/meshes/visual/Neck2.stl" scale="1.0 1.0 1.0"/>
         </geometry>
-        <material name="${head_color}"/>
+        <material name="${COLOR_LINK_HEAD}"/>
       </visual>
       <collision>
@@ -84,5 +75,5 @@
           <cylinder length="0.002" radius="0.003"/>
         </geometry>
-        <material name="${camera_color}"/>
+        <material name="${COLOR_LINK_CAMERA}"/>
       </visual>
       <collision>

File: urdf/sciurus17_left_arm.xacro (robot description, xacro)
@@ -1,23 +1,5 @@
 <?xml version="1.0"?>
 <robot xmlns:xacro="http://ros.org/wiki/xacro">
-  <xacro:macro name="sciurus17_left_arm"
-    params="arm_joint1_lower_limit
-            arm_joint1_upper_limit
-            arm_joint2_lower_limit
-            arm_joint2_upper_limit
-            arm_joint3_lower_limit
-            arm_joint3_upper_limit
-            arm_joint4_lower_limit
-            arm_joint4_upper_limit
-            arm_joint5_lower_limit
-            arm_joint5_upper_limit
-            arm_joint6_lower_limit
-            arm_joint6_upper_limit
-            arm_joint7_lower_limit
-            arm_joint7_upper_limit
-            arm_joints_effort_limit
-            arm_joints_velocity_limit
-            arm_color
-            ">
+  <xacro:macro name="sciurus17_left_arm">
     <joint name="${NAME_JOINT_ARM_L_1}" type="revolute">
       <parent link="${NAME_LINK_BODY}" />
@@ -25,8 +7,8 @@
       <origin xyz="0.08083 0.0965 0.2885" rpy="0 0 0"/>
       <limit
-        lower="${arm_joint1_lower_limit}"
-        upper="${arm_joint1_upper_limit}"
-        effort="${arm_joints_effort_limit}"
-        velocity="${arm_joints_velocity_limit}"/>
+        lower="${JOINT_ARM_L_1_LOWER_LIMIT}"
+        upper="${JOINT_ARM_L_1_UPPER_LIMIT}"
+        effort="${EFFORT_LIMIT}"
+        velocity="${VELOCITY_LIMIT}"/>
       <axis xyz="0 1 0"/>
       <dynamics damping="1.0e-6" friction="0.8"/>
@@ -38,5 +20,5 @@
           <mesh filename="package://sciurus17_description/meshes/visual/L_Link1.stl" scale="1.0 1.0 1.0"/>
         </geometry>
-        <material name="${arm_color}"/>
+        <material name="${COLOR_LINK_ARM}"/>
       </visual>
       <collision>
@@ -57,8 +39,8 @@
       <origin xyz="0.0 0.064 0.0" rpy="0 0 0"/>
       <limit
-        lower="${arm_joint2_lower_limit}"
-        upper="${arm_joint2_upper_limit}"
-        effort="${arm_joints_effort_limit}"
-        velocity="${arm_joints_velocity_limit}"/>
+        lower="${JOINT_ARM_L_2_LOWER_LIMIT}"
+        upper="${JOINT_ARM_L_2_UPPER_LIMIT}"
+        effort="${EFFORT_LIMIT}"
+        velocity="${VELOCITY_LIMIT}"/>
       <axis xyz="-1 0 0"/>
       <dynamics damping="1.0e-6" friction="0.8"/>
@@ -70,5 +52,5 @@
           <mesh filename="package://sciurus17_description/meshes/visual/L_Link2.stl" scale="-1.0 1.0 -1.0"/>
         </geometry>
-        <material name="${arm_color}"/>
+        <material name="${COLOR_LINK_ARM}"/>
       </visual>
       <collision>
@@ -89,8 +71,8 @@
       <origin xyz="0.0 0.065 0.0" rpy="0 0 0"/>
       <limit
-        lower="${arm_joint3_lower_limit}"
-        upper="${arm_joint3_upper_limit}"
-        effort="${arm_joints_effort_limit}"
-        velocity="${arm_joints_velocity_limit}"/>
+        lower="${JOINT_ARM_L_3_LOWER_LIMIT}"
+        upper="${JOINT_ARM_L_3_UPPER_LIMIT}"
+        effort="${EFFORT_LIMIT}"
+        velocity="${VELOCITY_LIMIT}"/>
       <axis xyz="0 1 0"/>
       <dynamics damping="1.0e-6" friction="0.8"/>
@@ -102,5 +84,5 @@
           <mesh filename="package://sciurus17_description/meshes/visual/L_Link3.stl" scale="1.0 1.0 1.0"/>
         </geometry>
-        <material name="${arm_color}"/>
+        <material name="${COLOR_LINK_ARM}"/>
       </visual>
       <collision>
@@ -121,8 +103,8 @@
       <origin xyz="0.0 0.185 0.0" rpy="0 0 0"/>
       <limit
-        lower="${arm_joint4_lower_limit}"
-        upper="${arm_joint4_upper_limit}"
-        effort="${arm_joints_effort_limit}"
-        velocity="${arm_joints_velocity_limit}"/>
+        lower="${JOINT_ARM_L_4_LOWER_LIMIT}"
+        upper="${JOINT_ARM_L_4_UPPER_LIMIT}"
+        effort="${EFFORT_LIMIT}"
+        velocity="${VELOCITY_LIMIT}"/>
       <axis xyz="0 0 1"/>
       <dynamics damping="1.0e-6" friction="0.8"/>
@@ -134,5 +116,5 @@
           <mesh filename="package://sciurus17_description/meshes/visual/L_Link4.stl" scale="1.0 1.0 1.0"/>
         </geometry>
-        <material name="${arm_color}"/>
+        <material name="${COLOR_LINK_ARM}"/>
       </visual>
       <collision>
@@ -153,8 +135,8 @@
       <origin xyz="0.0 0.121 0.0" rpy="0 0 0"/>
       <limit
-        lower="${arm_joint5_lower_limit}"
-        upper="${arm_joint5_upper_limit}"
-        effort="${arm_joints_effort_limit}"
-        velocity="${arm_joints_velocity_limit}"/>
+        lower="${JOINT_ARM_L_5_LOWER_LIMIT}"
+        upper="${JOINT_ARM_L_5_UPPER_LIMIT}"
+        effort="${EFFORT_LIMIT}"
+        velocity="${VELOCITY_LIMIT}"/>
       <axis xyz="0 1 0"/>
       <dynamics damping="1.0e-6" friction="0.8"/>
@@ -166,5 +148,5 @@
           <mesh filename="package://sciurus17_description/meshes/visual/L_Link5.stl" scale="1.0 1.0 1.0"/>
         </geometry>
-        <material name="${arm_color}"/>
+        <material name="${COLOR_LINK_ARM}"/>
       </visual>
       <visual>
@@ -209,5 +191,5 @@
           <cylinder length="0.001" radius="0.001"/>
         </geometry>
-        <material name="${arm_color}"/>
+        <material name="${COLOR_LINK_ARM}"/>
       </visual>
       <collision>
@@ -223,8 +205,8 @@
       <origin xyz="0.0 0.129 0.0" rpy="0 0 0"/>
       <limit
-        lower="${arm_joint6_lower_limit}"
-        upper="${arm_joint6_upper_limit}"
-        effort="${arm_joints_effort_limit}"
-        velocity="${arm_joints_velocity_limit}"/>
+        lower="${JOINT_ARM_L_6_LOWER_LIMIT}"
+        upper="${JOINT_ARM_L_6_UPPER_LIMIT}"
+        effort="${EFFORT_LIMIT}"
+        velocity="${VELOCITY_LIMIT}"/>
       <axis xyz="0 0 1"/>
       <dynamics damping="1.0e-6" friction="0.8"/>
@@ -236,5 +218,5 @@
           <mesh filename="package://sciurus17_description/meshes/visual/L_Link6.stl" scale="1.0 1.0 1.0"/>
         </geometry>
-        <material name="${arm_color}"/>
+        <material name="${COLOR_LINK_ARM}"/>
       </visual>
       <collision>
@@ -255,8 +237,8 @@
       <origin xyz="0.0 0.0191 0.0" rpy="0 0 0"/>
       <limit
-        lower="${arm_joint7_lower_limit}"
-        upper="${arm_joint7_upper_limit}"
-        effort="${arm_joints_effort_limit}"
-        velocity="${arm_joints_velocity_limit}"/>
+        lower="${JOINT_ARM_L_7_LOWER_LIMIT}"
+        upper="${JOINT_ARM_L_7_UPPER_LIMIT}"
+        effort="${EFFORT_LIMIT}"
+        velocity="${VELOCITY_LIMIT}"/>
       <axis xyz="0 1 0"/>
       <dynamics damping="1.0e-6" friction="0.8"/>

File: urdf/sciurus17_left_hand.xacro (robot description, xacro)
@@ -1,11 +1,5 @@
 <?xml version="1.0"?>
 <robot xmlns:xacro="http://ros.org/wiki/xacro">
-  <xacro:macro name="sciurus17_left_hand"
-    params="hand_joints_lower_limit
-            hand_joints_upper_limit
-            hand_joints_effort_limit
-            hand_joints_velocity_limit
-            hand_color
-            ">
+  <xacro:macro name="sciurus17_left_hand">
     <link name="${NAME_LINK_ARM_L_7}">
       <visual>
@@ -14,5 +8,5 @@
           <mesh filename="package://sciurus17_description/meshes/visual/L_Link7.stl" scale="1.0 1.0 1.0"/>
         </geometry>
-        <material name="${hand_color}"/>
+        <material name="${COLOR_LINK_HAND}"/>
       </visual>
       <collision>
@@ -33,8 +27,8 @@
       <origin xyz="0.012 0.024 0.0" rpy="0 0 0"/>
       <limit
-        lower="${hand_joints_lower_limit}"
-        upper="${hand_joints_upper_limit}"
-        effort="${hand_joints_effort_limit}"
-        velocity="${hand_joints_velocity_limit}"/>
+        lower="${JOINT_HAND_L_LOWER_LIMIT}"
+        upper="${JOINT_HAND_L_UPPER_LIMIT}"
+        effort="${EFFORT_LIMIT}"
+        velocity="${VELOCITY_LIMIT}"/>
       <axis xyz="0 0 1"/>
       <dynamics damping="1.0e-6" friction="0.8"/>
@@ -46,5 +40,5 @@
           <mesh filename="package://sciurus17_description/meshes/visual/L_HandA.stl" scale="1.0 1.0 1.0"/>
         </geometry>
-        <material name="${hand_color}"/>
+        <material name="${COLOR_LINK_HAND}"/>
       </visual>
       <collision>
@@ -65,8 +59,8 @@
       <origin xyz="-0.012 0.024 0.0" rpy="0 0 0"/>
       <limit
-        lower="${hand_joints_lower_limit}"
-        upper="${hand_joints_upper_limit}"
-        effort="${hand_joints_effort_limit}"
-        velocity="${hand_joints_velocity_limit}"/>
+        lower="${JOINT_HAND_L_LOWER_LIMIT}"
+        upper="${JOINT_HAND_L_UPPER_LIMIT}"
+        effort="${EFFORT_LIMIT}"
+        velocity="${VELOCITY_LIMIT}"/>
       <axis xyz="0 0 -1"/>
       <mimic joint="${NAME_JOINT_HAND_L_A}" multiplier="1" offset="0"/>
@@ -79,5 +73,5 @@
           <mesh filename="package://sciurus17_description/meshes/visual/L_HandB.stl" scale="1.0 1.0 1.0"/>
         </geometry>
-        <material name="${hand_color}"/>
+        <material name="${COLOR_LINK_HAND}"/>
       </visual>
       <collision>

File: urdf/sciurus17_right_arm.xacro (robot description, xacro)
@@ -1,23 +1,5 @@
 <?xml version="1.0"?>
 <robot xmlns:xacro="http://ros.org/wiki/xacro">
-  <xacro:macro name="sciurus17_right_arm"
-    params="arm_joint1_lower_limit
-            arm_joint1_upper_limit
-            arm_joint2_lower_limit
-            arm_joint2_upper_limit
-            arm_joint3_lower_limit
-            arm_joint3_upper_limit
-            arm_joint4_lower_limit
-            arm_joint4_upper_limit
-            arm_joint5_lower_limit
-            arm_joint5_upper_limit
-            arm_joint6_lower_limit
-            arm_joint6_upper_limit
-            arm_joint7_lower_limit
-            arm_joint7_upper_limit
-            arm_joints_effort_limit
-            arm_joints_velocity_limit
-            arm_color
-            ">
+  <xacro:macro name="sciurus17_right_arm">
     <joint name="${NAME_JOINT_ARM_R_1}" type="revolute">
       <parent link="${NAME_LINK_BODY}" />
@@ -25,8 +7,8 @@
       <origin xyz="0.08083 -0.0965 0.2885" rpy="0 0 0"/>
       <limit
-        lower="${arm_joint1_lower_limit}"
-        upper="${arm_joint1_upper_limit}"
-        effort="${arm_joints_effort_limit}"
-        velocity="${arm_joints_velocity_limit}"/>
+        lower="${JOINT_ARM_R_1_LOWER_LIMIT}"
+        upper="${JOINT_ARM_R_1_UPPER_LIMIT}"
+        effort="${EFFORT_LIMIT}"
+        velocity="${VELOCITY_LIMIT}"/>
       <axis xyz="0 -1 0"/>
       <dynamics damping="1.0e-6" friction="0.8"/>
@@ -38,5 +20,5 @@
           <mesh filename="package://sciurus17_description/meshes/visual/R_Link1.stl" scale="1.0 1.0 1.0"/>
         </geometry>
-        <material name="${arm_color}"/>
+        <material name="${COLOR_LINK_ARM}"/>
       </visual>
       <collision>
@@ -57,8 +39,8 @@
       <origin xyz="0.0 -0.064 0.0" rpy="0 0 0"/>
       <limit
-        lower="${arm_joint2_lower_limit}"
-        upper="${arm_joint2_upper_limit}"
-        effort="${arm_joints_effort_limit}"
-        velocity="${arm_joints_velocity_limit}"/>
+        lower="${JOINT_ARM_R_2_LOWER_LIMIT}"
+        upper="${JOINT_ARM_R_2_UPPER_LIMIT}"
+        effort="${EFFORT_LIMIT}"
+        velocity="${VELOCITY_LIMIT}"/>
       <axis xyz="-1 0 0"/>
       <dynamics damping="1.0e-6" friction="0.8"/>
@@ -70,5 +52,5 @@
           <mesh filename="package://sciurus17_description/meshes/visual/R_Link2.stl" scale="1.0 1.0 1.0"/>
         </geometry>
-        <material name="${arm_color}"/>
+        <material name="${COLOR_LINK_ARM}"/>
       </visual>
       <collision>
@@ -89,8 +71,8 @@
       <origin xyz="0.0 -0.065 0.0" rpy="0 0 0"/>
       <limit
-        lower="${arm_joint3_lower_limit}"
-        upper="${arm_joint3_upper_limit}"
-        effort="${arm_joints_effort_limit}"
-        velocity="${arm_joints_velocity_limit}"/>
+        lower="${JOINT_ARM_R_3_LOWER_LIMIT}"
+        upper="${JOINT_ARM_R_3_UPPER_LIMIT}"
+        effort="${EFFORT_LIMIT}"
+        velocity="${VELOCITY_LIMIT}"/>
       <axis xyz="0 -1 0"/>
       <dynamics damping="1.0e-6" friction="0.8"/>
@@ -102,5 +84,5 @@
           <mesh filename="package://sciurus17_description/meshes/visual/L_Link3.stl" scale="1.0 -1.0 1.0"/>
         </geometry>
-        <material name="${arm_color}"/>
+        <material name="${COLOR_LINK_ARM}"/>
       </visual>
       <collision>
@@ -121,8 +103,8 @@
       <origin xyz="0.0 -0.185 0.0" rpy="0 0 0"/>
       <limit
-        lower="${arm_joint4_lower_limit}"
-        upper="${arm_joint4_upper_limit}"
-        effort="${arm_joints_effort_limit}"
-        velocity="${arm_joints_velocity_limit}"/>
+        lower="${JOINT_ARM_R_4_LOWER_LIMIT}"
+        upper="${JOINT_ARM_R_4_UPPER_LIMIT}"
+        effort="${EFFORT_LIMIT}"
+        velocity="${VELOCITY_LIMIT}"/>
       <axis xyz="0 0 1"/>
       <dynamics damping="1.0e-6" friction="0.8"/>
@@ -134,5 +116,5 @@
           <mesh filename="package://sciurus17_description/meshes/visual/R_Link4.stl" scale="1.0 1.0 1.0"/>
         </geometry>
-        <material name="${arm_color}"/>
+        <material name="${COLOR_LINK_ARM}"/>
       </visual>
       <collision>
@@ -153,8 +135,8 @@
       <origin xyz="0.0 -0.121 0.0" rpy="0 0 0"/>
       <limit
-        lower="${arm_joint5_lower_limit}"
-        upper="${arm_joint5_upper_limit}"
-        effort="${arm_joints_effort_limit}"
-        velocity="${arm_joints_velocity_limit}"/>
+        lower="${JOINT_ARM_R_5_LOWER_LIMIT}"
+        upper="${JOINT_ARM_R_5_UPPER_LIMIT}"
+        effort="${EFFORT_LIMIT}"
+        velocity="${VELOCITY_LIMIT}"/>
       <axis xyz="0 -1 0"/>
       <dynamics damping="1.0e-6" friction="0.8"/>
@@ -166,5 +148,5 @@
           <mesh filename="package://sciurus17_description/meshes/visual/R_Link5.stl" scale="1.0 1.0 1.0"/>
         </geometry>
-        <material name="${arm_color}"/>
+        <material name="${COLOR_LINK_ARM}"/>
       </visual>
       <visual>
@@ -209,5 +191,5 @@
           <cylinder length="0.001" radius="0.001"/>
         </geometry>
-        <material name="${arm_color}"/>
+        <material name="${COLOR_LINK_ARM}"/>
       </visual>
       <collision>
@@ -223,8 +205,8 @@
       <origin xyz="0.0 -0.129 0.0" rpy="0 0 0"/>
       <limit
-        lower="${arm_joint6_lower_limit}"
-        upper="${arm_joint6_upper_limit}"
-        effort="${arm_joints_effort_limit}"
-        velocity="${arm_joints_velocity_limit}"/>
+        lower="${JOINT_ARM_R_6_LOWER_LIMIT}"
+        upper="${JOINT_ARM_R_6_UPPER_LIMIT}"
+        effort="${EFFORT_LIMIT}"
+        velocity="${VELOCITY_LIMIT}"/>
       <axis xyz="0 0 1"/>
       <dynamics damping="1.0e-6" friction="0.8"/>
@@ -236,5 +218,5 @@
           <mesh filename="package://sciurus17_description/meshes/visual/R_Link6.stl" scale="1.0 1.0 1.0"/>
         </geometry>
-        <material name="${arm_color}"/>
+        <material name="${COLOR_LINK_ARM}"/>
       </visual>
       <collision>
@@ -255,8 +237,8 @@
       <origin xyz="0.0 -0.0191 0.0" rpy="0 0 0"/>
       <limit
-        lower="${arm_joint7_lower_limit}"
-        upper="${arm_joint7_upper_limit}"
-        effort="${arm_joints_effort_limit}"
-        velocity="${arm_joints_velocity_limit}"/>
+        lower="${JOINT_ARM_R_7_LOWER_LIMIT}"
+        upper="${JOINT_ARM_R_7_UPPER_LIMIT}"
+        effort="${EFFORT_LIMIT}"
+        velocity="${VELOCITY_LIMIT}"/>
       <axis xyz="0 -1 0"/>
       <dynamics damping="1.0e-6" friction="0.8"/>
