Commit message: macroの引数によるパラメータ設定を削除

File: urdf/sciurus17_right_hand.xacro (robot description, xacro)
@@ -1,11 +1,5 @@
 <?xml version="1.0"?>
 <robot xmlns:xacro="http://ros.org/wiki/xacro">
-  <xacro:macro name="sciurus17_right_hand"
-    params="hand_joints_lower_limit
-            hand_joints_upper_limit
-            hand_joints_effort_limit
-            hand_joints_velocity_limit
-            hand_color
-            ">
+  <xacro:macro name="sciurus17_right_hand">
     <link name="${NAME_LINK_ARM_R_7}">
       <visual>
@@ -14,5 +8,5 @@
           <mesh filename="package://sciurus17_description/meshes/visual/R_Link7.stl" scale="1.0 1.0 1.0"/>
         </geometry>
-        <material name="${hand_color}"/>
+        <material name="${COLOR_LINK_HAND}"/>
       </visual>
       <collision>
@@ -33,8 +27,8 @@
       <origin xyz="0.012 -0.024 0.0" rpy="0 0 0"/>
       <limit
-        lower="${hand_joints_lower_limit}"
-        upper="${hand_joints_upper_limit}"
-        effort="${hand_joints_effort_limit}"
-        velocity="${hand_joints_velocity_limit}"/>
+        lower="${JOINT_HAND_R_LOWER_LIMIT}"
+        upper="${JOINT_HAND_R_UPPER_LIMIT}"
+        effort="${EFFORT_LIMIT}"
+        velocity="${VELOCITY_LIMIT}"/>
       <axis xyz="0 0 1"/>
       <dynamics damping="1.0e-6" friction="0.8"/>
@@ -47,5 +41,5 @@
           <mesh filename="package://sciurus17_description/meshes/visual/R_HandA.stl" scale="1.0 1.0 1.0"/>
         </geometry>
-        <material name="${hand_color}"/>
+        <material name="${COLOR_LINK_HAND}"/>
       </visual>
       <collision>
@@ -66,8 +60,8 @@
       <origin xyz="-0.012 -0.024 0.0" rpy="0 0 0"/>
       <limit
-        lower="${hand_joints_lower_limit}"
-        upper="${hand_joints_upper_limit}"
-        effort="${hand_joints_effort_limit}"
-        velocity="${hand_joints_velocity_limit}"/>
+        lower="${JOINT_HAND_R_LOWER_LIMIT}"
+        upper="${JOINT_HAND_R_UPPER_LIMIT}"
+        effort="${EFFORT_LIMIT}"
+        velocity="${VELOCITY_LIMIT}"/>
       <axis xyz="0 0 -1"/>
       <mimic joint="${NAME_JOINT_HAND_R_A}" multiplier="1" offset="0"/>
@@ -81,5 +75,5 @@
           <mesh filename="package://sciurus17_description/meshes/visual/R_HandB.stl" scale="1.0 1.0 1.0"/>
         </geometry>
-        <material name="${hand_color}"/>
+        <material name="${COLOR_LINK_HAND}"/>
       </visual>
       <collision>

Commit message: cameraのproperty名変更

File: urdf/sciurus17.urdf.xacro (robot description, xacro)
@@ -17,5 +17,5 @@
   <xacro:property name="NAME_LINK_NECK_1" value="neck_yaw_link"/>
   <xacro:property name="NAME_LINK_NECK_2" value="neck_pitch_link"/>
-  <xacro:property name="NAME_LINK_CAMERA" value="camera_link"/>
+  <xacro:property name="NAME_LINK_HEAD_CAMERA" value="camera_link"/>
   <xacro:property name="NAME_LINK_CHEST_CAMERA" value="chest_camera_link"/>
   <xacro:property name="NAME_LINK_ARM_R_1" value="r_link1"/>
@@ -43,5 +43,5 @@
   <xacro:property name="NAME_JOINT_NECK_1" value="neck_yaw_joint"/>
   <xacro:property name="NAME_JOINT_NECK_2" value="neck_pitch_joint"/>
-  <xacro:property name="NAME_JOINT_CAMERA" value="head_camera_joint"/>
+  <xacro:property name="NAME_JOINT_HEAD_CAMERA" value="head_camera_joint"/>
   <xacro:property name="NAME_JOINT_CHEST_CAMERA" value="chest_camera_joint"/>
   <xacro:property name="NAME_JOINT_ARM_R_1" value="r_arm_joint1"/>

File: urdf/sciurus17_head.xacro (robot description, xacro)
@@ -64,10 +64,10 @@
       </inertial>
     </link>
-    <joint name="${NAME_JOINT_CAMERA}" type="fixed">
+    <joint name="${NAME_JOINT_HEAD_CAMERA}" type="fixed">
       <parent link="${NAME_LINK_NECK_2}" />
-      <child link="${NAME_LINK_CAMERA}" />
+      <child link="${NAME_LINK_HEAD_CAMERA}" />
       <origin xyz="0.081785 0.020 0.091" rpy="0 0 0"/>
     </joint>
-    <link name="${NAME_LINK_CAMERA}">
+    <link name="${NAME_LINK_HEAD_CAMERA}">
       <visual>
         <origin xyz="0 0 0" rpy="0 0 0"/>
@@ -90,5 +90,5 @@
       <material>Gazebo/White</material>
     </gazebo>
-    <gazebo reference="${NAME_LINK_CAMERA}">
+    <gazebo reference="${NAME_LINK_HEAD_CAMERA}">
       <material>Gazebo/Black</material>
     </gazebo>

Commit message: 頭部カメラリンクをhead_camera_linkに変更
Co-authored-by: Shota Aoki <macakasit@gmail.com>

File: urdf/sciurus17.urdf.xacro (robot description, xacro)
@@ -17,5 +17,5 @@
   <xacro:property name="NAME_LINK_NECK_1" value="neck_yaw_link"/>
   <xacro:property name="NAME_LINK_NECK_2" value="neck_pitch_link"/>
-  <xacro:property name="NAME_LINK_HEAD_CAMERA" value="camera_link"/>
+  <xacro:property name="NAME_LINK_HEAD_CAMERA" value="head_camera_link"/>
   <xacro:property name="NAME_LINK_CHEST_CAMERA" value="chest_camera_link"/>
   <xacro:property name="NAME_LINK_ARM_R_1" value="r_link1"/>

Commit message: use_gazeboオプション追加

File: urdf/sciurus17.urdf.xacro (robot description, xacro)
@@ -1,4 +1,9 @@
 <?xml version="1.0"?>
-<robot name="sciurus17" xmlns:xacro="http://ros.org/wiki/xacro" >
+<robot
+    name="sciurus17"
+    xmlns:xacro="http://ros.org/wiki/xacro"
+    xmlns:sensor="http://playerstage.sourceforge.net/gazebo/xmlschema/#sensor"
+    xmlns:controller="http://playerstage.sourceforge.net/gazebo/xmlschema/#controller"
+    xmlns:interface="http://playerstage.sourceforge.net/gazebo/xmlschema/#interface">
   <xacro:include filename="$(find sciurus17_description)/urdf/sciurus17_body.xacro"/>
   <xacro:include filename="$(find sciurus17_description)/urdf/sciurus17_head.xacro"/>
@@ -7,4 +12,6 @@
   <xacro:include filename="$(find sciurus17_description)/urdf/sciurus17_left_arm.xacro"/>
   <xacro:include filename="$(find sciurus17_description)/urdf/sciurus17_left_hand.xacro"/>
+  <xacro:include filename="$(find sciurus17_description)/urdf/sciurus17_gazebo.xacro"/>
+  <xacro:arg name="use_gazebo" default="false" />
   <material name="white">
     <color rgba="0.9 0.9 0.9 1.0"/>
@@ -111,46 +118,4 @@
   <xacro:property name="COLOR_LINK_HAND" value="red"/>
   <xacro:property name="COLOR_LINK_CAMERA" value="white"/>
-  <xacro:arg name="use_gazebo_simulation" default="false" />
-  <xacro:arg name="load_trans1" default="false" />
-  <xacro:arg name="load_trans2" default="false" />
-  <xacro:arg name="load_trans3" default="false" />
-  <xacro:arg name="use_effort_right_arm" default="false" />
-  <xacro:property name="right_arm_interface" value="position"/>
-  <xacro:if value="$(arg use_effort_right_arm)">
-    <xacro:property name="right_arm_interface" value="effort"/>
-  </xacro:if>
-  <xacro:arg name="use_effort_left_wrist" default="false" />
-  <xacro:property name="left_wrist_interface" value="position"/>
-  <xacro:if value="$(arg use_effort_left_wrist)">
-    <xacro:property name="left_wrist_interface" value="effort"/>
-  </xacro:if>
-  <xacro:if value="$(arg use_gazebo_simulation)">
-    <xacro:include filename="$(find sciurus17_description)/urdf/sciurus17_gazebo.xacro"/>
-    <xacro:if value="$(arg load_trans1)">
-      <xacro:default_transmission joint_name="r_arm_joint1" interface="${right_arm_interface}"/>
-      <xacro:default_transmission joint_name="r_arm_joint2" interface="${right_arm_interface}"/>
-      <xacro:default_transmission joint_name="r_arm_joint3" interface="${right_arm_interface}"/>
-      <xacro:default_transmission joint_name="r_arm_joint4" interface="${right_arm_interface}"/>
-      <xacro:default_transmission joint_name="r_arm_joint5" interface="${right_arm_interface}"/>
-      <xacro:default_transmission joint_name="r_arm_joint6" interface="${right_arm_interface}"/>
-      <xacro:default_transmission joint_name="r_arm_joint7" interface="${right_arm_interface}"/>
-      <xacro:default_transmission joint_name="r_hand_joint"/>
-    </xacro:if>
-    <xacro:if value="$(arg load_trans2)">
-      <xacro:default_transmission joint_name="l_arm_joint1"/>
-      <xacro:default_transmission joint_name="l_arm_joint2"/>
-      <xacro:default_transmission joint_name="l_arm_joint3"/>
-      <xacro:default_transmission joint_name="l_arm_joint4"/>
-      <xacro:default_transmission joint_name="l_arm_joint5"/>
-      <xacro:default_transmission joint_name="l_arm_joint6"/>
-      <xacro:default_transmission joint_name="l_arm_joint7" interface="${left_wrist_interface}"/>
-      <xacro:default_transmission joint_name="l_hand_joint"/>
-    </xacro:if>
-    <xacro:if value="$(arg load_trans3)">
-      <xacro:default_transmission joint_name="waist_yaw_joint"/>
-      <xacro:default_transmission joint_name="neck_yaw_joint"/>
-      <xacro:default_transmission joint_name="neck_pitch_joint"/>
-    </xacro:if>
-  </xacro:if>
   <!-- Used for fixing robot 'base_link'  to Gazebo 'world' -->
   <link name="world"/>
@@ -165,3 +130,6 @@
   <xacro:sciurus17_left_arm/>
   <xacro:sciurus17_left_hand/>
+  <xacro:if value="$(arg use_gazebo)">
+    <xacro:gazebo_robot_settings/>
+  </xacro:if>
 </robot>

Commit message: ign_ros2_control追加

File: urdf/sciurus17.urdf.xacro (robot description, xacro)
@@ -13,5 +13,10 @@
   <xacro:include filename="$(find sciurus17_description)/urdf/sciurus17_left_hand.xacro"/>
   <xacro:include filename="$(find sciurus17_description)/urdf/sciurus17_gazebo.xacro"/>
+  <xacro:include filename="$(find sciurus17_description)/urdf/sciurus17.gazebo_ros2_control.xacro"/>
   <xacro:arg name="use_gazebo" default="false" />
+  <xacro:arg name="gz_control_config_package" default="" />
+  <xacro:arg name="gz_control_config_file_path" default="" />
+  <xacro:property name="GZ_CONTROL_CONFIG_PACKAGE" value="$(arg gz_control_config_package)"/>
+  <xacro:property name="GZ_CONTROL_CONFIG_FILE_PATH" value="$(arg gz_control_config_file_path)"/>
   <material name="white">
     <color rgba="0.9 0.9 0.9 1.0"/>
@@ -132,4 +137,5 @@
   <xacro:if value="$(arg use_gazebo)">
     <xacro:gazebo_robot_settings/>
+    <xacro:sciurus17_gazebo_ros2_control_settings/>
   </xacro:if>
 </robot>

File: urdf/sciurus17_gazebo.xacro (robot description, xacro)
@@ -26,4 +26,9 @@
   </xacro:macro>
   <xacro:macro name="gazebo_robot_settings">
+    <gazebo>
+      <plugin filename="libign_ros2_control-system.so" name="ign_ros2_control::IgnitionROS2ControlPlugin">
+        <parameters>$(find ${GZ_CONTROL_CONFIG_PACKAGE})/${GZ_CONTROL_CONFIG_FILE_PATH}</parameters>
+      </plugin>
+    </gazebo>
     <gazebo reference="${NAME_LINK_BASE}">
       <xacro:material_gazebo_white/>

Commit message: joint_limit値の調整

File: urdf/sciurus17.urdf.xacro (robot description, xacro)
@@ -91,5 +91,7 @@
   <xacro:property name="JOINT_ARM_R_3_LOWER_LIMIT" value="${radians(-90)}"/>
   <xacro:property name="JOINT_ARM_R_3_UPPER_LIMIT" value="${radians(90)}"/>
-  <xacro:property name="JOINT_ARM_R_4_LOWER_LIMIT" value="${radians(0)}"/>
+  <!-- Gazeboの挙動がlimit付近で不安定なため、limitをサーボの可動範囲より少し大きくする -->
+  <!-- 参照: https://github.com/rt-net/sciurus17_description/pull/6 -->
+  <xacro:property name="JOINT_ARM_R_4_LOWER_LIMIT" value="${radians(-0.001)}"/>
   <xacro:property name="JOINT_ARM_R_4_UPPER_LIMIT" value="${radians(157)}"/>
   <xacro:property name="JOINT_ARM_R_5_LOWER_LIMIT" value="${radians(-90)}"/>
@@ -99,5 +101,7 @@
   <xacro:property name="JOINT_ARM_R_7_LOWER_LIMIT" value="${radians(-170)}"/>
   <xacro:property name="JOINT_ARM_R_7_UPPER_LIMIT" value="${radians(170)}"/>
-  <xacro:property name="JOINT_HAND_R_LOWER_LIMIT" value="${radians(0)}"/>
+  <!-- Gazeboの挙動がlimit付近で不安定なため、limitをサーボの可動範囲より少し大きくする -->
+  <!-- 参照: https://github.com/rt-net/sciurus17_description/pull/6 -->
+  <xacro:property name="JOINT_HAND_R_LOWER_LIMIT" value="${radians(-0.001)}"/>
   <xacro:property name="JOINT_HAND_R_UPPER_LIMIT" value="${radians(86)}"/>
   <xacro:property name="JOINT_ARM_L_1_LOWER_LIMIT" value="${radians(-90)}"/>
@@ -108,5 +112,7 @@
   <xacro:property name="JOINT_ARM_L_3_UPPER_LIMIT" value="${radians(90)}"/>
   <xacro:property name="JOINT_ARM_L_4_LOWER_LIMIT" value="${radians(-157)}"/>
-  <xacro:property name="JOINT_ARM_L_4_UPPER_LIMIT" value="${radians(0)}"/>
+  <!-- Gazeboの挙動がlimit付近で不安定なため、limitをサーボの可動範囲より少し大きくする -->
+  <!-- 参照: https://github.com/rt-net/sciurus17_description/pull/6 -->
+  <xacro:property name="JOINT_ARM_L_4_UPPER_LIMIT" value="${radians(0.001)}"/>
   <xacro:property name="JOINT_ARM_L_5_LOWER_LIMIT" value="${radians(-90)}"/>
   <xacro:property name="JOINT_ARM_L_5_UPPER_LIMIT" value="${radians(90)}"/>
@@ -116,5 +122,7 @@
   <xacro:property name="JOINT_ARM_L_7_UPPER_LIMIT" value="${radians(170)}"/>
   <xacro:property name="JOINT_HAND_L_LOWER_LIMIT" value="${radians(-86)}"/>
-  <xacro:property name="JOINT_HAND_L_UPPER_LIMIT" value="${radians(0)}"/>
+  <!-- Gazeboの挙動がlimit付近で不安定なため、limitをサーボの可動範囲より少し大きくする -->
+  <!-- 参照: https://github.com/rt-net/sciurus17_description/pull/6 -->
+  <xacro:property name="JOINT_HAND_L_UPPER_LIMIT" value="${radians(0.001)}"/>
   <xacro:property name="COLOR_LINK_BASE" value="white"/>
   <xacro:property name="COLOR_LINK_BODY" value="white"/>

Commit message: 関節可動範囲の調整

File: urdf/sciurus17.urdf.xacro (robot description, xacro)
@@ -93,5 +93,5 @@
   <!-- Gazeboの挙動がlimit付近で不安定なため、limitをサーボの可動範囲より少し大きくする -->
   <!-- 参照: https://github.com/rt-net/sciurus17_description/pull/6 -->
-  <xacro:property name="JOINT_ARM_R_4_LOWER_LIMIT" value="${radians(-0.001)}"/>
+  <xacro:property name="JOINT_ARM_R_4_LOWER_LIMIT" value="${radians(-0.01)}"/>
   <xacro:property name="JOINT_ARM_R_4_UPPER_LIMIT" value="${radians(157)}"/>
   <xacro:property name="JOINT_ARM_R_5_LOWER_LIMIT" value="${radians(-90)}"/>
@@ -103,5 +103,5 @@
   <!-- Gazeboの挙動がlimit付近で不安定なため、limitをサーボの可動範囲より少し大きくする -->
   <!-- 参照: https://github.com/rt-net/sciurus17_description/pull/6 -->
-  <xacro:property name="JOINT_HAND_R_LOWER_LIMIT" value="${radians(-0.001)}"/>
+  <xacro:property name="JOINT_HAND_R_LOWER_LIMIT" value="${radians(-0.01)}"/>
   <xacro:property name="JOINT_HAND_R_UPPER_LIMIT" value="${radians(86)}"/>
   <xacro:property name="JOINT_ARM_L_1_LOWER_LIMIT" value="${radians(-90)}"/>
@@ -114,5 +114,5 @@
   <!-- Gazeboの挙動がlimit付近で不安定なため、limitをサーボの可動範囲より少し大きくする -->
   <!-- 参照: https://github.com/rt-net/sciurus17_description/pull/6 -->
-  <xacro:property name="JOINT_ARM_L_4_UPPER_LIMIT" value="${radians(0.001)}"/>
+  <xacro:property name="JOINT_ARM_L_4_UPPER_LIMIT" value="${radians(0.01)}"/>
   <xacro:property name="JOINT_ARM_L_5_LOWER_LIMIT" value="${radians(-90)}"/>
   <xacro:property name="JOINT_ARM_L_5_UPPER_LIMIT" value="${radians(90)}"/>
@@ -124,5 +124,5 @@
   <!-- Gazeboの挙動がlimit付近で不安定なため、limitをサーボの可動範囲より少し大きくする -->
   <!-- 参照: https://github.com/rt-net/sciurus17_description/pull/6 -->
-  <xacro:property name="JOINT_HAND_L_UPPER_LIMIT" value="${radians(0.001)}"/>
+  <xacro:property name="JOINT_HAND_L_UPPER_LIMIT" value="${radians(0.01)}"/>
   <xacro:property name="COLOR_LINK_BASE" value="white"/>
   <xacro:property name="COLOR_LINK_BODY" value="white"/>

Commit message: GazeboでのMoveIt動作に対応 (#6)
* control_configパス追加

* ign_ros2_control追加

* dummy_mimic joint追加

* test修正

* joint_limit値の調整

* 干渉が生じるモデルを修正

* Gazebo上での初期姿勢設定

* 関節可動範囲の調整

File: urdf/sciurus17.urdf.xacro (robot description, xacro)
@@ -13,5 +13,10 @@
   <xacro:include filename="$(find sciurus17_description)/urdf/sciurus17_left_hand.xacro"/>
   <xacro:include filename="$(find sciurus17_description)/urdf/sciurus17_gazebo.xacro"/>
+  <xacro:include filename="$(find sciurus17_description)/urdf/sciurus17.gazebo_ros2_control.xacro"/>
   <xacro:arg name="use_gazebo" default="false" />
+  <xacro:arg name="gz_control_config_package" default="" />
+  <xacro:arg name="gz_control_config_file_path" default="" />
+  <xacro:property name="GZ_CONTROL_CONFIG_PACKAGE" value="$(arg gz_control_config_package)"/>
+  <xacro:property name="GZ_CONTROL_CONFIG_FILE_PATH" value="$(arg gz_control_config_file_path)"/>
   <material name="white">
     <color rgba="0.9 0.9 0.9 1.0"/>
@@ -86,5 +91,7 @@
   <xacro:property name="JOINT_ARM_R_3_LOWER_LIMIT" value="${radians(-90)}"/>
   <xacro:property name="JOINT_ARM_R_3_UPPER_LIMIT" value="${radians(90)}"/>
-  <xacro:property name="JOINT_ARM_R_4_LOWER_LIMIT" value="${radians(0)}"/>
+  <!-- Gazeboの挙動がlimit付近で不安定なため、limitをサーボの可動範囲より少し大きくする -->
+  <!-- 参照: https://github.com/rt-net/sciurus17_description/pull/6 -->
+  <xacro:property name="JOINT_ARM_R_4_LOWER_LIMIT" value="${radians(-0.01)}"/>
   <xacro:property name="JOINT_ARM_R_4_UPPER_LIMIT" value="${radians(157)}"/>
   <xacro:property name="JOINT_ARM_R_5_LOWER_LIMIT" value="${radians(-90)}"/>
@@ -94,5 +101,7 @@
   <xacro:property name="JOINT_ARM_R_7_LOWER_LIMIT" value="${radians(-170)}"/>
   <xacro:property name="JOINT_ARM_R_7_UPPER_LIMIT" value="${radians(170)}"/>
-  <xacro:property name="JOINT_HAND_R_LOWER_LIMIT" value="${radians(0)}"/>
+  <!-- Gazeboの挙動がlimit付近で不安定なため、limitをサーボの可動範囲より少し大きくする -->
+  <!-- 参照: https://github.com/rt-net/sciurus17_description/pull/6 -->
+  <xacro:property name="JOINT_HAND_R_LOWER_LIMIT" value="${radians(-0.01)}"/>
   <xacro:property name="JOINT_HAND_R_UPPER_LIMIT" value="${radians(86)}"/>
   <xacro:property name="JOINT_ARM_L_1_LOWER_LIMIT" value="${radians(-90)}"/>
@@ -103,5 +112,7 @@
   <xacro:property name="JOINT_ARM_L_3_UPPER_LIMIT" value="${radians(90)}"/>
   <xacro:property name="JOINT_ARM_L_4_LOWER_LIMIT" value="${radians(-157)}"/>
-  <xacro:property name="JOINT_ARM_L_4_UPPER_LIMIT" value="${radians(0)}"/>
+  <!-- Gazeboの挙動がlimit付近で不安定なため、limitをサーボの可動範囲より少し大きくする -->
+  <!-- 参照: https://github.com/rt-net/sciurus17_description/pull/6 -->
+  <xacro:property name="JOINT_ARM_L_4_UPPER_LIMIT" value="${radians(0.01)}"/>
   <xacro:property name="JOINT_ARM_L_5_LOWER_LIMIT" value="${radians(-90)}"/>
   <xacro:property name="JOINT_ARM_L_5_UPPER_LIMIT" value="${radians(90)}"/>
@@ -111,5 +122,7 @@
   <xacro:property name="JOINT_ARM_L_7_UPPER_LIMIT" value="${radians(170)}"/>
   <xacro:property name="JOINT_HAND_L_LOWER_LIMIT" value="${radians(-86)}"/>
-  <xacro:property name="JOINT_HAND_L_UPPER_LIMIT" value="${radians(0)}"/>
+  <!-- Gazeboの挙動がlimit付近で不安定なため、limitをサーボの可動範囲より少し大きくする -->
+  <!-- 参照: https://github.com/rt-net/sciurus17_description/pull/6 -->
+  <xacro:property name="JOINT_HAND_L_UPPER_LIMIT" value="${radians(0.01)}"/>
   <xacro:property name="COLOR_LINK_BASE" value="white"/>
   <xacro:property name="COLOR_LINK_BODY" value="white"/>
@@ -132,4 +145,5 @@
   <xacro:if value="$(arg use_gazebo)">
     <xacro:gazebo_robot_settings/>
+    <xacro:sciurus17_gazebo_ros2_control_settings/>
   </xacro:if>
 </robot>

Commit message: 実機の起動に必要なパラメータ追加

File: urdf/sciurus17.urdf.xacro (robot description, xacro)
@@ -6,4 +6,5 @@
     xmlns:controller="http://playerstage.sourceforge.net/gazebo/xmlschema/#controller"
     xmlns:interface="http://playerstage.sourceforge.net/gazebo/xmlschema/#interface">
+  <xacro:include filename="$(find sciurus17_description)/urdf/sciurus17.ros2_control.xacro"/>
   <xacro:include filename="$(find sciurus17_description)/urdf/sciurus17_body.xacro"/>
   <xacro:include filename="$(find sciurus17_description)/urdf/sciurus17_head.xacro"/>
@@ -15,6 +16,14 @@
   <xacro:include filename="$(find sciurus17_description)/urdf/sciurus17.gazebo_ros2_control.xacro"/>
   <xacro:arg name="use_gazebo" default="false" />
+  <xacro:arg name="port_name" default="/dev/sciurus17spine" />
+  <xacro:arg name="baudrate" default="3000000" />
+  <xacro:arg name="timeout_seconds" default="1.0" />
+  <xacro:arg name="manipulator_config_file_path" default="" />
   <xacro:arg name="gz_control_config_package" default="" />
   <xacro:arg name="gz_control_config_file_path" default="" />
+  <xacro:property name="PORT_NAME" value="$(arg port_name)"/>
+  <xacro:property name="BAUDRATE" value="$(arg baudrate)"/>
+  <xacro:property name="TIMEOUT_SECONDS" value="$(arg timeout_seconds)"/>
+  <xacro:property name="MANIPULATOR_CONFIG_FILE_PATH" value="$(arg manipulator_config_file_path)"/>
   <xacro:property name="GZ_CONTROL_CONFIG_PACKAGE" value="$(arg gz_control_config_package)"/>
   <xacro:property name="GZ_CONTROL_CONFIG_FILE_PATH" value="$(arg gz_control_config_file_path)"/>
@@ -143,4 +152,7 @@
   <xacro:sciurus17_left_arm/>
   <xacro:sciurus17_left_hand/>
+  <xacro:unless value="$(arg use_gazebo)">
+    <xacro:sciurus17_ros2_control_settings/>
+  </xacro:unless>
   <xacro:if value="$(arg use_gazebo)">
     <xacro:gazebo_robot_settings/>

Commit message: 設定順序修正

File: urdf/sciurus17.urdf.xacro (robot description, xacro)
@@ -60,6 +60,6 @@
   <xacro:property name="NAME_LINK_GRIPPER_L_B" value="l_gripperB_link"/>
   <xacro:property name="NAME_LINK_ARMARKER_L" value="l_link5_armarker"/>
+  <xacro:property name="NAME_JOINT_BASE" value="base_link_to_world_joint"/>
   <xacro:property name="NAME_JOINT_BODY" value="waist_yaw_joint"/>
-  <xacro:property name="NAME_JOINT_BASE" value="base_link_to_world_joint"/>
   <xacro:property name="NAME_JOINT_NECK_1" value="neck_yaw_joint"/>
   <xacro:property name="NAME_JOINT_NECK_2" value="neck_pitch_joint"/>

Commit message: グリッパのjoint limit調整

File: urdf/sciurus17.urdf.xacro (robot description, xacro)
@@ -112,5 +112,5 @@
   <!-- Gazeboの挙動がlimit付近で不安定なため、limitをサーボの可動範囲より少し大きくする -->
   <!-- 参照: https://github.com/rt-net/sciurus17_description/pull/6 -->
-  <xacro:property name="JOINT_GRIPPER_R_LOWER_LIMIT" value="${radians(-0.01)}"/>
+  <xacro:property name="JOINT_GRIPPER_R_LOWER_LIMIT" value="${radians(-0.05)}"/>
   <xacro:property name="JOINT_GRIPPER_R_UPPER_LIMIT" value="${radians(86)}"/>
   <xacro:property name="JOINT_ARM_L_1_LOWER_LIMIT" value="${radians(-90)}"/>
@@ -133,5 +133,5 @@
   <!-- Gazeboの挙動がlimit付近で不安定なため、limitをサーボの可動範囲より少し大きくする -->
   <!-- 参照: https://github.com/rt-net/sciurus17_description/pull/6 -->
-  <xacro:property name="JOINT_GRIPPER_L_UPPER_LIMIT" value="${radians(0.01)}"/>
+  <xacro:property name="JOINT_GRIPPER_L_UPPER_LIMIT" value="${radians(0.05)}"/>
   <xacro:property name="COLOR_LINK_BASE" value="white"/>
   <xacro:property name="COLOR_LINK_BODY" value="white"/>
