Commit message: カメラ追加

File: urdf/sciurus17.urdf.xacro (robot description, xacro)
@@ -38,6 +38,8 @@
   <xacro:property name="NAME_LINK_NECK_1" value="neck_yaw_link"/>
   <xacro:property name="NAME_LINK_NECK_2" value="neck_pitch_link"/>
-  <xacro:property name="NAME_LINK_HEAD_CAMERA" value="head_camera_link"/>
-  <xacro:property name="NAME_LINK_CHEST_CAMERA" value="chest_camera_link"/>
+  <xacro:property name="NAME_HEAD_CAMERA_PREFIX" value="head_camera"/>
+  <xacro:property name="NAME_CHEST_CAMERA_PREFIX" value="chest_camera"/>
+  <xacro:property name="NAME_LINK_HEAD_CAMERA" value="${NAME_HEAD_CAMERA_PREFIX}_link"/>
+  <xacro:property name="NAME_LINK_CHEST_CAMERA" value="${NAME_CHEST_CAMERA_PREFIX}_link"/>
   <xacro:property name="NAME_LINK_ARM_R_1" value="r_link1"/>
   <xacro:property name="NAME_LINK_ARM_R_2" value="r_link2"/>
@@ -158,4 +160,16 @@
     <xacro:gazebo_robot_settings/>
     <xacro:sciurus17_gazebo_ros2_control_settings/>
+    <joint name="${NAME_HEAD_CAMERA_PREFIX}_color_joint" type="fixed">
+      <origin xyz="0 0.015 0" rpy="0 0 0" />
+      <parent link="${NAME_LINK_HEAD_CAMERA}" />
+      <child link="${NAME_HEAD_CAMERA_PREFIX}_color_frame" />
+    </joint>
+    <link name="${NAME_HEAD_CAMERA_PREFIX}_color_frame"/>
+    <joint name="${NAME_HEAD_CAMERA_PREFIX}_color_optical_joint" type="fixed">
+      <origin xyz="0 0 0" rpy="${radians(-90)} 0 ${radians(-90)}" />
+      <parent link="${NAME_HEAD_CAMERA_PREFIX}_color_frame" />
+      <child link="${NAME_HEAD_CAMERA_PREFIX}_color_optical_frame" />
+    </joint>
+    <link name="${NAME_HEAD_CAMERA_PREFIX}_color_optical_frame"/>
   </xacro:if>
 </robot>

File: urdf/sciurus17_gazebo.xacro (robot description, xacro)
@@ -37,7 +37,4 @@
       <xacro:material_gazebo_white/>
     </gazebo>
-    <gazebo reference="${NAME_LINK_CHEST_CAMERA}">
-      <xacro:material_gazebo_black/>
-    </gazebo>
     <gazebo reference="${NAME_LINK_NECK_1}">
       <xacro:material_gazebo_white/>
@@ -46,6 +43,56 @@
       <xacro:material_gazebo_white/>
     </gazebo>
-    <gazebo reference="${NAME_LINK_HEAD_CAMERA}">
+    <gazebo>
+      <plugin filename="ignition-gazebo-sensors-system" name="ignition::gazebo::systems::Sensors">
+        <render_engine>ogre2</render_engine>
+      </plugin>
+    </gazebo>
+    <gazebo reference="${NAME_HEAD_CAMERA_PREFIX}_color_frame">
       <xacro:material_gazebo_black/>
+      <sensor name="sim_realsense_d415" type="rgbd_camera">
+        <update_rate>10</update_rate>
+        <always_on>true</always_on>
+        <topic>${NAME_HEAD_CAMERA_PREFIX}</topic>
+        <ignition_frame_id>${NAME_HEAD_CAMERA_PREFIX}_color_frame</ignition_frame_id>
+        <camera name="realsense_d415">
+          <horizontal_fov>${radians(69.4)}</horizontal_fov>
+          <image>
+            <width>640</width>
+            <height>360</height>
+          </image>
+          <clip>
+            <near>0.1</near>
+            <far>10.0</far>
+          </clip>
+          <depth_camera>
+            <clip>
+              <near>0.1</near>
+              <far>3.0</far>
+            </clip>
+          </depth_camera>
+          <optical_frame_id>${NAME_HEAD_CAMERA_PREFIX}_color_optical_frame</optical_frame_id>
+        </camera>
+      </sensor>
+    </gazebo>
+    <gazebo reference="${NAME_LINK_CHEST_CAMERA}">
+      <xacro:material_gazebo_black/>
+      <sensor name="${NAME_CHEST_CAMERA_PREFIX}" type="camera">
+        <pose relative_to="${NAME_LINK_CHEST_CAMERA}">0 0 0 ${radians(90)} ${radians(-90)} 0</pose>
+        <update_rate>10</update_rate>
+        <always_on>true</always_on>
+        <topic>${NAME_CHEST_CAMERA_PREFIX}/image_raw</topic>
+        <ignition_frame_id>${NAME_LINK_CHEST_CAMERA}</ignition_frame_id>
+        <camera name="${NAME_CHEST_CAMERA_PREFIX}">
+          <horizontal_fov>${radians(120)}</horizontal_fov>
+          <image>
+            <width>640</width>
+            <height>360</height>
+          </image>
+          <clip>
+            <near>0.1</near>
+            <far>10.0</far>
+          </clip>
+        </camera>
+      </sensor>
     </gazebo>
     <gazebo reference="${NAME_LINK_ARM_R_1}">

Commit message: カメラパラメータ設定

File: urdf/sciurus17.urdf.xacro (robot description, xacro)
@@ -28,4 +28,6 @@
   <xacro:property name="GZ_CONTROL_CONFIG_PACKAGE" value="$(arg gz_control_config_package)"/>
   <xacro:property name="GZ_CONTROL_CONFIG_FILE_PATH" value="$(arg gz_control_config_file_path)"/>
+  <xacro:property name="NAME_HEAD_CAMERA_PREFIX" value="head_camera"/>
+  <xacro:property name="NAME_CHEST_CAMERA_PREFIX" value="chest_camera"/>
   <material name="white">
     <color rgba="0.9 0.9 0.9 1.0"/>
@@ -38,6 +40,4 @@
   <xacro:property name="NAME_LINK_NECK_1" value="neck_yaw_link"/>
   <xacro:property name="NAME_LINK_NECK_2" value="neck_pitch_link"/>
-  <xacro:property name="NAME_HEAD_CAMERA_PREFIX" value="head_camera"/>
-  <xacro:property name="NAME_CHEST_CAMERA_PREFIX" value="chest_camera"/>
   <xacro:property name="NAME_LINK_HEAD_CAMERA" value="${NAME_HEAD_CAMERA_PREFIX}_link"/>
   <xacro:property name="NAME_LINK_CHEST_CAMERA" value="${NAME_CHEST_CAMERA_PREFIX}_link"/>

File: urdf/sciurus17_gazebo.xacro (robot description, xacro)
@@ -56,8 +56,12 @@
         <ignition_frame_id>${NAME_HEAD_CAMERA_PREFIX}_color_frame</ignition_frame_id>
         <camera name="realsense_d415">
-          <horizontal_fov>${radians(69.4)}</horizontal_fov>
+          <xacro:property name="head_camera_width" value="640"/>
+          <xacro:property name="head_camera_height" value="360"/>
+          <xacro:property name="head_camera_hfov" value="${radians(69.4)}"/>
+          <xacro:property name="head_camera_focal_length" value="${head_camera_width / (2 * tan(head_camera_hfov / 2))}"/>
+          <horizontal_fov>${head_camera_hfov}</horizontal_fov>
           <image>
-            <width>640</width>
-            <height>360</height>
+            <width>${head_camera_width}</width>
+            <height>${head_camera_height}</height>
           </image>
           <clip>
@@ -72,4 +76,21 @@
           </depth_camera>
           <optical_frame_id>${NAME_HEAD_CAMERA_PREFIX}_color_optical_frame</optical_frame_id>
+          <lens>
+            <intrinsics>
+              <fx>${head_camera_focal_length}</fx>
+              <fy>${head_camera_focal_length}</fy>
+              <cx>${(head_camera_width + 1) / 2}</cx>
+              <cy>${(head_camera_height + 1) / 2}</cy>
+              <s>1.0</s>
+            </intrinsics>
+            <projection>
+              <p_fx>${head_camera_focal_length}</p_fx>
+              <p_fy>${head_camera_focal_length}</p_fy>
+              <p_cx>${(head_camera_width + 1) / 2}</p_cx>
+              <p_cy>${(head_camera_height + 1) / 2}</p_cy>
+              <tx>0</tx>
+              <ty>0</ty>
+            </projection>
+          </lens>
         </camera>
       </sensor>
@@ -84,8 +105,12 @@
         <ignition_frame_id>${NAME_LINK_CHEST_CAMERA}</ignition_frame_id>
         <camera name="${NAME_CHEST_CAMERA_PREFIX}">
+          <xacro:property name="chest_camera_width" value="640"/>
+          <xacro:property name="chest_camera_height" value="360"/>
+          <xacro:property name="chest_camera_hfov" value="${radians(120)}"/>
+          <xacro:property name="chest_camera_focal_length" value="${chest_camera_width / (2 * tan(chest_camera_hfov / 2))}"/>
           <horizontal_fov>${radians(120)}</horizontal_fov>
           <image>
-            <width>640</width>
-            <height>360</height>
+            <width>${chest_camera_width}</width>
+            <height>${chest_camera_height}</height>
           </image>
           <clip>
@@ -93,4 +118,21 @@
             <far>10.0</far>
           </clip>
+          <lens>
+            <intrinsics>
+              <fx>${chest_camera_focal_length}</fx>
+              <fy>${chest_camera_focal_length}</fy>
+              <cx>${(chest_camera_width + 1) / 2}</cx>
+              <cy>${(chest_camera_height + 1) / 2}</cy>
+              <s>1.0</s>
+            </intrinsics>
+            <projection>
+              <p_fx>${chest_camera_focal_length}</p_fx>
+              <p_fy>${chest_camera_focal_length}</p_fy>
+              <p_cx>${(chest_camera_width + 1) / 2}</p_cx>
+              <p_cy>${(chest_camera_height + 1) / 2}</p_cy>
+              <tx>0</tx>
+              <ty>0</ty>
+            </projection>
+          </lens>
         </camera>
       </sensor>

Commit message: Gazebo上のカメラの有無選択オプション追加

File: urdf/sciurus17.urdf.xacro (robot description, xacro)
@@ -16,4 +16,6 @@
   <xacro:include filename="$(find sciurus17_description)/urdf/sciurus17.gazebo_ros2_control.xacro"/>
   <xacro:arg name="use_gazebo" default="false" />
+  <xacro:arg name="use_head_camera" default="false" />
+  <xacro:arg name="use_chest_camera" default="false" />
   <xacro:arg name="port_name" default="/dev/sciurus17spine" />
   <xacro:arg name="baudrate" default="3000000" />
@@ -22,4 +24,6 @@
   <xacro:arg name="gz_control_config_package" default="" />
   <xacro:arg name="gz_control_config_file_path" default="" />
+  <xacro:property name="USE_HEAD_CAMERA" value="$(arg use_head_camera)"/>
+  <xacro:property name="USE_CHEST_CAMERA" value="$(arg use_chest_camera)"/>
   <xacro:property name="PORT_NAME" value="$(arg port_name)"/>
   <xacro:property name="BAUDRATE" value="$(arg baudrate)"/>

File: urdf/sciurus17_gazebo.xacro (robot description, xacro)
@@ -50,91 +50,95 @@
     <gazebo reference="${NAME_HEAD_CAMERA_PREFIX}_color_frame">
       <xacro:material_gazebo_black/>
-      <sensor name="sim_realsense_d415" type="rgbd_camera">
-        <update_rate>10</update_rate>
-        <always_on>true</always_on>
-        <topic>${NAME_HEAD_CAMERA_PREFIX}</topic>
-        <ignition_frame_id>${NAME_HEAD_CAMERA_PREFIX}_color_frame</ignition_frame_id>
-        <camera name="realsense_d415">
-          <xacro:property name="head_camera_width" value="640"/>
-          <xacro:property name="head_camera_height" value="360"/>
-          <xacro:property name="head_camera_hfov" value="${radians(69.4)}"/>
-          <xacro:property name="head_camera_focal_length" value="${head_camera_width / (2 * tan(head_camera_hfov / 2))}"/>
-          <horizontal_fov>${head_camera_hfov}</horizontal_fov>
-          <image>
-            <width>${head_camera_width}</width>
-            <height>${head_camera_height}</height>
-          </image>
-          <clip>
-            <near>0.1</near>
-            <far>10.0</far>
-          </clip>
-          <depth_camera>
+      <xacro:if value="${USE_HEAD_CAMERA}">
+        <sensor name="sim_realsense_d415" type="rgbd_camera">
+          <update_rate>10</update_rate>
+          <always_on>true</always_on>
+          <topic>${NAME_HEAD_CAMERA_PREFIX}</topic>
+          <ignition_frame_id>${NAME_HEAD_CAMERA_PREFIX}_color_frame</ignition_frame_id>
+          <camera name="realsense_d415">
+            <xacro:property name="head_camera_width" value="640"/>
+            <xacro:property name="head_camera_height" value="360"/>
+            <xacro:property name="head_camera_hfov" value="${radians(69.4)}"/>
+            <xacro:property name="head_camera_focal_length" value="${head_camera_width / (2 * tan(head_camera_hfov / 2))}"/>
+            <horizontal_fov>${head_camera_hfov}</horizontal_fov>
+            <image>
+              <width>${head_camera_width}</width>
+              <height>${head_camera_height}</height>
+            </image>
             <clip>
               <near>0.1</near>
-              <far>3.0</far>
+              <far>10.0</far>
             </clip>
-          </depth_camera>
-          <optical_frame_id>${NAME_HEAD_CAMERA_PREFIX}_color_optical_frame</optical_frame_id>
-          <lens>
-            <intrinsics>
-              <fx>${head_camera_focal_length}</fx>
-              <fy>${head_camera_focal_length}</fy>
-              <cx>${(head_camera_width + 1) / 2}</cx>
-              <cy>${(head_camera_height + 1) / 2}</cy>
-              <s>1.0</s>
-            </intrinsics>
-            <projection>
-              <p_fx>${head_camera_focal_length}</p_fx>
-              <p_fy>${head_camera_focal_length}</p_fy>
-              <p_cx>${(head_camera_width + 1) / 2}</p_cx>
-              <p_cy>${(head_camera_height + 1) / 2}</p_cy>
-              <tx>0</tx>
-              <ty>0</ty>
-            </projection>
-          </lens>
-        </camera>
-      </sensor>
+            <depth_camera>
+              <clip>
+                <near>0.1</near>
+                <far>3.0</far>
+              </clip>
+            </depth_camera>
+            <optical_frame_id>${NAME_HEAD_CAMERA_PREFIX}_color_optical_frame</optical_frame_id>
+            <lens>
+              <intrinsics>
+                <fx>${head_camera_focal_length}</fx>
+                <fy>${head_camera_focal_length}</fy>
+                <cx>${(head_camera_width + 1) / 2}</cx>
+                <cy>${(head_camera_height + 1) / 2}</cy>
+                <s>1.0</s>
+              </intrinsics>
+              <projection>
+                <p_fx>${head_camera_focal_length}</p_fx>
+                <p_fy>${head_camera_focal_length}</p_fy>
+                <p_cx>${(head_camera_width + 1) / 2}</p_cx>
+                <p_cy>${(head_camera_height + 1) / 2}</p_cy>
+                <tx>0</tx>
+                <ty>0</ty>
+              </projection>
+            </lens>
+          </camera>
+        </sensor>
+      </xacro:if>
     </gazebo>
     <gazebo reference="${NAME_LINK_CHEST_CAMERA}">
       <xacro:material_gazebo_black/>
-      <sensor name="${NAME_CHEST_CAMERA_PREFIX}" type="camera">
-        <pose relative_to="${NAME_LINK_CHEST_CAMERA}">0 0 0 ${radians(90)} ${radians(-90)} 0</pose>
-        <update_rate>10</update_rate>
-        <always_on>true</always_on>
-        <topic>${NAME_CHEST_CAMERA_PREFIX}/image_raw</topic>
-        <ignition_frame_id>${NAME_LINK_CHEST_CAMERA}</ignition_frame_id>
-        <camera name="${NAME_CHEST_CAMERA_PREFIX}">
-          <xacro:property name="chest_camera_width" value="640"/>
-          <xacro:property name="chest_camera_height" value="360"/>
-          <xacro:property name="chest_camera_hfov" value="${radians(120)}"/>
-          <xacro:property name="chest_camera_focal_length" value="${chest_camera_width / (2 * tan(chest_camera_hfov / 2))}"/>
-          <horizontal_fov>${radians(120)}</horizontal_fov>
-          <image>
-            <width>${chest_camera_width}</width>
-            <height>${chest_camera_height}</height>
-          </image>
-          <clip>
-            <near>0.1</near>
-            <far>10.0</far>
-          </clip>
-          <lens>
-            <intrinsics>
-              <fx>${chest_camera_focal_length}</fx>
-              <fy>${chest_camera_focal_length}</fy>
-              <cx>${(chest_camera_width + 1) / 2}</cx>
-              <cy>${(chest_camera_height + 1) / 2}</cy>
-              <s>1.0</s>
-            </intrinsics>
-            <projection>
-              <p_fx>${chest_camera_focal_length}</p_fx>
-              <p_fy>${chest_camera_focal_length}</p_fy>
-              <p_cx>${(chest_camera_width + 1) / 2}</p_cx>
-              <p_cy>${(chest_camera_height + 1) / 2}</p_cy>
-              <tx>0</tx>
-              <ty>0</ty>
-            </projection>
-          </lens>
-        </camera>
-      </sensor>
+      <xacro:if value="${USE_CHEST_CAMERA}">
+        <sensor name="${NAME_CHEST_CAMERA_PREFIX}" type="camera">
+          <pose relative_to="${NAME_LINK_CHEST_CAMERA}">0 0 0 ${radians(90)} ${radians(-90)} 0</pose>
+          <update_rate>10</update_rate>
+          <always_on>true</always_on>
+          <topic>${NAME_CHEST_CAMERA_PREFIX}/image_raw</topic>
+          <ignition_frame_id>${NAME_LINK_CHEST_CAMERA}</ignition_frame_id>
+          <camera name="${NAME_CHEST_CAMERA_PREFIX}">
+            <xacro:property name="chest_camera_width" value="640"/>
+            <xacro:property name="chest_camera_height" value="360"/>
+            <xacro:property name="chest_camera_hfov" value="${radians(120)}"/>
+            <xacro:property name="chest_camera_focal_length" value="${chest_camera_width / (2 * tan(chest_camera_hfov / 2))}"/>
+            <horizontal_fov>${radians(120)}</horizontal_fov>
+            <image>
+              <width>${chest_camera_width}</width>
+              <height>${chest_camera_height}</height>
+            </image>
+            <clip>
+              <near>0.1</near>
+              <far>10.0</far>
+            </clip>
+            <lens>
+              <intrinsics>
+                <fx>${chest_camera_focal_length}</fx>
+                <fy>${chest_camera_focal_length}</fy>
+                <cx>${(chest_camera_width + 1) / 2}</cx>
+                <cy>${(chest_camera_height + 1) / 2}</cy>
+                <s>1.0</s>
+              </intrinsics>
+              <projection>
+                <p_fx>${chest_camera_focal_length}</p_fx>
+                <p_fy>${chest_camera_focal_length}</p_fy>
+                <p_cx>${(chest_camera_width + 1) / 2}</p_cx>
+                <p_cy>${(chest_camera_height + 1) / 2}</p_cy>
+                <tx>0</tx>
+                <ty>0</ty>
+              </projection>
+            </lens>
+          </camera>
+        </sensor>
+      </xacro:if>
     </gazebo>
     <gazebo reference="${NAME_LINK_ARM_R_1}">

Commit message: camera_link上の円柱モデルを削除

File: urdf/sciurus17.urdf.xacro (robot description, xacro)
@@ -145,5 +145,4 @@
   <xacro:property name="COLOR_LINK_ARM" value="white"/>
   <xacro:property name="COLOR_LINK_GRIPPER" value="red"/>
-  <xacro:property name="COLOR_LINK_CAMERA" value="white"/>
   <!-- Used for fixing robot 'base_link'  to Gazebo 'world' -->
   <link name="world"/>

File: urdf/sciurus17_body.xacro (robot description, xacro)
@@ -57,19 +57,5 @@
       <origin xyz="0.114576 0.0 0.217659" rpy="-2.7925268032 0 -1.5707963268"/>
     </joint>
-    <link name="${NAME_LINK_CHEST_CAMERA}">
-      <visual>
-        <origin xyz="0 0 0" rpy="0 0 0"/>
-        <geometry>
-          <cylinder length="0.002" radius="0.003"/>
-        </geometry>
-        <material name="${COLOR_LINK_CAMERA}"/>
-      </visual>
-      <collision>
-        <origin xyz="0.0 0.0 0.0" rpy="0 0 0"/>
-        <geometry>
-          <cylinder length="0.002" radius="0.003"/>
-        </geometry>
-      </collision>
-    </link>
+    <link name="${NAME_LINK_CHEST_CAMERA}"/>
   </xacro:macro>
 </robot>

File: urdf/sciurus17_gazebo.xacro (robot description, xacro)
@@ -49,5 +49,4 @@
     </gazebo>
     <gazebo reference="${NAME_HEAD_CAMERA_PREFIX}_color_frame">
-      <xacro:material_gazebo_black/>
       <xacro:if value="${USE_HEAD_CAMERA}">
         <sensor name="sim_realsense_d415" type="rgbd_camera">
@@ -99,5 +98,4 @@
     </gazebo>
     <gazebo reference="${NAME_LINK_CHEST_CAMERA}">
-      <xacro:material_gazebo_black/>
       <xacro:if value="${USE_CHEST_CAMERA}">
         <sensor name="${NAME_CHEST_CAMERA_PREFIX}" type="camera">

File: urdf/sciurus17_head.xacro (robot description, xacro)
@@ -69,19 +69,5 @@
       <origin xyz="0.081785 0.020 0.091" rpy="0 0 0"/>
     </joint>
-    <link name="${NAME_LINK_HEAD_CAMERA}">
-      <visual>
-        <origin xyz="0 0 0" rpy="0 0 0"/>
-        <geometry>
-          <cylinder length="0.002" radius="0.003"/>
-        </geometry>
-        <material name="${COLOR_LINK_CAMERA}"/>
-      </visual>
-      <collision>
-        <origin xyz="0.0 0.0 0.0" rpy="0 0 0"/>
-        <geometry>
-          <cylinder length="0.002" radius="0.003"/>
-        </geometry>
-      </collision>
-    </link>
+    <link name="${NAME_LINK_HEAD_CAMERA}"/>
   </xacro:macro>
 </robot>

Commit message: use_head_cameraオプションをuse_gazebo_head_cameraに変更

File: urdf/sciurus17.urdf.xacro (robot description, xacro)
@@ -16,6 +16,6 @@
   <xacro:include filename="$(find sciurus17_description)/urdf/sciurus17.gazebo_ros2_control.xacro"/>
   <xacro:arg name="use_gazebo" default="false" />
-  <xacro:arg name="use_head_camera" default="false" />
-  <xacro:arg name="use_chest_camera" default="false" />
+  <xacro:arg name="use_gazebo_head_camera" default="false" />
+  <xacro:arg name="use_gazebo_chest_camera" default="false" />
   <xacro:arg name="port_name" default="/dev/sciurus17spine" />
   <xacro:arg name="baudrate" default="3000000" />
@@ -24,6 +24,6 @@
   <xacro:arg name="gz_control_config_package" default="" />
   <xacro:arg name="gz_control_config_file_path" default="" />
-  <xacro:property name="USE_HEAD_CAMERA" value="$(arg use_head_camera)"/>
-  <xacro:property name="USE_CHEST_CAMERA" value="$(arg use_chest_camera)"/>
+  <xacro:property name="USE_GAZEBO_HEAD_CAMERA" value="$(arg use_gazebo_head_camera)"/>
+  <xacro:property name="USE_GAZEBO_CHEST_CAMERA" value="$(arg use_gazebo_chest_camera)"/>
   <xacro:property name="PORT_NAME" value="$(arg port_name)"/>
   <xacro:property name="BAUDRATE" value="$(arg baudrate)"/>

File: urdf/sciurus17_gazebo.xacro (robot description, xacro)
@@ -48,5 +48,5 @@
       </plugin>
     </gazebo>
-    <xacro:if value="${USE_HEAD_CAMERA}">
+    <xacro:if value="${USE_GAZEBO_HEAD_CAMERA}">
       <gazebo reference="${NAME_HEAD_CAMERA_PREFIX}_color_frame">
         <sensor name="sim_realsense_d415" type="rgbd_camera">
@@ -97,5 +97,5 @@
       </gazebo>
     </xacro:if>
-    <xacro:if value="${USE_CHEST_CAMERA}">
+    <xacro:if value="${USE_GAZEBO_CHEST_CAMERA}">
       <gazebo reference="${NAME_LINK_CHEST_CAMERA}">
         <sensor name="${NAME_CHEST_CAMERA_PREFIX}" type="camera">
