Commit message: Gazebo上の機体にカメラを追加 (#13)
* カメラ追加

* カメラパラメータ設定

* Gazebo上のカメラの有無選択オプション追加

* camera_link上の円柱モデルを削除

* use_head_cameraのtest追加

* スタイル修正

* テスト修正

* スタイル修正

* 胸カメラ画角修正

Co-authored-by: Shota Aoki <macakasit@gmail.com>

* use_head_cameraオプションをuse_gazebo_head_cameraに変更

---------

Co-authored-by: Shota Aoki <macakasit@gmail.com>

File: urdf/sciurus17.urdf.xacro (robot description, xacro)
@@ -16,4 +16,6 @@
   <xacro:include filename="$(find sciurus17_description)/urdf/sciurus17.gazebo_ros2_control.xacro"/>
   <xacro:arg name="use_gazebo" default="false" />
+  <xacro:arg name="use_gazebo_head_camera" default="false" />
+  <xacro:arg name="use_gazebo_chest_camera" default="false" />
   <xacro:arg name="port_name" default="/dev/sciurus17spine" />
   <xacro:arg name="baudrate" default="3000000" />
@@ -22,4 +24,6 @@
   <xacro:arg name="gz_control_config_package" default="" />
   <xacro:arg name="gz_control_config_file_path" default="" />
+  <xacro:property name="USE_GAZEBO_HEAD_CAMERA" value="$(arg use_gazebo_head_camera)"/>
+  <xacro:property name="USE_GAZEBO_CHEST_CAMERA" value="$(arg use_gazebo_chest_camera)"/>
   <xacro:property name="PORT_NAME" value="$(arg port_name)"/>
   <xacro:property name="BAUDRATE" value="$(arg baudrate)"/>
@@ -28,4 +32,6 @@
   <xacro:property name="GZ_CONTROL_CONFIG_PACKAGE" value="$(arg gz_control_config_package)"/>
   <xacro:property name="GZ_CONTROL_CONFIG_FILE_PATH" value="$(arg gz_control_config_file_path)"/>
+  <xacro:property name="NAME_HEAD_CAMERA_PREFIX" value="head_camera"/>
+  <xacro:property name="NAME_CHEST_CAMERA_PREFIX" value="chest_camera"/>
   <material name="white">
     <color rgba="0.9 0.9 0.9 1.0"/>
@@ -38,6 +44,6 @@
   <xacro:property name="NAME_LINK_NECK_1" value="neck_yaw_link"/>
   <xacro:property name="NAME_LINK_NECK_2" value="neck_pitch_link"/>
-  <xacro:property name="NAME_LINK_HEAD_CAMERA" value="head_camera_link"/>
-  <xacro:property name="NAME_LINK_CHEST_CAMERA" value="chest_camera_link"/>
+  <xacro:property name="NAME_LINK_HEAD_CAMERA" value="${NAME_HEAD_CAMERA_PREFIX}_link"/>
+  <xacro:property name="NAME_LINK_CHEST_CAMERA" value="${NAME_CHEST_CAMERA_PREFIX}_link"/>
   <xacro:property name="NAME_LINK_ARM_R_1" value="r_link1"/>
   <xacro:property name="NAME_LINK_ARM_R_2" value="r_link2"/>
@@ -139,5 +145,4 @@
   <xacro:property name="COLOR_LINK_ARM" value="white"/>
   <xacro:property name="COLOR_LINK_GRIPPER" value="red"/>
-  <xacro:property name="COLOR_LINK_CAMERA" value="white"/>
   <!-- Used for fixing robot 'base_link'  to Gazebo 'world' -->
   <link name="world"/>
@@ -158,4 +163,16 @@
     <xacro:gazebo_robot_settings/>
     <xacro:sciurus17_gazebo_ros2_control_settings/>
+    <joint name="${NAME_HEAD_CAMERA_PREFIX}_color_joint" type="fixed">
+      <origin xyz="0 0.015 0" rpy="0 0 0" />
+      <parent link="${NAME_LINK_HEAD_CAMERA}" />
+      <child link="${NAME_HEAD_CAMERA_PREFIX}_color_frame" />
+    </joint>
+    <link name="${NAME_HEAD_CAMERA_PREFIX}_color_frame"/>
+    <joint name="${NAME_HEAD_CAMERA_PREFIX}_color_optical_joint" type="fixed">
+      <origin xyz="0 0 0" rpy="${radians(-90)} 0 ${radians(-90)}" />
+      <parent link="${NAME_HEAD_CAMERA_PREFIX}_color_frame" />
+      <child link="${NAME_HEAD_CAMERA_PREFIX}_color_optical_frame" />
+    </joint>
+    <link name="${NAME_HEAD_CAMERA_PREFIX}_color_optical_frame"/>
   </xacro:if>
 </robot>

File: urdf/sciurus17_gazebo.xacro (robot description, xacro)
@@ -37,7 +37,4 @@
       <xacro:material_gazebo_white/>
     </gazebo>
-    <gazebo reference="${NAME_LINK_CHEST_CAMERA}">
-      <xacro:material_gazebo_black/>
-    </gazebo>
     <gazebo reference="${NAME_LINK_NECK_1}">
       <xacro:material_gazebo_white/>
@@ -46,7 +43,101 @@
       <xacro:material_gazebo_white/>
     </gazebo>
-    <gazebo reference="${NAME_LINK_HEAD_CAMERA}">
-      <xacro:material_gazebo_black/>
-    </gazebo>
+    <gazebo>
+      <plugin filename="ignition-gazebo-sensors-system" name="ignition::gazebo::systems::Sensors">
+        <render_engine>ogre2</render_engine>
+      </plugin>
+    </gazebo>
+    <xacro:if value="${USE_GAZEBO_HEAD_CAMERA}">
+      <gazebo reference="${NAME_HEAD_CAMERA_PREFIX}_color_frame">
+        <sensor name="sim_realsense_d415" type="rgbd_camera">
+          <update_rate>10</update_rate>
+          <always_on>true</always_on>
+          <topic>${NAME_HEAD_CAMERA_PREFIX}</topic>
+          <ignition_frame_id>${NAME_HEAD_CAMERA_PREFIX}_color_frame</ignition_frame_id>
+          <camera name="realsense_d415">
+            <xacro:property name="head_camera_width" value="640"/>
+            <xacro:property name="head_camera_height" value="360"/>
+            <xacro:property name="head_camera_hfov" value="${radians(69.4)}"/>
+            <xacro:property name="head_camera_focal_length" value="${head_camera_width / (2 * tan(head_camera_hfov / 2))}"/>
+            <horizontal_fov>${head_camera_hfov}</horizontal_fov>
+            <image>
+              <width>${head_camera_width}</width>
+              <height>${head_camera_height}</height>
+            </image>
+            <clip>
+              <near>0.1</near>
+              <far>10.0</far>
+            </clip>
+            <depth_camera>
+              <clip>
+                <near>0.1</near>
+                <far>3.0</far>
+              </clip>
+            </depth_camera>
+            <optical_frame_id>${NAME_HEAD_CAMERA_PREFIX}_color_optical_frame</optical_frame_id>
+            <lens>
+              <intrinsics>
+                <fx>${head_camera_focal_length}</fx>
+                <fy>${head_camera_focal_length}</fy>
+                <cx>${(head_camera_width + 1) / 2}</cx>
+                <cy>${(head_camera_height + 1) / 2}</cy>
+                <s>1.0</s>
+              </intrinsics>
+              <projection>
+                <p_fx>${head_camera_focal_length}</p_fx>
+                <p_fy>${head_camera_focal_length}</p_fy>
+                <p_cx>${(head_camera_width + 1) / 2}</p_cx>
+                <p_cy>${(head_camera_height + 1) / 2}</p_cy>
+                <tx>0</tx>
+                <ty>0</ty>
+              </projection>
+            </lens>
+          </camera>
+        </sensor>
+      </gazebo>
+    </xacro:if>
+    <xacro:if value="${USE_GAZEBO_CHEST_CAMERA}">
+      <gazebo reference="${NAME_LINK_CHEST_CAMERA}">
+        <sensor name="${NAME_CHEST_CAMERA_PREFIX}" type="camera">
+          <pose relative_to="${NAME_LINK_CHEST_CAMERA}">0 0 0 ${radians(90)} ${radians(-90)} 0</pose>
+          <update_rate>10</update_rate>
+          <always_on>true</always_on>
+          <topic>${NAME_CHEST_CAMERA_PREFIX}/image_raw</topic>
+          <ignition_frame_id>${NAME_LINK_CHEST_CAMERA}</ignition_frame_id>
+          <camera name="${NAME_CHEST_CAMERA_PREFIX}">
+            <xacro:property name="chest_camera_width" value="640"/>
+            <xacro:property name="chest_camera_height" value="360"/>
+            <xacro:property name="chest_camera_hfov" value="${radians(120)}"/>
+            <xacro:property name="chest_camera_focal_length" value="${chest_camera_width / (2 * tan(chest_camera_hfov / 2))}"/>
+            <horizontal_fov>${chest_camera_hfov}</horizontal_fov>
+            <image>
+              <width>${chest_camera_width}</width>
+              <height>${chest_camera_height}</height>
+            </image>
+            <clip>
+              <near>0.1</near>
+              <far>10.0</far>
+            </clip>
+            <lens>
+              <intrinsics>
+                <fx>${chest_camera_focal_length}</fx>
+                <fy>${chest_camera_focal_length}</fy>
+                <cx>${(chest_camera_width + 1) / 2}</cx>
+                <cy>${(chest_camera_height + 1) / 2}</cy>
+                <s>1.0</s>
+              </intrinsics>
+              <projection>
+                <p_fx>${chest_camera_focal_length}</p_fx>
+                <p_fy>${chest_camera_focal_length}</p_fy>
+                <p_cx>${(chest_camera_width + 1) / 2}</p_cx>
+                <p_cy>${(chest_camera_height + 1) / 2}</p_cy>
+                <tx>0</tx>
+                <ty>0</ty>
+              </projection>
+            </lens>
+          </camera>
+        </sensor>
+      </gazebo>
+    </xacro:if>
     <gazebo reference="${NAME_LINK_ARM_R_1}">
       <xacro:material_gazebo_white/>

Commit message: プランニングできるように可動範囲を微調整

File: urdf/sciurus17.urdf.xacro (robot description, xacro)
@@ -102,5 +102,6 @@
   <xacro:property name="JOINT_ARM_R_1_LOWER_LIMIT" value="${radians(-90)}"/>
   <xacro:property name="JOINT_ARM_R_1_UPPER_LIMIT" value="${radians(90)}"/>
-  <xacro:property name="JOINT_ARM_R_2_LOWER_LIMIT" value="${radians(-90)}"/>
+  <!-- 初期角度が範囲外だとプランニングで失敗するため範囲を広げる -->
+  <xacro:property name="JOINT_ARM_R_2_LOWER_LIMIT" value="${radians(-92)}"/>
   <xacro:property name="JOINT_ARM_R_2_UPPER_LIMIT" value="${radians(0)}"/>
   <xacro:property name="JOINT_ARM_R_3_LOWER_LIMIT" value="${radians(-90)}"/>
@@ -122,6 +123,7 @@
   <xacro:property name="JOINT_ARM_L_1_LOWER_LIMIT" value="${radians(-90)}"/>
   <xacro:property name="JOINT_ARM_L_1_UPPER_LIMIT" value="${radians(90)}"/>
+  <!-- 初期角度が範囲外だとプランニングで失敗するため範囲を広げる -->
   <xacro:property name="JOINT_ARM_L_2_LOWER_LIMIT" value="${radians(0)}"/>
-  <xacro:property name="JOINT_ARM_L_2_UPPER_LIMIT" value="${radians(90)}"/>
+  <xacro:property name="JOINT_ARM_L_2_UPPER_LIMIT" value="${radians(92)}"/>
   <xacro:property name="JOINT_ARM_L_3_LOWER_LIMIT" value="${radians(-90)}"/>
   <xacro:property name="JOINT_ARM_L_3_UPPER_LIMIT" value="${radians(90)}"/>

Commit message: 手首の可動範囲を広げる

File: urdf/sciurus17.urdf.xacro (robot description, xacro)
@@ -113,5 +113,6 @@
   <xacro:property name="JOINT_ARM_R_5_LOWER_LIMIT" value="${radians(-90)}"/>
   <xacro:property name="JOINT_ARM_R_5_UPPER_LIMIT" value="${radians(90)}"/>
-  <xacro:property name="JOINT_ARM_R_6_LOWER_LIMIT" value="${radians(-120)}"/>
+  <!-- 初期角度が範囲外だとプランニングで失敗するため範囲を広げる -->
+  <xacro:property name="JOINT_ARM_R_6_LOWER_LIMIT" value="${radians(-123)}"/>
   <xacro:property name="JOINT_ARM_R_6_UPPER_LIMIT" value="${radians(60)}"/>
   <xacro:property name="JOINT_ARM_R_7_LOWER_LIMIT" value="${radians(-170)}"/>
@@ -135,5 +136,6 @@
   <xacro:property name="JOINT_ARM_L_5_UPPER_LIMIT" value="${radians(90)}"/>
   <xacro:property name="JOINT_ARM_L_6_LOWER_LIMIT" value="${radians(-60)}"/>
-  <xacro:property name="JOINT_ARM_L_6_UPPER_LIMIT" value="${radians(120)}"/>
+  <!-- 初期角度が範囲外だとプランニングで失敗するため範囲を広げる -->
+  <xacro:property name="JOINT_ARM_L_6_UPPER_LIMIT" value="${radians(123)}"/>
   <xacro:property name="JOINT_ARM_L_7_LOWER_LIMIT" value="${radians(-170)}"/>
   <xacro:property name="JOINT_ARM_L_7_UPPER_LIMIT" value="${radians(170)}"/>
