Commit message: Add new branch dev/sciurus_lift

File: urdf/sciurus17.urdf.xacro (robot description, xacro)
@@ -15,25 +15,6 @@
   <xacro:include filename="$(find sciurus17_description)/urdf/sciurus17_gazebo.xacro"/>
   <xacro:include filename="$(find sciurus17_description)/urdf/sciurus17.gazebo_ros2_control.xacro"/>
-  <xacro:arg name="use_gazebo" default="false" />
-  <xacro:arg name="use_gazebo_head_camera" default="false" />
-  <xacro:arg name="use_gazebo_chest_camera" default="false" />
-  <xacro:arg name="use_mock_components" default="false" />
-  <xacro:arg name="port_name" default="/dev/sciurus17spine" />
-  <xacro:arg name="baudrate" default="3000000" />
-  <xacro:arg name="timeout_seconds" default="1.0" />
-  <xacro:arg name="manipulator_config_file_path" default="" />
-  <xacro:arg name="gz_control_config_package" default="" />
-  <xacro:arg name="gz_control_config_file_path" default="" />
-  <xacro:property name="USE_GAZEBO_HEAD_CAMERA" value="$(arg use_gazebo_head_camera)"/>
-  <xacro:property name="USE_GAZEBO_CHEST_CAMERA" value="$(arg use_gazebo_chest_camera)"/>
-  <xacro:property name="USE_MOCK_COMPONENTS" value="$(arg use_mock_components)"/>
-  <xacro:property name="PORT_NAME" value="$(arg port_name)"/>
-  <xacro:property name="BAUDRATE" value="$(arg baudrate)"/>
-  <xacro:property name="TIMEOUT_SECONDS" value="$(arg timeout_seconds)"/>
-  <xacro:property name="MANIPULATOR_CONFIG_FILE_PATH" value="$(arg manipulator_config_file_path)"/>
-  <xacro:property name="GZ_CONTROL_CONFIG_PACKAGE" value="$(arg gz_control_config_package)"/>
-  <xacro:property name="GZ_CONTROL_CONFIG_FILE_PATH" value="$(arg gz_control_config_file_path)"/>
-  <xacro:property name="NAME_HEAD_CAMERA_PREFIX" value="head_camera"/>
-  <xacro:property name="NAME_CHEST_CAMERA_PREFIX" value="chest_camera"/>
+  <xacro:property name="ROBOT_NAME" value="sciurus17"/>
+  <xacro:include filename="$(find sciurus17_description)/urdf/sciurus17.params.xacro"/>
   <material name="white">
     <color rgba="0.9 0.9 0.9 1.0"/>
@@ -42,108 +23,4 @@
     <color rgba="0.8984375 0.0 0.0703125 1"/>
   </material>
-  <xacro:property name="NAME_LINK_BASE" value="base_link"/>
-  <xacro:property name="NAME_LINK_BODY" value="body_link"/>
-  <xacro:property name="NAME_LINK_NECK_1" value="neck_yaw_link"/>
-  <xacro:property name="NAME_LINK_NECK_2" value="neck_pitch_link"/>
-  <xacro:property name="NAME_LINK_HEAD_CAMERA" value="${NAME_HEAD_CAMERA_PREFIX}_link"/>
-  <xacro:property name="NAME_LINK_CHEST_CAMERA" value="${NAME_CHEST_CAMERA_PREFIX}_link"/>
-  <xacro:property name="NAME_LINK_ARM_R_1" value="r_link1"/>
-  <xacro:property name="NAME_LINK_ARM_R_2" value="r_link2"/>
-  <xacro:property name="NAME_LINK_ARM_R_3" value="r_link3"/>
-  <xacro:property name="NAME_LINK_ARM_R_4" value="r_link4"/>
-  <xacro:property name="NAME_LINK_ARM_R_5" value="r_link5"/>
-  <xacro:property name="NAME_LINK_ARM_R_6" value="r_link6"/>
-  <xacro:property name="NAME_LINK_ARM_R_7" value="r_link7"/>
-  <xacro:property name="NAME_LINK_GRIPPER_R_A" value="r_gripperA_link"/>
-  <xacro:property name="NAME_LINK_GRIPPER_R_B" value="r_gripperB_link"/>
-  <xacro:property name="NAME_LINK_ARMARKER_R" value="r_link5_armarker"/>
-  <xacro:property name="NAME_LINK_ARM_L_1" value="l_link1"/>
-  <xacro:property name="NAME_LINK_ARM_L_2" value="l_link2"/>
-  <xacro:property name="NAME_LINK_ARM_L_3" value="l_link3"/>
-  <xacro:property name="NAME_LINK_ARM_L_4" value="l_link4"/>
-  <xacro:property name="NAME_LINK_ARM_L_5" value="l_link5"/>
-  <xacro:property name="NAME_LINK_ARM_L_6" value="l_link6"/>
-  <xacro:property name="NAME_LINK_ARM_L_7" value="l_link7"/>
-  <xacro:property name="NAME_LINK_GRIPPER_L_A" value="l_gripperA_link"/>
-  <xacro:property name="NAME_LINK_GRIPPER_L_B" value="l_gripperB_link"/>
-  <xacro:property name="NAME_LINK_ARMARKER_L" value="l_link5_armarker"/>
-  <xacro:property name="NAME_JOINT_BASE" value="base_link_to_world_joint"/>
-  <xacro:property name="NAME_JOINT_BODY" value="waist_yaw_joint"/>
-  <xacro:property name="NAME_JOINT_NECK_1" value="neck_yaw_joint"/>
-  <xacro:property name="NAME_JOINT_NECK_2" value="neck_pitch_joint"/>
-  <xacro:property name="NAME_JOINT_HEAD_CAMERA" value="head_camera_joint"/>
-  <xacro:property name="NAME_JOINT_CHEST_CAMERA" value="chest_camera_joint"/>
-  <xacro:property name="NAME_JOINT_ARM_R_1" value="r_arm_joint1"/>
-  <xacro:property name="NAME_JOINT_ARM_R_2" value="r_arm_joint2"/>
-  <xacro:property name="NAME_JOINT_ARM_R_3" value="r_arm_joint3"/>
-  <xacro:property name="NAME_JOINT_ARM_R_4" value="r_arm_joint4"/>
-  <xacro:property name="NAME_JOINT_ARM_R_5" value="r_arm_joint5"/>
-  <xacro:property name="NAME_JOINT_ARM_R_6" value="r_arm_joint6"/>
-  <xacro:property name="NAME_JOINT_ARM_R_7" value="r_arm_joint7"/>
-  <xacro:property name="NAME_JOINT_GRIPPER_R_A" value="r_gripper_joint"/>
-  <xacro:property name="NAME_JOINT_GRIPPER_R_B" value="r_gripper_mimic_joint"/>
-  <xacro:property name="NAME_JOINT_ARMARKER_R" value="r_arm_armarker"/>
-  <xacro:property name="NAME_JOINT_ARM_L_1" value="l_arm_joint1"/>
-  <xacro:property name="NAME_JOINT_ARM_L_2" value="l_arm_joint2"/>
-  <xacro:property name="NAME_JOINT_ARM_L_3" value="l_arm_joint3"/>
-  <xacro:property name="NAME_JOINT_ARM_L_4" value="l_arm_joint4"/>
-  <xacro:property name="NAME_JOINT_ARM_L_5" value="l_arm_joint5"/>
-  <xacro:property name="NAME_JOINT_ARM_L_6" value="l_arm_joint6"/>
-  <xacro:property name="NAME_JOINT_ARM_L_7" value="l_arm_joint7"/>
-  <xacro:property name="NAME_JOINT_GRIPPER_L_A" value="l_gripper_joint"/>
-  <xacro:property name="NAME_JOINT_GRIPPER_L_B" value="l_gripper_mimic_joint"/>
-  <xacro:property name="NAME_JOINT_ARMARKER_L" value="l_arm_armarker"/>
-  <xacro:property name="EFFORT_LIMIT" value="4.0"/>
-  <xacro:property name="VELOCITY_LIMIT" value="5.969211435"/>
-  <xacro:property name="JOINT_BODY_LOWER_LIMIT" value="${radians(-110)}"/>
-  <xacro:property name="JOINT_BODY_UPPER_LIMIT" value="${radians(110)}"/>
-  <xacro:property name="JOINT_NECK_1_LOWER_LIMIT" value="${radians(-165)}"/>
-  <xacro:property name="JOINT_NECK_1_UPPER_LIMIT" value="${radians(165)}"/>
-  <xacro:property name="JOINT_NECK_2_LOWER_LIMIT" value="${radians(-90)}"/>
-  <xacro:property name="JOINT_NECK_2_UPPER_LIMIT" value="${radians(55)}"/>
-  <xacro:property name="JOINT_ARM_R_1_LOWER_LIMIT" value="${radians(-90)}"/>
-  <xacro:property name="JOINT_ARM_R_1_UPPER_LIMIT" value="${radians(90)}"/>
-  <!-- 初期角度が範囲外だとプランニングで失敗するため範囲を広げる -->
-  <xacro:property name="JOINT_ARM_R_2_LOWER_LIMIT" value="${radians(-92)}"/>
-  <xacro:property name="JOINT_ARM_R_2_UPPER_LIMIT" value="${radians(0)}"/>
-  <xacro:property name="JOINT_ARM_R_3_LOWER_LIMIT" value="${radians(-90)}"/>
-  <xacro:property name="JOINT_ARM_R_3_UPPER_LIMIT" value="${radians(90)}"/>
-  <!-- Gazeboの挙動がlimit付近で不安定なため、limitをサーボの可動範囲より少し大きくする -->
-  <!-- 参照: https://github.com/rt-net/sciurus17_description/pull/6 -->
-  <xacro:property name="JOINT_ARM_R_4_LOWER_LIMIT" value="${radians(-0.01)}"/>
-  <xacro:property name="JOINT_ARM_R_4_UPPER_LIMIT" value="${radians(157)}"/>
-  <xacro:property name="JOINT_ARM_R_5_LOWER_LIMIT" value="${radians(-90)}"/>
-  <xacro:property name="JOINT_ARM_R_5_UPPER_LIMIT" value="${radians(90)}"/>
-  <!-- 初期角度が範囲外だとプランニングで失敗するため範囲を広げる -->
-  <xacro:property name="JOINT_ARM_R_6_LOWER_LIMIT" value="${radians(-123)}"/>
-  <xacro:property name="JOINT_ARM_R_6_UPPER_LIMIT" value="${radians(60)}"/>
-  <xacro:property name="JOINT_ARM_R_7_LOWER_LIMIT" value="${radians(-170)}"/>
-  <xacro:property name="JOINT_ARM_R_7_UPPER_LIMIT" value="${radians(170)}"/>
-  <!-- Gazeboの挙動がlimit付近で不安定なため、limitをサーボの可動範囲より少し大きくする -->
-  <!-- 参照: https://github.com/rt-net/sciurus17_description/pull/6 -->
-  <xacro:property name="JOINT_GRIPPER_R_LOWER_LIMIT" value="${radians(-0.05)}"/>
-  <xacro:property name="JOINT_GRIPPER_R_UPPER_LIMIT" value="${radians(86)}"/>
-  <xacro:property name="JOINT_ARM_L_1_LOWER_LIMIT" value="${radians(-90)}"/>
-  <xacro:property name="JOINT_ARM_L_1_UPPER_LIMIT" value="${radians(90)}"/>
-  <!-- 初期角度が範囲外だとプランニングで失敗するため範囲を広げる -->
-  <xacro:property name="JOINT_ARM_L_2_LOWER_LIMIT" value="${radians(0)}"/>
-  <xacro:property name="JOINT_ARM_L_2_UPPER_LIMIT" value="${radians(92)}"/>
-  <xacro:property name="JOINT_ARM_L_3_LOWER_LIMIT" value="${radians(-90)}"/>
-  <xacro:property name="JOINT_ARM_L_3_UPPER_LIMIT" value="${radians(90)}"/>
-  <xacro:property name="JOINT_ARM_L_4_LOWER_LIMIT" value="${radians(-157)}"/>
-  <!-- Gazeboの挙動がlimit付近で不安定なため、limitをサーボの可動範囲より少し大きくする -->
-  <!-- 参照: https://github.com/rt-net/sciurus17_description/pull/6 -->
-  <xacro:property name="JOINT_ARM_L_4_UPPER_LIMIT" value="${radians(0.01)}"/>
-  <xacro:property name="JOINT_ARM_L_5_LOWER_LIMIT" value="${radians(-90)}"/>
-  <xacro:property name="JOINT_ARM_L_5_UPPER_LIMIT" value="${radians(90)}"/>
-  <xacro:property name="JOINT_ARM_L_6_LOWER_LIMIT" value="${radians(-60)}"/>
-  <!-- 初期角度が範囲外だとプランニングで失敗するため範囲を広げる -->
-  <xacro:property name="JOINT_ARM_L_6_UPPER_LIMIT" value="${radians(123)}"/>
-  <xacro:property name="JOINT_ARM_L_7_LOWER_LIMIT" value="${radians(-170)}"/>
-  <xacro:property name="JOINT_ARM_L_7_UPPER_LIMIT" value="${radians(170)}"/>
-  <xacro:property name="JOINT_GRIPPER_L_LOWER_LIMIT" value="${radians(-86)}"/>
-  <!-- Gazeboの挙動がlimit付近で不安定なため、limitをサーボの可動範囲より少し大きくする -->
-  <!-- 参照: https://github.com/rt-net/sciurus17_description/pull/6 -->
-  <xacro:property name="JOINT_GRIPPER_L_UPPER_LIMIT" value="${radians(0.05)}"/>
   <xacro:property name="COLOR_LINK_BASE" value="white"/>
   <xacro:property name="COLOR_LINK_BODY" value="white"/>
@@ -151,9 +28,11 @@
   <xacro:property name="COLOR_LINK_ARM" value="white"/>
   <xacro:property name="COLOR_LINK_GRIPPER" value="red"/>
+  <xacro:property name="NAME_WORLD_LINK" value="world"/>
   <!-- Used for fixing robot 'base_link'  to Gazebo 'world' -->
   <link name="world"/>
   <joint name="${NAME_JOINT_BASE}" type="fixed">
-    <parent link="world"/>
+    <parent link="${NAME_WORLD_LINK}"/>
     <child link="${NAME_LINK_BASE}"/>
+    <origin rpy="0 0 0.0" xyz="0.0 0.0 0.0"/>
   </joint>
   <xacro:sciurus17_body/>

File: urdf/sciurus17_body.xacro (robot description, xacro)
@@ -16,7 +16,7 @@
       </collision>
       <inertial>
-        <origin rpy="0 0 0" xyz="-24.012e-03 0.139e-03 59.566e-03"/>
-        <inertia ixx="6398092.663e-09" ixy="-6808.969e-09" ixz="-331509.04e-09" iyy="7611664.357e-09" iyz="2026.354e-09" izz="6331936.461e-09"/>
-        <mass value="1722.937e-03"/>
+        <mass value="0.558729"/>
+        <origin xyz="-16.908e-03 0.229e-03 35.241e-03" rpy="0 0 0"/>
+        <inertia ixx="571563.874e-09" ixy="1950.733e-09" iyy="1152259.602e-09" ixz="-18241.875e-09" iyz="1010.978e-09" izz="1419689.940e-09" />
       </inertial>
     </link>
@@ -24,5 +24,5 @@
       <parent link="${NAME_LINK_BASE}" />
       <child link="${NAME_LINK_BODY}" />
-      <origin xyz="0.0 0.0 0.1315" rpy="0 0 0"/>
+      <origin xyz="0.0 0.0 0.0515" rpy="0 0 0"/>
       <limit
         lower="${JOINT_BODY_LOWER_LIMIT}"
@@ -47,7 +47,7 @@
       </collision>
       <inertial>
-       <origin rpy="0 0 0" xyz="57.11e-03 0.372e-03 238.229e-03"/>
-        <inertia ixx="15601031.58e-09" ixy="-15890.903e-09" ixz="-3805596.494e-09" iyy="13969734.5e-09" iyz="-20695.221e-09" izz="8327993.097e-09"/>
-        <mass value="1482.929e-03"/>
+        <mass value="1.566769"/>
+        <origin xyz="57.037e-03 0.359e-03 165.478e-03" rpy="0 0 0"/>
+        <inertia ixx="12482584.603e-09" ixy="-16505.487e-09" iyy="10797139.881e-09" ixz="-3288844.562e-09" iyz="-31874.858e-09" izz="8446450.442e-09" />
       </inertial>
     </link>

File: urdf/sciurus17_head.xacro (robot description, xacro)
@@ -5,5 +5,8 @@
       <parent link="${NAME_LINK_BODY}" />
       <child link="${NAME_LINK_NECK_1}" />
+      <!--
       <origin xyz="0.08083 0.0 0.3395" rpy="0 0 0"/>
+      -->
+      <origin xyz="0.08083 0.0 0.2595" rpy="0 0 0"/>
       <limit
         lower="${JOINT_NECK_1_LOWER_LIMIT}"

File: urdf/sciurus17_left_arm.xacro (robot description, xacro)
@@ -5,5 +5,8 @@
       <parent link="${NAME_LINK_BODY}" />
       <child link="${NAME_LINK_ARM_L_1}" />
+      <!--
       <origin xyz="0.08083 0.0965 0.2885" rpy="0 0 0"/>
+      -->
+      <origin xyz="0.08083 0.0965 0.2085" rpy="0 0 0"/>
       <limit
         lower="${JOINT_ARM_L_1_LOWER_LIMIT}"

File: urdf/sciurus17_left_gripper.xacro (robot description, xacro)
@@ -58,5 +58,5 @@
     -->
     <joint name="${NAME_JOINT_GRIPPER_L_B}_mimic" type="fixed">
-      <parent link="world" />
+      <parent link="${NAME_WORLD_LINK}" />
       <child link="dummy_mimic_fix_l" />
     </joint>

File: urdf/sciurus17_right_arm.xacro (robot description, xacro)
@@ -5,5 +5,8 @@
       <parent link="${NAME_LINK_BODY}" />
       <child link="${NAME_LINK_ARM_R_1}" />
+      <!--
       <origin xyz="0.08083 -0.0965 0.2885" rpy="0 0 0"/>
+      -->
+      <origin xyz="0.08083 -0.0965 0.2085" rpy="0 0 0"/>
       <limit
         lower="${JOINT_ARM_R_1_LOWER_LIMIT}"

File: urdf/sciurus17_right_gripper.xacro (robot description, xacro)
@@ -59,5 +59,5 @@
     -->
     <joint name="${NAME_JOINT_GRIPPER_R_B}_mimic" type="fixed">
-      <parent link="world" />
+      <parent link="${NAME_WORLD_LINK}" />
       <child link="dummy_mimic_fix_r" />
     </joint>

Commit message: use_gazeboがtrueの時だけworldリンクを定義する

File: urdf/sciurus17.urdf.xacro (robot description, xacro)
@@ -151,10 +151,12 @@
   <xacro:property name="COLOR_LINK_ARM" value="white"/>
   <xacro:property name="COLOR_LINK_GRIPPER" value="red"/>
-  <!-- Used for fixing robot 'base_link'  to Gazebo 'world' -->
-  <link name="world"/>
-  <joint name="${NAME_JOINT_BASE}" type="fixed">
-    <parent link="world"/>
-    <child link="${NAME_LINK_BASE}"/>
-  </joint>
+  <xacro:if value="$(arg use_gazebo)">
+    <!-- Used for fixing robot 'base_link'  to Gazebo 'world' -->
+    <link name="world"/>
+    <joint name="${NAME_JOINT_BASE}" type="fixed">
+      <parent link="world"/>
+      <child link="${NAME_LINK_BASE}"/>
+    </joint>
+  </xacro:if>
   <xacro:sciurus17_body/>
   <xacro:sciurus17_head/>
