Commit message: マテリアルのproperty定義を廃止

File: urdf/sciurus17.urdf.xacro (robot description, xacro)
@@ -94,9 +94,4 @@
   <!-- 参照: https://github.com/rt-net/sciurus17_description/pull/6 -->
   <xacro:property name="JOINT_GRIPPER_L_UPPER_LIMIT" value="${radians(0.05)}"/>
-  <xacro:property name="COLOR_LINK_BASE" value="white"/>
-  <xacro:property name="COLOR_LINK_BODY" value="white"/>
-  <xacro:property name="COLOR_LINK_HEAD" value="white"/>
-  <xacro:property name="COLOR_LINK_ARM" value="white"/>
-  <xacro:property name="COLOR_LINK_GRIPPER" value="red"/>
   <!-- Used for fixing robot 'base_link'  to Gazebo 'world' -->
   <link name="world"/>

File: urdf/sciurus17_body.xacro (robot description, xacro)
@@ -7,5 +7,5 @@
           <mesh filename="package://sciurus17_description/meshes/visual/Base.stl" scale="1.0 1.0 1.0"/>
         </geometry>
-        <material name="${COLOR_LINK_BASE}"/>
+        <material name="white"/>
       </visual>
       <collision>
@@ -38,5 +38,5 @@
           <mesh filename="package://sciurus17_description/meshes/visual/Body.stl" scale="1.0 1.0 1.0"/>
         </geometry>
-        <material name="${COLOR_LINK_BODY}"/>
+        <material name="white"/>
       </visual>
       <collision>

File: urdf/sciurus17_head.xacro (robot description, xacro)
@@ -19,5 +19,5 @@
           <mesh filename="package://sciurus17_description/meshes/visual/Neck1.stl" scale="1.0 1.0 1.0"/>
         </geometry>
-        <material name="${COLOR_LINK_HEAD}"/>
+        <material name="white"/>
       </visual>
       <collision>
@@ -50,5 +50,5 @@
           <mesh filename="package://sciurus17_description/meshes/visual/Neck2.stl" scale="1.0 1.0 1.0"/>
         </geometry>
-        <material name="${COLOR_LINK_HEAD}"/>
+        <material name="white"/>
       </visual>
       <collision>

File: urdf/sciurus17_left_arm.xacro (robot description, xacro)
@@ -20,5 +20,5 @@
           <mesh filename="package://sciurus17_description/meshes/visual/L_Link1.stl" scale="1.0 1.0 1.0"/>
         </geometry>
-        <material name="${COLOR_LINK_ARM}"/>
+        <material name="white"/>
       </visual>
       <collision>
@@ -52,5 +52,5 @@
           <mesh filename="package://sciurus17_description/meshes/visual/L_Link2.stl" scale="1.0 1.0 1.0"/>
         </geometry>
-        <material name="${COLOR_LINK_ARM}"/>
+        <material name="white"/>
       </visual>
       <collision>
@@ -84,5 +84,5 @@
           <mesh filename="package://sciurus17_description/meshes/visual/L_Link3.stl" scale="1.0 1.0 1.0"/>
         </geometry>
-        <material name="${COLOR_LINK_ARM}"/>
+        <material name="white"/>
       </visual>
       <collision>
@@ -116,5 +116,5 @@
           <mesh filename="package://sciurus17_description/meshes/visual/L_Link4.stl" scale="1.0 1.0 1.0"/>
         </geometry>
-        <material name="${COLOR_LINK_ARM}"/>
+        <material name="white"/>
       </visual>
       <collision>
@@ -148,5 +148,5 @@
           <mesh filename="package://sciurus17_description/meshes/visual/L_Link5.stl" scale="1.0 1.0 1.0"/>
         </geometry>
-        <material name="${COLOR_LINK_ARM}"/>
+        <material name="white"/>
       </visual>
       <visual>
@@ -191,5 +191,5 @@
           <cylinder length="0.001" radius="0.001"/>
         </geometry>
-        <material name="${COLOR_LINK_ARM}"/>
+        <material name="white"/>
       </visual>
       <collision>
@@ -218,5 +218,5 @@
           <mesh filename="package://sciurus17_description/meshes/visual/L_Link6.stl" scale="1.0 1.0 1.0"/>
         </geometry>
-        <material name="${COLOR_LINK_ARM}"/>
+        <material name="white"/>
       </visual>
       <collision>

File: urdf/sciurus17_left_gripper.xacro (robot description, xacro)
@@ -8,5 +8,5 @@
           <mesh filename="package://sciurus17_description/meshes/visual/L_Link7.stl" scale="1.0 1.0 1.0"/>
         </geometry>
-        <material name="${COLOR_LINK_GRIPPER}"/>
+        <material name="red"/>
       </visual>
       <collision>
@@ -40,5 +40,5 @@
           <mesh filename="package://sciurus17_description/meshes/visual/L_GripperA.stl" scale="1.0 1.0 1.0"/>
         </geometry>
-        <material name="${COLOR_LINK_GRIPPER}"/>
+        <material name="red"/>
       </visual>
       <collision>
@@ -73,5 +73,5 @@
           <mesh filename="package://sciurus17_description/meshes/visual/L_GripperB.stl" scale="1.0 1.0 1.0"/>
         </geometry>
-        <material name="${COLOR_LINK_GRIPPER}"/>
+        <material name="red"/>
       </visual>
       <collision>

File: urdf/sciurus17_right_arm.xacro (robot description, xacro)
@@ -20,5 +20,5 @@
           <mesh filename="package://sciurus17_description/meshes/visual/R_Link1.stl" scale="1.0 1.0 1.0"/>
         </geometry>
-        <material name="${COLOR_LINK_ARM}"/>
+        <material name="white"/>
       </visual>
       <collision>
@@ -52,5 +52,5 @@
           <mesh filename="package://sciurus17_description/meshes/visual/R_Link2.stl" scale="1.0 1.0 1.0"/>
         </geometry>
-        <material name="${COLOR_LINK_ARM}"/>
+        <material name="white"/>
       </visual>
       <collision>
@@ -84,5 +84,5 @@
           <mesh filename="package://sciurus17_description/meshes/visual/L_Link3.stl" scale="1.0 1.0 1.0"/>
         </geometry>
-        <material name="${COLOR_LINK_ARM}"/>
+        <material name="white"/>
       </visual>
       <collision>
@@ -116,5 +116,5 @@
           <mesh filename="package://sciurus17_description/meshes/visual/R_Link4.stl" scale="1.0 1.0 1.0"/>
         </geometry>
-        <material name="${COLOR_LINK_ARM}"/>
+        <material name="white"/>
       </visual>
       <collision>
@@ -148,5 +148,5 @@
           <mesh filename="package://sciurus17_description/meshes/visual/R_Link5.stl" scale="1.0 1.0 1.0"/>
         </geometry>
-        <material name="${COLOR_LINK_ARM}"/>
+        <material name="white"/>
       </visual>
       <visual>
@@ -191,5 +191,5 @@
           <cylinder length="0.001" radius="0.001"/>
         </geometry>
-        <material name="${COLOR_LINK_ARM}"/>
+        <material name="white"/>
       </visual>
       <collision>
@@ -218,5 +218,5 @@
           <mesh filename="package://sciurus17_description/meshes/visual/R_Link6.stl" scale="1.0 1.0 1.0"/>
         </geometry>
-        <material name="${COLOR_LINK_ARM}"/>
+        <material name="white"/>
       </visual>
       <collision>

File: urdf/sciurus17_right_gripper.xacro (robot description, xacro)
@@ -8,5 +8,5 @@
           <mesh filename="package://sciurus17_description/meshes/visual/R_Link7.stl" scale="1.0 1.0 1.0"/>
         </geometry>
-        <material name="${COLOR_LINK_GRIPPER}"/>
+        <material name="red"/>
       </visual>
       <collision>
@@ -41,5 +41,5 @@
           <mesh filename="package://sciurus17_description/meshes/visual/R_GripperA.stl" scale="1.0 1.0 1.0"/>
         </geometry>
-        <material name="${COLOR_LINK_GRIPPER}"/>
+        <material name="red"/>
       </visual>
       <collision>
@@ -75,5 +75,5 @@
           <mesh filename="package://sciurus17_description/meshes/visual/R_GripperB.stl" scale="1.0 1.0 1.0"/>
         </geometry>
-        <material name="${COLOR_LINK_GRIPPER}"/>
+        <material name="red"/>
       </visual>
       <collision>

Commit message: カメラリンク名のprefixを廃止

File: urdf/sciurus17.urdf.xacro (robot description, xacro)
@@ -25,6 +25,4 @@
   <xacro:arg name="gz_control_config_package" default="" />
   <xacro:arg name="gz_control_config_file_path" default="" />
-  <xacro:property name="NAME_HEAD_CAMERA_PREFIX" value="head_camera"/>
-  <xacro:property name="NAME_CHEST_CAMERA_PREFIX" value="chest_camera"/>
   <material name="white">
     <color rgba="0.9 0.9 0.9 1.0"/>
@@ -112,16 +110,16 @@
       gz_control_config_file_path="$(arg gz_control_config_file_path)"/>
     <xacro:sciurus17_gazebo_ros2_control_settings/>
-    <joint name="${NAME_HEAD_CAMERA_PREFIX}_color_joint" type="fixed">
+    <joint name="head_camera_color_joint" type="fixed">
       <origin xyz="0 0.015 0" rpy="0 0 0" />
       <parent link="head_camera_link" />
-      <child link="${NAME_HEAD_CAMERA_PREFIX}_color_frame" />
+      <child link="head_camera_color_frame" />
     </joint>
-    <link name="${NAME_HEAD_CAMERA_PREFIX}_color_frame"/>
-    <joint name="${NAME_HEAD_CAMERA_PREFIX}_color_optical_joint" type="fixed">
+    <link name="head_camera_color_frame"/>
+    <joint name="head_camera_color_optical_joint" type="fixed">
       <origin xyz="0 0 0" rpy="${radians(-90)} 0 ${radians(-90)}" />
-      <parent link="${NAME_HEAD_CAMERA_PREFIX}_color_frame" />
-      <child link="${NAME_HEAD_CAMERA_PREFIX}_color_optical_frame" />
+      <parent link="head_camera_color_frame" />
+      <child link="head_camera_color_optical_frame" />
     </joint>
-    <link name="${NAME_HEAD_CAMERA_PREFIX}_color_optical_frame"/>
+    <link name="head_camera_color_optical_frame"/>
   </xacro:if>
 </robot>

File: urdf/sciurus17_gazebo.xacro (robot description, xacro)
@@ -53,10 +53,10 @@
     </gazebo>
     <xacro:if value="${use_gazebo_head_camera}">
-      <gazebo reference="${NAME_HEAD_CAMERA_PREFIX}_color_frame">
+      <gazebo reference="head_camera_color_frame">
         <sensor name="sim_realsense_d415" type="rgbd_camera">
           <update_rate>10</update_rate>
           <always_on>true</always_on>
-          <topic>${NAME_HEAD_CAMERA_PREFIX}</topic>
-          <frame_id>${NAME_HEAD_CAMERA_PREFIX}_color_frame</frame_id>
+          <topic>head_camera</topic>
+          <frame_id>head_camera_color_frame</frame_id>
           <camera name="realsense_d415">
             <xacro:property name="head_camera_width" value="640"/>
@@ -79,5 +79,5 @@
               </clip>
             </depth_camera>
-            <optical_frame_id>${NAME_HEAD_CAMERA_PREFIX}_color_optical_frame</optical_frame_id>
+            <optical_frame_id>head_camera_color_optical_frame</optical_frame_id>
             <lens>
               <intrinsics>
@@ -103,11 +103,11 @@
     <xacro:if value="${use_gazebo_chest_camera}">
       <gazebo reference="chest_camera_link">
-        <sensor name="${NAME_CHEST_CAMERA_PREFIX}" type="camera">
+        <sensor name="chest_camera" type="camera">
           <pose relative_to="chest_camera_link">0 0 0 ${radians(90)} ${radians(-90)} 0</pose>
           <update_rate>10</update_rate>
           <always_on>true</always_on>
-          <topic>${NAME_CHEST_CAMERA_PREFIX}/image_raw</topic>
+          <topic>chest_camera/image_raw</topic>
           <frame_id>chest_camera_link</frame_id>
-          <camera name="${NAME_CHEST_CAMERA_PREFIX}">
+          <camera name="chest_camera">
             <xacro:property name="chest_camera_width" value="640"/>
             <xacro:property name="chest_camera_height" value="360"/>
